Commit message: sort files

File: src/robot_model/robot/robot.urdf.xacro (robot description, xacro)
@@ -5,4 +5,5 @@
 	<xacro:include filename="$(find robot_model)/urdf/body/robot_body.urdf.xacro" />
 	<xacro:include filename="$(find robot_model)/urdf/robot_model.gazebo.xacro" />
+	<xacro:include filename="$(find robot_model)/urdf/lidar.xacro" />
 	<!-- Wheel parameters -->
 	<xacro:property name="wheel_offset_x" value="0.2225" />    <!-- x,y,z in translation from base_link to the center of the wheel -->
@@ -26,4 +27,7 @@
 			<origin xyz="-${wheel_offset_x} -${wheel_offset_y} ${wheel_offset_z}" rpy="0 0 0" />
 		</xacro:omni_wheel>
+		<xacro:lidar parent="robot_body_link" laser_name="1">
+			<origin xyz="0 0 0.3" rpy="0 0 0" />
+		</xacro:lidar>
 	</xacro:macro>
 	<xacro:robot />

File: src/robot_model/urdf/wheel/omni_wheel.urdf.xacro (robot description, xacro)
@@ -1,5 +1,5 @@
 <?xml version="1.0"?>
 <robot name="wheel" xmlns:xacro="http://www.ros.org/wiki/xacro">
-  <xacro:include filename="inertial.urdf.xacro"/>
+  <xacro:include filename="$(find robot_model)/urdf/physics/inertial.urdf.xacro"/>
   <xacro:property name="PI" value="3.1415926535897931" />
   <!-- Wheels -->

Commit message: ultrasonic (broken)

File: src/robot_model/robot/robot.urdf.xacro (robot description, xacro)
@@ -5,5 +5,5 @@
 	<xacro:include filename="$(find robot_model)/urdf/body/robot_body.urdf.xacro" />
 	<xacro:include filename="$(find robot_model)/urdf/robot_model.gazebo.xacro" />
-	<xacro:include filename="$(find robot_model)/urdf/sensors/lidar.xacro" />
+	<xacro:include filename="$(find robot_model)/urdf/sensors/sensors.xacro" />
 	<!-- Wheel parameters -->
 	<xacro:property name="wheel_offset_x" value="0.2225" />    <!-- x,y,z in translation from base_link to the center of the wheel -->
@@ -30,4 +30,7 @@
 			<origin xyz="0 0 0.3" rpy="0 0 0" />
 		</xacro:lidar>
+		<!-- <xacro:ultrasonic parent="robot_body_link" sensor_name="1">
+			<origin xyz="0.1 0 0.3" rpy="0 0 0" />
+		</xacro:ultrasonic> -->
 	</xacro:macro>
 	<xacro:robot />
@@ -43,4 +46,6 @@
 			<joint_name>back_left_wheel_joint</joint_name>
 			<joint_name>back_right_wheel_joint</joint_name>
+			<joint_name>1_laser_joint</joint_name>
+			<!-- <joint_name>ultrasonic</joint_name> -->
 		</plugin>
 	</gazebo>

File: src/robot_model/urdf/material.xacro (robot description, xacro)
@@ -1,5 +1,5 @@
 <?xml version="1.0"?>
-<robot>
-    <material name="white" xmlns:xacro="http://www.ros.org/wiki/xacro">
+<robot xmlns:xacro="http://www.ros.org/wiki/xacro">
+    <material name="white">
         <color rgba="1 1 1 1" />
     </material>

File: src/robot_model/urdf/sensors/sensors.xacro (robot description, xacro)
@@ -56,3 +56,48 @@
         </gazebo>
     </xacro:macro>
+    <xacro:macro name="ultrasonic" params="parent *origin sensor_name">
+        <joint name="${sensor_name}_ultrasonic_joint" type="fixed">
+            <parent link="${parent}" />
+            <child link="${sensor_name}_ultrasonic_frame" />
+            <xacro:insert_block name="origin" />
+        </joint>
+        <link name="${sensor_name}_ultrasonic_frame">
+            <visual>
+                <geometry>
+                    <cylinder radius="0.05" length="0.04" />
+                </geometry>
+                <material name="blue" />
+            </visual>
+            <collision>
+                <geometry>
+                    <cylinder radius="0.05" length="0.04" />
+                </geometry>
+            </collision>
+            <inertial>
+                <origin xyz="0 0 0" rpy="0 0 0" />
+                <mass value="0.1" />
+                <xacro:cylinder_inertia m="0.1" h="0.04" r="0.05" />
+            </inertial>
+        </link>
+        <gazebo reference="${sensor_name}_ultrasonic_frame">
+            <material>Gazebo/Blue</material>
+            <sensor name="ultrasonic" type="sonar">
+                <pose> 0 0 0 0 0 0 </pose>
+                <visualize>true</visualize>
+                <update_rate>10</update_rate>
+                <sonar>
+                    <radiation>ultrasonic</radiation>
+                    <min_range>0.3</min_range>
+                    <max_range>12</max_range>
+                </sonar>
+                <plugin name="ultrasonic_controller" filename="libgazebo_ros_range.so">
+                    <ros>
+                        <argument>~/out:=range</argument>
+                    </ros>
+                    <output_type>sensor_msgs/Range</output_type>
+                    <frame_name>${sensor_name}_ultrasonic_frame</frame_name>
+                </plugin>
+            </sensor>
+        </gazebo>
+    </xacro:macro>
 </robot>

Commit message: Aligned ultrasonic

File: src/robot_model/robot/robot.urdf.xacro (robot description, xacro)
@@ -27,10 +27,10 @@
 			<origin xyz="-${wheel_offset_x} -${wheel_offset_y} ${wheel_offset_z}" rpy="0 0 0" />
 		</xacro:omni_wheel>
-		<xacro:lidar parent="robot_body_link" laser_name="1">
+		<!-- <xacro:lidar parent="robot_body_link" laser_name="1">
 			<origin xyz="0 0 0.3" rpy="0 0 0" />
-		</xacro:lidar>
-		<!-- <xacro:ultrasonic parent="robot_body_link" sensor_name="1">
-			<origin xyz="0.1 0 0.3" rpy="0 0 0" />
-		</xacro:ultrasonic> -->
+		</xacro:lidar> -->
+		<xacro:ultrasonic parent="robot_body_link" sensor_name="1">
+			<origin xyz="0.32 0 0.2" rpy="0 -77 0" />
+		</xacro:ultrasonic>
 	</xacro:macro>
 	<xacro:robot />
@@ -46,6 +46,4 @@
 			<joint_name>back_left_wheel_joint</joint_name>
 			<joint_name>back_right_wheel_joint</joint_name>
-			<!-- <joint_name>1_laser_joint</joint_name> -->
-			<!-- <joint_name>ultrasonic</joint_name> -->
 		</plugin>
 	</gazebo>

File: src/robot_model/urdf/sensors/sensors.xacro (robot description, xacro)
@@ -91,5 +91,5 @@
                     <max_range>12</max_range>
                 </sonar>
-                <plugin name="ultrasonic_controller" filename="libgazebo_ros_range.so">
+                <plugin name="ultrasonic_controller" filename="libgazebo_ros_sonar_plugin.so">
                     <ros>
                         <argument>~/out:=range</argument>
