Commit message: rename and move files

File: src/followme_robot_model/robot/robot.urdf.xacro (robot description, xacro)
@@ -2,8 +2,8 @@
 <robot name="robot" xmlns:xacro="http://www.ros.org/wiki/xacro">
 	<!-- Import summit XL wheels -->
-	<xacro:include filename="$(find robot_model)/urdf/wheel/omni_wheel.urdf.xacro" />
-	<xacro:include filename="$(find robot_model)/urdf/body/robot_body.urdf.xacro" />
-	<xacro:include filename="$(find robot_model)/urdf/robot_model.gazebo.xacro" />
-	<xacro:include filename="$(find robot_model)/urdf/sensors/sensors.xacro" />
+	<xacro:include filename="$(find followme_robot_model)/urdf/wheel/omni_wheel.urdf.xacro" />
+	<xacro:include filename="$(find followme_robot_model)/urdf/body/robot_body.urdf.xacro" />
+	<xacro:include filename="$(find followme_robot_model)/urdf/followme_robot_model.gazebo.xacro" />
+	<xacro:include filename="$(find followme_robot_model)/urdf/sensors/sensors.xacro" />
 	<!-- Wheel parameters -->
 	<xacro:property name="wheel_offset_x" value="0.2225" />    <!-- x,y,z in translation from base_link to the center of the wheel -->
@@ -27,7 +27,7 @@
 			<origin xyz="-${wheel_offset_x} -${wheel_offset_y} ${wheel_offset_z}" rpy="0 0 0" />
 		</xacro:omni_wheel>
-		<!-- <xacro:lidar parent="robot_body_link" laser_name="1">
+		<xacro:lidar parent="robot_body_link" laser_name="1">
 			<origin xyz="0 0 0.3" rpy="0 0 0" />
-		</xacro:lidar> -->
+		</xacro:lidar>
 		<xacro:ultrasonic parent="robot_body_link" sensor_name="1">
 			<origin xyz="0.32 0 0.2" rpy="0 -77 0" />

File: src/followme_robot_model/urdf/body/robot_body.urdf.xacro (robot description, xacro)
@@ -2,5 +2,5 @@
 <robot name="robot" xmlns:xacro="http://www.ros.org/wiki/xacro">
   <xacro:macro name="robot_body" params="wheel_radius">
-      <xacro:include filename="$(find robot_model)/urdf/robot_model.gazebo.xacro" />
+      <xacro:include filename="$(find followme_robot_model)/urdf/followme_robot_model.gazebo.xacro" />
 	  <!-- Robot mechanical and motor parameters -->
 	  <xacro:property name="PI" value="3.1415926535897931"/>
@@ -29,5 +29,5 @@
        <origin xyz="0 0 0" rpy="0 0 0" />
        <geometry>
-	       <mesh filename="file://$(find robot_model)/meshes/body/robot_body.dae"/>
+	       <mesh filename="file://$(find followme_robot_model)/meshes/body/robot_body.dae"/>
        </geometry>
        <material name="darkgrey">
@@ -38,5 +38,5 @@
        <origin xyz="0 0 0" rpy="0 0 0 " />
        <geometry>
-         <mesh filename="file://$(find robot_model)/meshes/body/robot_body.dae"/>
+         <mesh filename="file://$(find followme_robot_model)/meshes/body/robot_body.dae"/>
        </geometry>
     </collision>

File: src/followme_robot_model/urdf/sensors/sensors.xacro (robot description, xacro)
@@ -1,6 +1,6 @@
 <?xml version="1.0"?>
 <robot xmlns:xacro="http://www.ros.org/wiki/xacro">
-    <xacro:include filename="$(find robot_model)/urdf/physics/inertial.urdf.xacro" />
-    <xacro:include filename="$(find robot_model)/urdf/material.xacro" />
+    <xacro:include filename="$(find followme_robot_model)/urdf/physics/inertial.urdf.xacro" />
+    <xacro:include filename="$(find followme_robot_model)/urdf/material.xacro" />
     <xacro:macro name="lidar" params="parent *origin laser_name">
         <joint name="${laser_name}_laser_joint" type="fixed">

File: src/followme_robot_model/urdf/wheel/omni_wheel.urdf.xacro (robot description, xacro)
@@ -1,5 +1,5 @@
 <?xml version="1.0"?>
 <robot name="wheel" xmlns:xacro="http://www.ros.org/wiki/xacro">
-  <xacro:include filename="$(find robot_model)/urdf/physics/inertial.urdf.xacro"/>
+  <xacro:include filename="$(find followme_robot_model)/urdf/physics/inertial.urdf.xacro"/>
   <xacro:property name="PI" value="3.1415926535897931" />
   <!-- Wheels -->
@@ -24,5 +24,5 @@
         <origin xyz="0 0 0" rpy="0 0 0" />
         <geometry>
-          <mesh filename="file://$(find robot_model)/meshes/wheels/omni_wheel_${reflect}.dae" />
+          <mesh filename="file://$(find followme_robot_model)/meshes/wheels/omni_wheel_${reflect}.dae" />
         </geometry>
       </visual>

Commit message: changes

File: src/followme_robot_model/robot/robot.urdf.xacro (robot description, xacro)
@@ -27,5 +27,5 @@
 			<origin xyz="-${wheel_offset_x} -${wheel_offset_y} ${wheel_offset_z}" rpy="0 0 0" />
 		</xacro:omni_wheel>
-		<xacro:lidar parent="robot_body_link" laser_name="1">
+		<xacro:lidar parent="robot_body_link" laser_name="1" range="10">
 			<origin xyz="0 0 0.3" rpy="0 0 0" />
 		</xacro:lidar>

File: src/followme_robot_model/urdf/sensors/sensors.xacro (robot description, xacro)
@@ -3,5 +3,5 @@
     <xacro:include filename="$(find followme_robot_model)/urdf/physics/inertial.urdf.xacro" />
     <xacro:include filename="$(find followme_robot_model)/urdf/material.xacro" />
-    <xacro:macro name="lidar" params="parent *origin laser_name">
+    <xacro:macro name="lidar" params="parent *origin laser_name range:=12">
         <joint name="${laser_name}_laser_joint" type="fixed">
             <parent link="${parent}" />
@@ -43,5 +43,5 @@
                     <range>
                         <min>0.3</min>
-                        <max>12</max>
+                        <max>${range}</max>
                     </range>
                 </ray>
@@ -56,5 +56,5 @@
         </gazebo>
     </xacro:macro>
-    <xacro:macro name="ultrasonic" params="parent *origin sensor_name">
+    <xacro:macro name="ultrasonic" params="parent *origin sensor_name range:=12">
         <joint name="${sensor_name}_ultrasonic_joint" type="fixed">
             <parent link="${parent}" />
@@ -89,5 +89,5 @@
                     <radiation>ultrasonic</radiation>
                     <min_range>0.3</min_range>
-                    <max_range>12</max_range>
+                    <max_range>${range}</max_range>
                 </sonar>
                 <plugin name="ultrasonic_controller" filename="libgazebo_ros_sonar_plugin.so">

Commit message: Buggy Depth Camera

File: src/followme_robot_model/robot/robot.urdf.xacro (robot description, xacro)
@@ -30,7 +30,7 @@
 			<origin xyz="0 0 0.3" rpy="0 0 0" />
 		</xacro:lidar>
-		<xacro:ultrasonic parent="robot_body_link" sensor_name="1">
-			<origin xyz="0.32 0 0.2" rpy="0 -77 0" />
-		</xacro:ultrasonic>
+		<xacro:camera parent="robot_body_link" sensor_name="1" range="8">
+			<origin xyz="0.32 0 0.42" rpy="0 0 0" />
+		</xacro:camera>
 	</xacro:macro>
 	<xacro:robot />

File: src/followme_robot_model/urdf/sensors/sensors.xacro (robot description, xacro)
@@ -1,6 +1,6 @@
 <?xml version="1.0"?>
 <robot xmlns:xacro="http://www.ros.org/wiki/xacro">
-    <xacro:include filename="$(find followme_robot_model)/urdf/physics/inertial.urdf.xacro" />
-    <xacro:include filename="$(find followme_robot_model)/urdf/material.xacro" />
+    <xacro:include filename="$(find robot_model)/urdf/physics/inertial.urdf.xacro" />
+    <xacro:include filename="$(find robot_model)/urdf/material.xacro" />
     <xacro:macro name="lidar" params="parent *origin laser_name range:=12">
         <joint name="${laser_name}_laser_joint" type="fixed">
@@ -56,45 +56,54 @@
         </gazebo>
     </xacro:macro>
-    <xacro:macro name="ultrasonic" params="parent *origin sensor_name range:=12">
-        <joint name="${sensor_name}_ultrasonic_joint" type="fixed">
+    <xacro:macro name="camera" params="parent *origin sensor_name range:=8">
+        <joint name="${sensor_name}_camera_joint" type="fixed">
             <parent link="${parent}" />
-            <child link="${sensor_name}_ultrasonic_frame" />
+            <child link="${sensor_name}_camera_frame" />
             <xacro:insert_block name="origin" />
         </joint>
-        <link name="${sensor_name}_ultrasonic_frame">
+        <link name="${sensor_name}_camera_frame">
             <visual>
                 <geometry>
-                    <cylinder radius="0.05" length="0.04" />
+                    <box size="0.01 0.06 0.03"/>
                 </geometry>
-                <material name="blue" />
+                <material name="red" />
             </visual>
             <collision>
                 <geometry>
-                    <cylinder radius="0.05" length="0.04" />
+                    <box size="0.01 0.06 0.03"/>
                 </geometry>
             </collision>
             <inertial>
-                <origin xyz="0 0 0" rpy="0 0 0" />
+                <origin xyz="0 0 0" rpy="${PI} 0 0" />
                 <mass value="0.1" />
-                <xacro:cylinder_inertia m="0.1" h="0.04" r="0.05" />
+                <xacro:solid_cuboid_inertia m="0.1" h="0.01" d="0.06" w="0.03" />
             </inertial>
         </link>
-        <gazebo reference="${sensor_name}_ultrasonic_frame">
-            <material>Gazebo/Blue</material>
-            <sensor name="ultrasonic" type="sonar">
+        <gazebo reference="${sensor_name}_camera_frame">
+            <material>Gazebo/Red</material>
+            <sensor name="camera" type="depth">
                 <pose> 0 0 0 0 0 0 </pose>
                 <visualize>true</visualize>
                 <update_rate>10</update_rate>
-                <sonar>
-                    <radiation>ultrasonic</radiation>
-                    <min_range>0.3</min_range>
-                    <max_range>${range}</max_range>
-                </sonar>
-                <plugin name="ultrasonic_controller" filename="libgazebo_ros_sonar_plugin.so">
+                <camera>
+                    <horizontal_fov>1.089</horizontal_fov>
+                    <image>
+                        <format>B8R8G8</format>
+                        <width>640</width>
+                        <height>480</height>
+                    </image>
+                    <clip>
+                        <near>0.05</near>
+                        <far>${range}</far>
+                    </clip>
+                </camera>
+                <plugin name="camera_controller" filename="libgazebo_ros_camera.so">
                     <ros>
                         <argument>~/out:=range</argument>
                     </ros>
                     <output_type>sensor_msgs/Range</output_type>
-                    <frame_name>${sensor_name}_ultrasonic_frame</frame_name>
+                    <frame_name>${sensor_name}_camera_frame</frame_name>
+                    <min_depth>0.1</min_depth>
+                    <max_depth>100.0</max_depth>
                 </plugin>
             </sensor>

Commit message: try to fix sensor output

File: src/followme_robot_model/robot/robot.urdf.xacro (robot description, xacro)
@@ -27,7 +27,7 @@
 			<origin xyz="-${wheel_offset_x} -${wheel_offset_y} ${wheel_offset_z}" rpy="0 0 0" />
 		</xacro:omni_wheel>
-		<xacro:lidar parent="robot_body_link" laser_name="1" range="10">
+		<!-- <xacro:lidar parent="robot_body_link" laser_name="1" range="10">
 			<origin xyz="0 0 0.3" rpy="0 0 0" />
-		</xacro:lidar>
+		</xacro:lidar> -->
 		<xacro:camera parent="robot_body_link" sensor_name="1" range="8">
 			<origin xyz="0.32 0 0.42" rpy="0 0 0" />

File: src/followme_robot_model/urdf/sensors/sensors.xacro (robot description, xacro)
@@ -1,6 +1,6 @@
 <?xml version="1.0"?>
 <robot xmlns:xacro="http://www.ros.org/wiki/xacro">
-    <xacro:include filename="$(find robot_model)/urdf/physics/inertial.urdf.xacro" />
-    <xacro:include filename="$(find robot_model)/urdf/material.xacro" />
+    <xacro:include filename="$(find followme_robot_model)/urdf/physics/inertial.urdf.xacro" />
+    <xacro:include filename="$(find followme_robot_model)/urdf/material.xacro" />
     <xacro:macro name="lidar" params="parent *origin laser_name range:=12">
         <joint name="${laser_name}_laser_joint" type="fixed">
@@ -58,4 +58,5 @@
     <xacro:macro name="camera" params="parent *origin sensor_name range:=8">
         <joint name="${sensor_name}_camera_joint" type="fixed">
+            <axis xyz="0 1 0" />
             <parent link="${parent}" />
             <child link="${sensor_name}_camera_frame" />
@@ -75,5 +76,5 @@
             </collision>
             <inertial>
-                <origin xyz="0 0 0" rpy="${PI} 0 0" />
+                <origin xyz="0 0 0" rpy="0 0 0" />
                 <mass value="0.1" />
                 <xacro:solid_cuboid_inertia m="0.1" h="0.01" d="0.06" w="0.03" />
@@ -104,7 +105,31 @@
                     <output_type>sensor_msgs/Range</output_type>
                     <frame_name>${sensor_name}_camera_frame</frame_name>
-                    <min_depth>0.1</min_depth>
+                    <min_depth>0.01</min_depth>
                     <max_depth>100.0</max_depth>
                 </plugin>
+                <!-- <plugin name="camera_plugin" filename="libgazebo_ros_openni_kinect.so">
+                    <baseline>0.2</baseline>
+                    <alwaysOn>true</alwaysOn>
+                    <updateRate>0.0</updateRate>
+                    <cameraName>${sensor_name}_camera_ir</cameraName>
+                    <imageTopicName>/camera/color/image_raw</imageTopicName>
+                    <cameraInfoTopicName>/camera/color/camera_info</cameraInfoTopicName>
+                    <depthImageTopicName>/camera/depth/image_raw</depthImageTopicName>
+                    <depthImageCameraInfoTopicName>/camera/depth/camera_info</depthImageCameraInfoTopicName>
+                    <pointCloudTopicName>/camera/depth/points</pointCloudTopicName>
+                    <frame_name>${sensor_name}_camera_frame</frame_name>
+                    <pointCloudCutoff>0.5</pointCloudCutoff>
+                    <pointCloudCutoffMax>3.0</pointCloudCutoffMax>
+                    <distortionK1>0</distortionK1>
+                    <distortionK2>0</distortionK2>
+                    <distortionK3>0</distortionK3>
+                    <distortionT1>0</distortionT1>
+                    <distortionT2>0</distortionT2>
+                    <CxPrime>0</CxPrime>
+                    <Cx>0</Cx>
+                    <Cy>0</Cy>
+                    <focalLength>0</focalLength>
+                    <hackBaseline>0</hackBaseline>
+                  </plugin> -->
             </sensor>
         </gazebo>

Commit message: setup working depth camera sensor for gazebo

File: src/followme_robot_model/robot/robot.urdf.xacro (robot description, xacro)
@@ -6,5 +6,5 @@
 	<xacro:include filename="$(find followme_robot_model)/urdf/followme_robot_model.gazebo.xacro" />
 	<xacro:include filename="$(find followme_robot_model)/urdf/sensors/lidar.xacro" />
-	<xacro:include filename="$(find followme_robot_model)/urdf/sensors/camera_depth.xacro" />
+	<!-- <xacro:include filename="$(find followme_robot_model)/urdf/sensors/camera_depth.xacro" /> -->
 	<!-- Wheel parameters -->
 	<xacro:property name="wheel_offset_x" value="0.2225" />    <!-- x,y,z in translation from base_link to the center of the wheel -->
@@ -31,7 +31,5 @@
 			<origin xyz="0 0 0.3" rpy="0 0 0" />
 		</xacro:lidar> -->
-		<xacro:camera parent="robot_body_link" camera_name="1" range="8">
-			<origin xyz="0.32 0 0.42" rpy="0 0 0" />
-		</xacro:camera>
+		<xacro:include filename="$(find followme_robot_model)/urdf/sensors/camera.xacro" />
 	</xacro:macro>
 	<xacro:robot />

File: src/followme_robot_model/urdf/sensors/camera_depth.xacro (robot description, xacro)
@@ -1,5 +1,5 @@
 <?xml version="1.0"?>
 <robot xmlns:xacro="http://www.ros.org/wiki/xacro">
-    <xacro:include filename="$(find robot_model)/urdf/physics/inertial.urdf.xacro" />
+    <xacro:include filename="$(find followme_robot_model)/urdf/physics/inertial.urdf.xacro" />
     <xacro:macro name="camera" params="parent *origin camera_name range:=8">
         <joint name="${camera_name}_camera_joint" type="fixed">
