Commit message: add sensors models and add sonic sensor to robot

File: src/followme_robot_model/robot/robot.urdf.xacro (robot description, xacro)
@@ -1,4 +1,4 @@
 <?xml version="1.0"?>
-<robot name="robot" xmlns:xacro="http://www.ros.org/wiki/xacro">
+<robot name="robot" xmlns:xacro="http://playerstage.sourceforge.net/gazebo/xmlschema/#interface">
 	<!-- Import summit XL wheels -->
 	<xacro:include filename="$(find followme_robot_model)/urdf/wheel/omni_wheel.urdf.xacro" />
@@ -6,4 +6,6 @@
 	<xacro:include filename="$(find followme_robot_model)/urdf/followme_robot_model.gazebo.xacro" />
 	<xacro:include filename="$(find followme_robot_model)/urdf/sensors/lidar.xacro" />
+	<xacro:include filename="$(find followme_robot_model)/urdf/sensors/imu.xacro" />
+	<xacro:include filename="$(find followme_robot_model)/urdf/sensors/sonar.xacro" />
 	<!-- <xacro:include filename="$(find followme_robot_model)/urdf/sensors/camera_depth.xacro" /> -->
 	<!-- Wheel parameters -->
@@ -31,18 +33,43 @@
 			<origin xyz="0 0 0.3" rpy="0 0 0" />
 		</xacro:lidar>
-		<xacro:include filename="$(find followme_robot_model)/urdf/sensors/camera.xacro" />
+		<xacro:imu_sensor parent="robot_body_link">
+			<origin xyz="0 0 0" rpy="0 0 0"/>
+		</xacro:imu_sensor>
+		<!-- <xacro:include filename="$(find followme_robot_model)/urdf/sensors/camera.xacro" /> -->
+		<xacro:sonar parent="robot_body_link" side="front" direction="mid">
+			<origin xyz="0.3 0 0.2" rpy="0 0 0"/>
+		</xacro:sonar>
+		<xacro:sonar parent="robot_body_link" side="front" direction="left">
+			<origin xyz="0.3 0.1 0.2" rpy="0 0 ${PI/8}"/>
+		</xacro:sonar>
+		<xacro:sonar parent="robot_body_link" side="front" direction="right">
+			<origin xyz="0.3 -0.1 0.2" rpy="0 0 -${PI/8}"/>
+		</xacro:sonar>
+		<xacro:sonar parent="robot_body_link" side="back" direction="mid">
+			<origin xyz="-0.3 0 0.2" rpy="0 0 ${PI}"/>
+		</xacro:sonar>
+		<xacro:sonar parent="robot_body_link" side="back" direction="left">
+			<origin xyz="-0.3 0.1 0.2" rpy="0 0 ${PI+PI/8}"/>
+		</xacro:sonar>
+		<xacro:sonar parent="robot_body_link" side="back" direction="right">
+			<origin xyz="-0.3 -0.1 0.2" rpy="0 0 ${PI+PI/8}"/>
+		</xacro:sonar>
 	</xacro:macro>
 	<xacro:robot />
 	<xacro:omni_steering />
-	<xacro:ros_joint_pose_trajectory />
+	<xacro:ros_joint_pose_trajectory fameName="robot_body_link" />
 	<gazebo>
 		<plugin name="gazebo_ros_joint_state_publisher"
 			filename="libgazebo_ros_joint_state_publisher.so">
-			<update_rate>${update_rate}</update_rate>
-			<joint_name>robot_footprint_joint</joint_name>
+			<!-- <joint_name>robot_footprint_joint</joint_name> -->
 			<joint_name>front_right_wheel_joint</joint_name>
 			<joint_name>front_left_wheel_joint</joint_name>
 			<joint_name>back_left_wheel_joint</joint_name>
 			<joint_name>back_right_wheel_joint</joint_name>
+			<always_on>true</always_on>
+			<update_rate>50.0</update_rate>
+			<!-- <ros>	 -->
+			<!-- <remapping>~/out:=scan</remapping> -->
+			<!-- </ros> -->
 		</plugin>
 	</gazebo>

File: src/followme_robot_model/urdf/followme_robot_model.gazebo.xacro (robot description, xacro)
@@ -1,4 +1,4 @@
 <?xml version="1.0"?>
-<robot xmlns:xacro="http://www.ros.org/wiki/xacro">
+<robot xmlns:xacro="http://playerstage.sourceforge.net/gazebo/xmlschema/#interface">
 	<xacro:macro name="omni_steering" params="">
 		<gazebo>
@@ -13,5 +13,5 @@
 		</gazebo>
 	</xacro:macro>
-	<xacro:macro name="loop" param="joints:=^ *element">
+	<xacro:macro name="loop" params="joints:=^ *element">
 		<xacro:if value="${joints}">
 			<xacro:property name="joint" value="${joints.pop(0)}"/>
@@ -22,6 +22,5 @@
 	<xacro:macro name="ros_joints_state_publisher" params="joints update_rate:=20">
 		<gazebo>
-			<plugin name="gazebo_ros_joint_state_publisher"
-				filename="libgazebo_ros_joint_state_publisher.so">
+			<plugin name="gazebo_ros_joint_state_publisher" filename="libgazebo_ros_joint_state_publisher.so">
 				<update_rate>${update_rate}</update_rate>
 				<xacro:loop joints="${joints}" />
@@ -31,6 +30,5 @@
 	<xacro:macro name="ros_joint_state_publisher" params="joint update_rate:=20">
 		<gazebo>
-			<plugin name="gazebo_ros_joint_state_publisher"
-				filename="libgazebo_ros_joint_state_publisher.so">
+			<plugin name="gazebo_ros_joint_state_publisher" filename="libgazebo_ros_joint_state_publisher.so">
 				<update_rate>${update_rate}</update_rate>
 				<joint_name>${joint}</joint_name>
@@ -38,9 +36,9 @@
 		</gazebo>
 	</xacro:macro>
-	<xacro:macro name="ros_joint_pose_trajectory">
+	<xacro:macro name="ros_joint_pose_trajectory" params="fameName">
 		<gazebo>
-			<plugin name="gazebo_ros_joint_pose_trajectory"
-				filename="libgazebo_ros_joint_pose_trajectory.so">
-				<update_rate>2</update_rate>
+			<plugin name="gazebo_ros_joint_pose_trajectory" filename="libgazebo_ros_joint_pose_trajectory.so">
+				<frame_name>${fameName}</frame_name>
+				<update_rate>50</update_rate>
 			</plugin>
 		</gazebo>

File: src/followme_robot_model/urdf/material.xacro (robot description, xacro)
@@ -1,4 +1,4 @@
 <?xml version="1.0"?>
-<robot xmlns:xacro="http://www.ros.org/wiki/xacro">
+<robot xmlns:xacro="http://playerstage.sourceforge.net/gazebo/xmlschema/#interface">
     <material name="white">
         <color rgba="1 1 1 1" />

File: src/followme_robot_model/urdf/sensors/camera.xacro (robot description, xacro)
@@ -1,4 +1,4 @@
 <?xml version="1.0"?>
-<robot xmlns:xacro="http://www.ros.org/wiki/xacro" >
+<robot xmlns:xacro="http://playerstage.sourceforge.net/gazebo/xmlschema/#interface" >
     <joint name="camera_joint" type="fixed">
         <parent link="robot_body_link"/>
@@ -48,5 +48,5 @@
                 <frame_name>camera_link_optical</frame_name>
                 <ros>
-                    <argument>~/out:=range</argument>
+                    <remapping>~/out:=range</remapping>
                 </ros>
                 <output_type>sensor_msgs/Range</output_type>

File: src/followme_robot_model/urdf/sensors/lidar.xacro (robot description, xacro)
@@ -1,6 +1,7 @@
 <?xml version="1.0"?>
-<robot xmlns:xacro="http://www.ros.org/wiki/xacro">
+<robot xmlns:xacro="http://playerstage.sourceforge.net/gazebo/xmlschema/#interface">
     <xacro:include filename="$(find followme_robot_model)/urdf/physics/inertial.urdf.xacro" />
     <xacro:include filename="$(find followme_robot_model)/urdf/material.xacro" />
+    <xacro:include filename="$(find followme_robot_model)/urdf/sensors/gazebo/lidar.gazebo" />
     <xacro:macro name="lidar" params="parent *origin laser_name range:=12">
         <joint name="${laser_name}_laser_joint" type="fixed">
@@ -10,49 +11,23 @@
         </joint>
         <link name="${laser_name}_laser_frame">
-            <visual>
-                <geometry>
-                    <cylinder radius="0.05" length="0.04" />
-                </geometry>
-                <material name="red" />
-            </visual>
             <collision>
                 <geometry>
-                    <cylinder radius="0.05" length="0.04" />
+                    <box size="0.1 0.1 0.1"/>
                 </geometry>
             </collision>
+            <visual>
+                <origin xyz="0 0 0" rpy="0 0 0"/>
+                <geometry>
+                    <box size="0.1 0.1 0.1"/>
+                    <!-- <mesh filename="package://followme_robot_model/meshes/hokuyo.dae"/> -->
+                </geometry>
+            </visual>
             <inertial>
-                <origin xyz="0 0 0" rpy="0 0 0" />
-                <mass value="0.1" />
-                <xacro:cylinder_inertia m="0.1" h="0.04" r="0.05" />
+                <mass value="1e-5" />
+                <origin xyz="0 0 0" rpy="0 0 0"/>
+                <xacro:solid_cuboid_inertia w="0.1" h="0.1" d="0.1" m="1e-5" />
             </inertial>
         </link>
-        <gazebo reference="${laser_name}_laser_frame">
-            <material>Gazebo/Red</material>
-            <sensor name="laser" type="ray">
-                <pose> 0 0 0 0 0 0 </pose>
-                <visualize>true</visualize>
-                <update_rate>10</update_rate>
-                <ray>
-                    <scan>
-                        <horizontal>
-                            <samples>360</samples>
-                            <min_angle>-3.14</min_angle>
-                            <max_angle>3.14</max_angle>
-                        </horizontal>
-                    </scan>
-                    <range>
-                        <min>0.3</min>
-                        <max>${range}</max>
-                    </range>
-                </ray>
-                <plugin name="laser_controller" filename="libgazebo_ros_ray_sensor.so">
-                    <ros>
-                        <argument>~/out:=scan</argument>
-                    </ros>
-                    <output_type>sensor_msgs/LaserScan</output_type>
-                    <frame_name>${laser_name}_laser_frame</frame_name>
-                </plugin>
-            </sensor>
-        </gazebo>
+        <xacro:lidar_gazebo reference="${laser_name}_laser_frame" />
     </xacro:macro>
 </robot>

File: src/followme_robot_model/urdf/wheel/omni_wheel.urdf.xacro (robot description, xacro)
@@ -1,15 +1,15 @@
 <?xml version="1.0"?>
-<robot name="wheel" xmlns:xacro="http://www.ros.org/wiki/xacro">
+<robot name="wheel"
+  xmlns:xacro="http://playerstage.sourceforge.net/gazebo/xmlschema/#interface">
   <xacro:include filename="$(find followme_robot_model)/urdf/physics/inertial.urdf.xacro"/>
   <xacro:property name="PI" value="3.1415926535897931" />
   <!-- Wheels -->
   <xacro:property name="wheel_height" value="0.087" />
-  <xacro:property name="wheel_mass" value="6.5" /> <!-- in kg-->
+  <xacro:property name="wheel_mass" value="6.5" />
+  <!-- in kg-->
   <xacro:macro name="cylinder_inertia" params="m r h">
-    <inertia  ixx="${m*(3*r*r+h*h)/12}" ixy = "0" ixz = "0"
-              iyy="${m*r*r/2}" iyz = "0"
-              izz="${m*(3*r*r+h*h)/12}" />
+    <inertia ixx="${m*(3*r*r+h*h)/12}" ixy = "0" ixz = "0" iyy="${m*r*r/2}" iyz = "0" izz="${m*(3*r*r+h*h)/12}" />
   </xacro:macro>
-  <xacro:macro name="omni_wheel" params="prefix parent *origin reflect wheel_radius update_rate:=20">
+  <xacro:macro name="omni_wheel" params="prefix parent *origin reflect wheel_radius">
     <joint name="${prefix}_wheel_joint" type="continuous">
       <parent link="${parent}"/>
@@ -28,7 +28,7 @@
       </visual>
       <collision>
-				<origin xyz="0 0 0" rpy="${PI/2} 0 0" />
+        <origin xyz="0 0 0" rpy="${PI/2} 0 0" />
         <geometry>
-					<cylinder length="${wheel_height}" radius="${wheel_radius}" />
+          <cylinder length="${wheel_height}" radius="${wheel_radius}" />
         </geometry>
       </collision>
@@ -36,5 +36,5 @@
         <mass value="${wheel_mass}" />
         <origin xyz="0 0 0" />
-        <xacro:cylinder_inertia  m="${wheel_mass}" r="${wheel_radius}" h="${wheel_height}" />
+        <xacro:cylinder_inertia m="${wheel_mass}" r="${wheel_radius}" h="${wheel_height}" />
       </inertial>
     </link>
@@ -42,18 +42,18 @@
     <transmission name="${prefix}_wheel_joint_trans">
       <type>transmission_interface/SimpleTransmission</type>
-      <joint name="${prefix}_wheel_joint" >
+      <joint name="${prefix}_wheel_joint">
         <hardwareInterface>hardware_interface/VelocityJointInterface</hardwareInterface>
       </joint>
       <actuator name="${prefix}_wheel_joint_motor">
-         <mechanicalReduction>1</mechanicalReduction>
+        <mechanicalReduction>1</mechanicalReduction>
       </actuator>
     </transmission>
     <gazebo reference="${prefix}_wheel_link">
-		<mu1 value="1.0"/>
-		<mu2 value="1.0"/>
-		<kp value="10000000.0" />
-		<kd value="1.0" />
-		<fdir1 value="1 0 0"/>
-        <turnGravityOff>false</turnGravityOff>
+      <mu1 value="1.0"/>
+      <mu2 value="1.0"/>
+      <kp value="10000000.0" />
+      <kd value="1.0" />
+      <fdir1 value="1 0 0"/>
+      <turnGravityOff>false</turnGravityOff>
     </gazebo>
   </xacro:macro>
