Commit message: refactored and fixed some stuff

File: src/followme_robot_model/urdf/physics/inertial.urdf.xacro (robot description, xacro)
@@ -10,5 +10,5 @@
   </xacro:macro>
   <!-- TODO Hollow sphere of radius r and mass m-->
-  <xacro:macro name="solid_sphere_inertia" params="m r">
+  <xacro:macro name="hollow_sphere_inertia" params="m r">
     <inertia  ixx="${(2*r*r*m)/3}" ixy = "0" ixz = "0"
               iyy="${(2*r*r*m)/3}" iyz = "0"
