Commit message: start redesign robot model

File: src/follow_me_robot/urdf/core/material.xacro (robot description, xacro)
@@ -16,3 +16,9 @@
         <color rgba="1 0 0 1"/>
     </material>
+    <material name="green">
+        <color rgba="0 1 0 1"/>
+    </material>
+    <material name="orange">
+        <color rgba="${255/255} ${108/255} ${10/255} 1.0"/>
+    </material>
 </robot>

File: src/follow_me_robot/urdf/core/omni_wheel.urdf.xacro (robot description, xacro)
@@ -1,15 +1,15 @@
 <?xml version="1.0"?>
 <robot name="wheel" xmlns:xacro="http://www.ros.org/wiki/xacro">
-  <xacro:include filename="$(find follow_me_robot)/urdf/core/inertial.urdf.xacro"/>
-  <xacro:property name="PI" value="3.1415926535897931" />
+  <xacro:include filename="./inertial.urdf.xacro"/>
   <!-- Wheels -->
-  <xacro:property name="wheel_height" value="0.087" />
   <xacro:property name="wheel_mass" value="6.5" /> <!-- in kg-->
-  <xacro:macro name="cylinder_inertia" params="m r h">
-    <inertia  ixx="${m*(3*r*r+h*h)/12}" ixy = "0" ixz = "0"
-              iyy="${m*r*r/2}" iyz = "0"
-              izz="${m*(3*r*r+h*h)/12}" />
+  <xacro:macro name="omni_wheel_geometry" params="wheel_height wheel_radius reflect">
+    <origin xyz="0 0 0" rpy="0 0 0" />
+    <geometry>
+      <mesh filename="meshes/omni_wheel_${reflect}.dae" />
+      <cylinder length="${wheel_height}" radius="${wheel_radius}" />
+    </geometry>
   </xacro:macro>
-  <xacro:macro name="omni_wheel" params="prefix parent *origin reflect wheel_radius update_rate:=20">
+  <xacro:macro name="omni_wheel" params="prefix parent *origin reflect wheel_height wheel_radius update_rate:=20">
     <joint name="${prefix}_wheel_joint" type="continuous">
       <parent link="${parent}"/>
@@ -22,11 +22,14 @@
     <link name="${prefix}_wheel_link">
       <visual>
-        <origin xyz="0 0 0" rpy="0 0 0" />
+      <xacro:omni_wheel_geometry reflect="${reflect}"
+        wheel_height="${wheel_height}"
+        wheel_radius="${wheel_radius}" />
+        <!-- <origin xyz="0 0 0" rpy="0 0 0" />
         <geometry>
           <mesh filename="file://$(find follow_me_robot)/meshes/omni_wheel_${reflect}.dae" />
-        </geometry>
+        </geometry> -->
       </visual>
       <collision>
-				<origin xyz="0 0 0" rpy="${PI/2} 0 0" />
+				<origin xyz="0 0 0" rpy="${pi/2} 0 0" />
         <geometry>
 					<cylinder length="${wheel_height}" radius="${wheel_radius}" />
@@ -36,5 +39,5 @@
         <mass value="${wheel_mass}" />
         <origin xyz="0 0 0" />
-        <xacro:cylinder_inertia  m="${wheel_mass}" r="${wheel_radius}" h="${wheel_height}" />
+        <xacro:solid_cylinder_inertia  m="${wheel_mass}" r="${wheel_radius}" h="${wheel_height}" />
       </inertial>
     </link>

File: src/follow_me_robot/urdf/core/robot_body.urdf.xacro (robot description, xacro)
@@ -1,18 +1,12 @@
 <?xml version="1.0"?>
 <robot name="robot" xmlns:xacro="http://www.ros.org/wiki/xacro">
-  <xacro:macro name="robot_body" params="wheel_radius">
-      <xacro:include filename="$(find follow_me_robot)/urdf/core/follow_me_robot.gazebo.xacro" />
+  <xacro:macro name="robot_body_geometry" >
+    </xacro:macro>
+  <xacro:macro name="robot_body" params="wheel_radius body_length body_with body_heigth">
+      <xacro:include filename="core/follow_me_robot.gazebo.xacro" />
 	  <!-- Robot mechanical and motor parameters -->
 	<!-- BASE FOOTPRINT -->
-		<link name="robot_footprint">
-		  <visual>
-			  <origin xyz="0 0 0" rpy="0 0 0" />
-			  <geometry>
-				 <box size="0.001 0.001 0.001" />
-			  </geometry>
-		  </visual>
-		</link>
 		<joint name="robot_footprint_joint" type="fixed">
-		  <parent link="robot_footprint"/>
+		  <parent link="base_footprint"/>
 		  <child link="robot_body_link" />
       <origin xyz="0 0 ${wheel_radius}" rpy="0 0 0" />
@@ -27,7 +21,7 @@
     <visual>
        <origin xyz="0 0 0" rpy="0 0 0" />
-       <geometry>
-	       <mesh filename="file://$(find follow_me_robot)/meshes/robot_body.dae"/>
-       </geometry>
+        <geometry>
+            <box size="${body_length} ${body_with} ${body_heigth}"/>
+        </geometry>
        <material name="darkgrey">
          <color rgba="0.1 0.1 0.1 1"/>
@@ -36,7 +30,5 @@
     <collision>
        <origin xyz="0 0 0" rpy="0 0 0 " />
-       <geometry>
-         <mesh filename="file://$(find follow_me_robot)/meshes/robot_body.dae"/>
-       </geometry>
+       <xacro:robot_body_geometry />
     </collision>
   </link>

File: src/follow_me_robot/urdf/robot.urdf.xacro (robot description, xacro)
@@ -1,35 +1,49 @@
 <?xml version="1.0"?>
 <robot name="robot" xmlns:xacro="http://www.ros.org/wiki/xacro">
+	<!-- Robot Size -->
+	<xacro:property name="body_length" value="0.80" />
+	<xacro:property name="body_with" value="0.5"/>
+	<xacro:property name="body_heigth" value="0.20"/>
+	<xacro:property name="wheel_height" value="0.087" />
 	<!-- Import summit XL wheels -->
-	<xacro:include filename="$(find follow_me_robot)/urdf/core/omni_wheel.urdf.xacro" />
-	<xacro:include filename="$(find follow_me_robot)/urdf/core/robot_body.urdf.xacro" />
-	<xacro:include filename="$(find follow_me_robot)/urdf/core/follow_me_robot.gazebo.xacro" />
-	<xacro:include filename="$(find follow_me_robot)/urdf/sensors/lidar.xacro" />
+	<xacro:include filename="core/omni_wheel.urdf.xacro" />
+	<xacro:include filename="core/robot_body.urdf.xacro" />
+	<xacro:include filename="core/follow_me_robot.gazebo.xacro" />
+	<xacro:include filename="sensors/lidar.xacro" />
+	<xacro:include filename="world_base.urdf.xacro" />
+	<xacro:include filename="sensors/camera.xacro" />
+	<xacro:include filename="sensors/gps.xacro" />
 	<!-- <xacro:include filename="$(find follow_me_robot)/urdf/sensors/camera_depth.xacro" /> -->
+	<!-- Additional params -->
 	<!-- Wheel parameters -->
-	<xacro:property name="wheel_offset_x" value="0.2225" />    <!-- x,y,z in translation from base_link to the center of the wheel -->
-	<xacro:property name="wheel_offset_y" value="0.2045" />
+	<xacro:property name="wheel_offset_x" value="0.25" />    <!-- x,y,z in translation from base_link to the center of the wheel -->
+	<xacro:property name="wheel_offset_y" value="${(body_with/2)+(wheel_height/2)+0.005}" />
 	<xacro:property name="wheel_offset_z" value="0.0" />
 	<xacro:property name="wheel_radius" value="0.127" />
-	<!-- Additional params -->
 	<xacro:property name="update_rate" value="20" />
 	<xacro:macro name="robot">
-		<xacro:robot_body wheel_radius="${wheel_radius}" />
-		<xacro:omni_wheel prefix="front_right" parent="robot_body_link" reflect="2" wheel_radius="${wheel_radius}" >
-			<origin xyz="${wheel_offset_x} -${wheel_offset_y} ${wheel_offset_z}" rpy="0 0 0" />
+		<xacro:robot_body wheel_radius="${wheel_radius}"
+		body_length="${body_length}"
+		body_with="${body_with}"
+		body_heigth="${body_heigth}"
+		/>
+		<xacro:omni_wheel prefix="front_right" parent="robot_body_link" reflect="2" wheel_height="${wheel_height}" wheel_radius="${wheel_radius}" >
+			<origin xyz="${wheel_offset_x} -${wheel_offset_y} ${wheel_offset_z}" rpy="${pi/2} 0 0" />
 		</xacro:omni_wheel>
-		<xacro:omni_wheel prefix="front_left" parent="robot_body_link" reflect="1" wheel_radius="${wheel_radius}">
-			<origin xyz="${wheel_offset_x} ${wheel_offset_y} ${wheel_offset_z}" rpy="0 0 0" />
+		<xacro:omni_wheel prefix="front_left" parent="robot_body_link" reflect="1" wheel_height="${wheel_height}" wheel_radius="${wheel_radius}">
+			<origin xyz="${wheel_offset_x} ${wheel_offset_y} ${wheel_offset_z}" rpy="${pi/2} 0 0" />
 		</xacro:omni_wheel>
-		<xacro:omni_wheel prefix="back_left" parent="robot_body_link" reflect="1" wheel_radius="${wheel_radius}">
-			<origin xyz="-${wheel_offset_x} ${wheel_offset_y} ${wheel_offset_z}" rpy="0 0 0" />
+		<xacro:omni_wheel prefix="back_left" parent="robot_body_link" reflect="1" wheel_height="${wheel_height}" wheel_radius="${wheel_radius}">
+			<origin xyz="-${wheel_offset_x} ${wheel_offset_y} ${wheel_offset_z}" rpy="${pi/2} 0 0" />
 		</xacro:omni_wheel>
-		<xacro:omni_wheel prefix="back_right" parent="robot_body_link" reflect="2" wheel_radius="${wheel_radius}">
-			<origin xyz="-${wheel_offset_x} -${wheel_offset_y} ${wheel_offset_z}" rpy="0 0 0" />
+		<xacro:omni_wheel prefix="back_right" parent="robot_body_link" reflect="2" wheel_height="${wheel_height}" wheel_radius="${wheel_radius}">
+			<origin xyz="-${wheel_offset_x} -${wheel_offset_y} ${wheel_offset_z}" rpy="${pi/2} 0 0" />
 		</xacro:omni_wheel>
 		<xacro:lidar parent="robot_body_link" laser_name="1">
-			<origin xyz="0 0 0.3" rpy="0 0 0" />
+			<origin xyz="0 0 ${body_heigth/2+0.03}" rpy="0 0 0" />
 		</xacro:lidar>
-		<xacro:include filename="$(find follow_me_robot)/urdf/sensors/camera.xacro" />
+		<xacro:camera camname="front" parent="robot_body_link">
+			<origin xyz="${body_length/2} 0 0.0"/>
+		</xacro:camera>
 	</xacro:macro>
 	<xacro:robot />

File: src/follow_me_robot/urdf/sensors/camera.xacro (robot description, xacro)
@@ -1,58 +1,31 @@
 <?xml version="1.0"?>
 <robot xmlns:xacro="http://www.ros.org/wiki/xacro" >
-    <joint name="camera_joint" type="fixed">
-        <parent link="robot_body_link"/>
-        <child link="camera_link"/>
-        <origin xyz="0 0 0.5" rpy="0 0 0"/>
+<xacro:macro name="camera" params="camname parent *origin">
+    <xacro:include filename="sensors/gazebo/cam.gazebo"/>
+    <joint name="${camname}_camera_joint" type="fixed">
+        <parent link="${parent}"/>
+        <child link="${camname}_camera_link"/>
+        <xacro:insert_block name="origin" />
     </joint>
-    <link name="camera_link">
+    <link name="${camname}_camera_link">
         <visual>
             <geometry>
                 <box size="0.010 0.03 0.03"/>
             </geometry>
-            <material name="black"/>
+            <material name="blue"/>
         </visual>
         <visual>
-            <origin xyz="0 0 -0.05"/>
+            <origin xyz="0.005 0 0" rpy="0 ${pi/2} 0"/>
             <geometry>
-                <cylinder radius="0.002" length="0.1"/>
+                <cylinder radius="0.01" length="0.01"/>
             </geometry>
-            <material name="black"/>
+            <material name="blue"/>
         </visual>
     </link>
-    <joint name="camera_optical_joint" type="fixed">
-        <parent link="camera_link"/>
-        <child link="camera_link_optical"/>
-        <origin xyz="0 0 0" rpy="${-pi/2} 0 ${-pi/2}"/>
-    </joint>
-    <link name="camera_link_optical"></link>
-    <gazebo reference="camera_link">
-        <material>Gazebo/Black</material>
-        <sensor name="camera" type="depth">
-            <pose> 0 0 0 0 0 0 </pose>
-            <visualize>true</visualize>
-            <update_rate>10</update_rate>
-            <camera>
-                <horizontal_fov>1.089</horizontal_fov>
-                <image>
-                    <format>R8G8B8</format>
-                    <width>640</width>
-                    <height>480</height>
-                </image>
-                <clip>
-                    <near>0.05</near>
-                    <far>8.0</far>
-                </clip>
-            </camera>
-            <plugin name="camera_controller" filename="libgazebo_ros_camera.so">
-                <frame_name>camera_link_optical</frame_name>
-                <ros>
-                    <argument>--ros-args --remap ~/out:=range</argument>
-                </ros>
-                <output_type>sensor_msgs/Range</output_type>
-                <min_depth>0.01</min_depth>
-                <max_depth>100.0</max_depth>
-            </plugin>
-        </sensor>
-    </gazebo>
+    <xacro:camgazebo
+        cam_name="${camname}"
+        parent="${camname}_camera_link" >
+        <origin xyz="0.01 0 0" rpy="${-pi/2} 0 ${-pi/2}"/>
+    </xacro:camgazebo>
+</xacro:macro>
 </robot>

File: src/follow_me_robot/urdf/sensors/camera_depth.xacro (robot description, xacro)
@@ -1,5 +1,5 @@
 <?xml version="1.0"?>
 <robot xmlns:xacro="http://www.ros.org/wiki/xacro">
-    <xacro:include filename="$(find follow_me_robot)/urdf/core/inertial.urdf.xacro" />
+    <xacro:include filename="core/inertial.urdf.xacro" />
     <xacro:macro name="camera" params="parent *origin camera_name">
         <joint name="${camera_name}_camera_joint" type="fixed">

File: src/follow_me_robot/urdf/sensors/imu.xacro (robot description, xacro)
@@ -2,5 +2,5 @@
 <robot name="follow_me_robot"
   xmlns:xacro="http://playerstage.sourceforge.net/gazebo/xmlschema/#interface">
-  <xacro:include filename="$(find follow_me_robot)/urdf/physics/inertial.urdf.xacro" />
+  <xacro:include filename="physics/inertial.urdf.xacro" />
   <xacro:macro name="imu_sensor" params="parent *origin">
     <joint name="imu_joint" type="fixed">
@@ -27,5 +27,5 @@
       </inertial>
     </link>
-    <xacro:include filename="$(find follow_me_robot)/urdf/sensors/gazebo/imu.gazebo"/>
+    <xacro:include filename="sensors/gazebo/imu.gazebo"/>
   </xacro:macro>
 </robot>

File: src/follow_me_robot/urdf/sensors/lidar.xacro (robot description, xacro)
@@ -1,6 +1,6 @@
 <?xml version="1.0"?>
 <robot xmlns:xacro="http://www.ros.org/wiki/xacro">
-    <xacro:include filename="$(find follow_me_robot)/urdf/core/inertial.urdf.xacro" />
-    <xacro:include filename="$(find follow_me_robot)/urdf/core/material.xacro" />
+    <xacro:include filename="../core/inertial.urdf.xacro" />
+    <xacro:include filename="../core/material.xacro" />
     <xacro:macro name="lidar" params="parent *origin laser_name">
         <joint name="${laser_name}_laser_joint" type="fixed">
@@ -24,5 +24,5 @@
                 <origin xyz="0 0 0" rpy="0 0 0" />
                 <mass value="0.1" />
-                <xacro:cylinder_inertia m="0.1" h="0.04" r="0.05" />
+                <xacro:solid_cylinder_inertia m="0.1" h="0.04" r="0.05" />
             </inertial>
         </link>

Commit message: fix robot build

File: src/follow_me_robot/urdf/core/material.xacro (robot description, xacro)
@@ -19,6 +19,6 @@
         <color rgba="0 1 0 1"/>
     </material>
-    <material name="orange">
+    <!-- <material name="orange">
         <color rgba="${255/255} ${108/255} ${10/255} 1.0"/>
-    </material>
+    </material> -->
 </robot>

File: src/follow_me_robot/urdf/robot.urdf.xacro (robot description, xacro)
@@ -1,4 +1,5 @@
 <?xml version="1.0"?>
-<robot name="robot" xmlns:xacro="http://www.ros.org/wiki/xacro">
+<robot name="robot"
+	xmlns:xacro="http://www.ros.org/wiki/xacro">
 	<!-- Robot Size -->
 	<xacro:property name="body_length" value="0.80" />
@@ -14,43 +15,46 @@
 	<xacro:include filename="sensors/camera.xacro" />
 	<xacro:include filename="sensors/gps.xacro" />
+	<xacro:include filename="sensors/imu.xacro" />
 	<!-- <xacro:include filename="$(find follow_me_robot)/urdf/sensors/camera_depth.xacro" /> -->
 	<!-- Additional params -->
 	<!-- Wheel parameters -->
-	<xacro:property name="wheel_offset_x" value="0.25" />    <!-- x,y,z in translation from base_link to the center of the wheel -->
+	<xacro:property name="wheel_offset_x" value="0.25" />
+	<!-- x,y,z in translation from base_link to the center of the wheel -->
 	<xacro:property name="wheel_offset_y" value="${(body_with/2)+(wheel_height/2)+0.005}" />
 	<xacro:property name="wheel_offset_z" value="0.0" />
 	<xacro:property name="wheel_radius" value="0.127" />
 	<xacro:property name="update_rate" value="20" />
-	<xacro:macro name="robot">
-		<xacro:robot_body wheel_radius="${wheel_radius}"
-		body_length="${body_length}"
-		body_with="${body_with}"
-		body_heigth="${body_heigth}"
-		/>
-		<xacro:omni_wheel prefix="front_right" parent="robot_body_link" reflect="2" wheel_height="${wheel_height}" wheel_radius="${wheel_radius}" >
-			<origin xyz="${wheel_offset_x} -${wheel_offset_y} ${wheel_offset_z}" rpy="${pi/2} 0 0" />
-		</xacro:omni_wheel>
-		<xacro:omni_wheel prefix="front_left" parent="robot_body_link" reflect="1" wheel_height="${wheel_height}" wheel_radius="${wheel_radius}">
-			<origin xyz="${wheel_offset_x} ${wheel_offset_y} ${wheel_offset_z}" rpy="${pi/2} 0 0" />
-		</xacro:omni_wheel>
-		<xacro:omni_wheel prefix="back_left" parent="robot_body_link" reflect="1" wheel_height="${wheel_height}" wheel_radius="${wheel_radius}">
-			<origin xyz="-${wheel_offset_x} ${wheel_offset_y} ${wheel_offset_z}" rpy="${pi/2} 0 0" />
-		</xacro:omni_wheel>
-		<xacro:omni_wheel prefix="back_right" parent="robot_body_link" reflect="2" wheel_height="${wheel_height}" wheel_radius="${wheel_radius}">
-			<origin xyz="-${wheel_offset_x} -${wheel_offset_y} ${wheel_offset_z}" rpy="${pi/2} 0 0" />
-		</xacro:omni_wheel>
-		<xacro:lidar parent="robot_body_link" laser_name="1">
-			<origin xyz="0 0 ${body_heigth/2+0.03}" rpy="0 0 0" />
-		</xacro:lidar>
-		<xacro:camera camname="front" parent="robot_body_link">
-			<origin xyz="${body_length/2} 0 0.0"/>
-		</xacro:camera>
-	</xacro:macro>
-	<xacro:robot />
+	<!-- <xacro:macro name="robot"> -->
+	<xacro:robot_body wheel_radius="${wheel_radius}" body_length="${body_length}" body_with="${body_with}" body_heigth="${body_heigth}" />
+	<xacro:omni_wheel prefix="front_right" parent="robot_body_link" reflect="2" wheel_height="${wheel_height}" wheel_radius="${wheel_radius}">
+		<origin xyz="${wheel_offset_x} -${wheel_offset_y} ${wheel_offset_z}" rpy="${pi/2} 0 0" />
+	</xacro:omni_wheel>
+	<xacro:omni_wheel prefix="front_left" parent="robot_body_link" reflect="1" wheel_height="${wheel_height}" wheel_radius="${wheel_radius}">
+		<origin xyz="${wheel_offset_x} ${wheel_offset_y} ${wheel_offset_z}" rpy="${pi/2} 0 0" />
+	</xacro:omni_wheel>
+	<xacro:omni_wheel prefix="back_left" parent="robot_body_link" reflect="1" wheel_height="${wheel_height}" wheel_radius="${wheel_radius}">
+		<origin xyz="-${wheel_offset_x} ${wheel_offset_y} ${wheel_offset_z}" rpy="${pi/2} 0 0" />
+	</xacro:omni_wheel>
+	<xacro:omni_wheel prefix="back_right" parent="robot_body_link" reflect="2" wheel_height="${wheel_height}" wheel_radius="${wheel_radius}">
+		<origin xyz="-${wheel_offset_x} -${wheel_offset_y} ${wheel_offset_z}" rpy="${pi/2} 0 0" />
+	</xacro:omni_wheel>
+	<xacro:lidar parent="robot_body_link" laser_name="1">
+		<origin xyz="0 0 ${body_heigth/2+0.03}" rpy="0 0 0" />
+	</xacro:lidar>
+	<xacro:camera camname="front" parent="robot_body_link">
+		<origin xyz="${body_length/2} 0 0.0"/>
+	</xacro:camera>
+	<xacro:gps parent="robot_body_link">
+		<origin xyz="0 0 0.0"/>
+	</xacro:gps>
+	<xacro:imu parent="robot_body_link">
+		<origin xyz="0 0 0.0"/>
+	</xacro:imu>
+	<!-- </xacro:macro>
+	<xacro:robot /> -->
 	<xacro:omni_steering />
 	<xacro:ros_joint_pose_trajectory />
 	<gazebo>
-		<plugin name="gazebo_ros_joint_state_publisher"
-			filename="libgazebo_ros_joint_state_publisher.so">
+		<plugin name="gazebo_ros_joint_state_publisher" filename="libgazebo_ros_joint_state_publisher.so">
 			<update_rate>${update_rate}</update_rate>
 			<joint_name>robot_footprint_joint</joint_name>

File: src/follow_me_robot/urdf/sensors/gps.xacro (robot description, xacro)
@@ -4,4 +4,5 @@
   <xacro:macro name="gps" params="parent *origin gps_name=main">
     <xacro:include filename="core/material.xacro"/>
+    <xacro:include filename="sensors/gazebo/gps.gazebo"/>
     <joint name="${gps_name}_gps_joint" type="fixed">
       <parent link="${parent}"/>
@@ -28,7 +29,9 @@
       </inertial>
     </link>
-    <gazebo reference="${gps_name}_gps_link">
+    <xacro:gazebogps gps_name="${gps_name}">
+    </xacro:gazebogps>
+    <!-- <gazebo >
       <material>Gazebo/Orange</material>
-    </gazebo>
+    </gazebo> -->
   </xacro:macro>
 </robot>

File: src/follow_me_robot/urdf/sensors/imu.xacro (robot description, xacro)
@@ -1,13 +1,14 @@
 <?xml version="1.0"?>
-<robot name="follow_me_robot"
+<robot name="sensor"
   xmlns:xacro="http://playerstage.sourceforge.net/gazebo/xmlschema/#interface">
-  <xacro:include filename="physics/inertial.urdf.xacro" />
-  <xacro:macro name="imu_sensor" params="parent *origin">
-    <joint name="imu_joint" type="fixed">
+  <xacro:macro name="imu" params="parent *origin imu_name=main">
+    <xacro:include filename="core/inertial.urdf.xacro" />
+    <xacro:include filename="sensors/gazebo/imu.gazebo"/>
+    <joint name="${imu_name}_imu_joint" type="fixed">
       <parent link="${parent}" />
-      <child link="imu_link" />
+      <child link="${imu_name}_imu_link" />
       <xacro:insert_block name="origin" />
     </joint>
-    <link name="imu_link">
+    <link name="${imu_name}_imu_link">
       <visual>
         <geometry>
@@ -27,5 +28,5 @@
       </inertial>
     </link>
-    <xacro:include filename="sensors/gazebo/imu.gazebo"/>
+    <xacro:gazeboimu imu_name="${imu_name}"/>
   </xacro:macro>
 </robot>

File: src/follow_me_robot/urdf/sensors/reciver.xacro (robot description, xacro)
@@ -1,5 +1,5 @@
 <?xml version="1.0"?>
 <robot xmlns:xacro="http://playerstage.sourceforge.net/gazebo/xmlschema/#interface">
-    <xacro:include filename="$(find follow_me_robot)/urdf/physics/inertial.urdf.xacro" />
+    <xacro:include filename="$(find follow_me_robot)/urdf/core/inertial.urdf.xacro" />
     <xacro:include filename="$(find follow_me_robot)/urdf/material.xacro" />
     <xacro:macro name="reciver" params="parent *origin">

File: src/follow_me_robot/urdf/sensors/sonar.xacro (robot description, xacro)
@@ -13,5 +13,5 @@
       <visual>
         <geometry>
-          <mesh filename="package://follow_me_robot/meshes/max_sonar_ez4.dae"/>
+          <mesh filename="package://follow_me_robot/urdf/meshes/max_sonar_ez4.dae"/>
         </geometry>
       </visual>
