Commit message: refactored project structure

File: src/follow_me_robot/urdf/core/follow_me_robot.gazebo.xacro (robot description, xacro)
@@ -13,5 +13,5 @@
 		</gazebo>
 	</xacro:macro>
-	<xacro:macro name="loop" param="joints:=^ *element">
+	<xacro:macro name="loop" params="joints:=^ *element">
 		<xacro:if value="${joints}">
 			<xacro:property name="joint" value="${joints.pop(0)}"/>

File: src/follow_me_robot/urdf/core/omni_wheel.urdf.xacro (robot description, xacro)
@@ -1,5 +1,5 @@
 <?xml version="1.0"?>
 <robot name="wheel" xmlns:xacro="http://www.ros.org/wiki/xacro">
-  <xacro:include filename="$(find followme_robot_model)/urdf/physics/inertial.urdf.xacro"/>
+  <xacro:include filename="$(find follow_me_robot)/urdf/core/inertial.urdf.xacro"/>
   <xacro:property name="PI" value="3.1415926535897931" />
   <!-- Wheels -->
@@ -24,5 +24,5 @@
         <origin xyz="0 0 0" rpy="0 0 0" />
         <geometry>
-          <mesh filename="file://$(find followme_robot_model)/meshes/wheels/omni_wheel_${reflect}.dae" />
+          <mesh filename="file://$(find follow_me_robot)/meshes/omni_wheel_${reflect}.dae" />
         </geometry>
       </visual>

File: src/follow_me_robot/urdf/core/robot_body.urdf.xacro (robot description, xacro)
@@ -2,7 +2,6 @@
 <robot name="robot" xmlns:xacro="http://www.ros.org/wiki/xacro">
   <xacro:macro name="robot_body" params="wheel_radius">
-      <xacro:include filename="$(find followme_robot_model)/urdf/followme_robot_model.gazebo.xacro" />
+      <xacro:include filename="$(find follow_me_robot)/urdf/core/follow_me_robot.gazebo.xacro" />
 	  <!-- Robot mechanical and motor parameters -->
-	  <xacro:property name="PI" value="3.1415926535897931"/>
 	<!-- BASE FOOTPRINT -->
 		<link name="robot_footprint">
@@ -29,5 +28,5 @@
        <origin xyz="0 0 0" rpy="0 0 0" />
        <geometry>
-	       <mesh filename="file://$(find followme_robot_model)/meshes/body/robot_body.dae"/>
+	       <mesh filename="file://$(find follow_me_robot)/meshes/robot_body.dae"/>
        </geometry>
        <material name="darkgrey">
@@ -38,5 +37,5 @@
        <origin xyz="0 0 0" rpy="0 0 0 " />
        <geometry>
-         <mesh filename="file://$(find followme_robot_model)/meshes/body/robot_body.dae"/>
+         <mesh filename="file://$(find follow_me_robot)/meshes/robot_body.dae"/>
        </geometry>
     </collision>

File: src/follow_me_robot/urdf/robot.urdf.xacro (robot description, xacro)
@@ -2,9 +2,9 @@
 <robot name="robot" xmlns:xacro="http://www.ros.org/wiki/xacro">
 	<!-- Import summit XL wheels -->
-	<xacro:include filename="$(find followme_robot_model)/urdf/wheel/omni_wheel.urdf.xacro" />
-	<xacro:include filename="$(find followme_robot_model)/urdf/body/robot_body.urdf.xacro" />
-	<xacro:include filename="$(find followme_robot_model)/urdf/followme_robot_model.gazebo.xacro" />
-	<xacro:include filename="$(find followme_robot_model)/urdf/sensors/lidar.xacro" />
-	<!-- <xacro:include filename="$(find followme_robot_model)/urdf/sensors/camera_depth.xacro" /> -->
+	<xacro:include filename="$(find follow_me_robot)/urdf/core/omni_wheel.urdf.xacro" />
+	<xacro:include filename="$(find follow_me_robot)/urdf/core/robot_body.urdf.xacro" />
+	<xacro:include filename="$(find follow_me_robot)/urdf/core/follow_me_robot.gazebo.xacro" />
+	<xacro:include filename="$(find follow_me_robot)/urdf/sensors/lidar.xacro" />
+	<!-- <xacro:include filename="$(find follow_me_robot)/urdf/sensors/camera_depth.xacro" /> -->
 	<!-- Wheel parameters -->
 	<xacro:property name="wheel_offset_x" value="0.2225" />    <!-- x,y,z in translation from base_link to the center of the wheel -->
@@ -31,5 +31,5 @@
 			<origin xyz="0 0 0.3" rpy="0 0 0" />
 		</xacro:lidar>
-		<xacro:include filename="$(find followme_robot_model)/urdf/sensors/camera.xacro" />
+		<xacro:include filename="$(find follow_me_robot)/urdf/sensors/camera.xacro" />
 	</xacro:macro>
 	<xacro:robot />

File: src/follow_me_robot/urdf/sensors/camera_depth.xacro (robot description, xacro)
@@ -1,6 +1,6 @@
 <?xml version="1.0"?>
 <robot xmlns:xacro="http://www.ros.org/wiki/xacro">
-    <xacro:include filename="$(find followme_robot_model)/urdf/physics/inertial.urdf.xacro" />
-    <xacro:macro name="camera" params="parent *origin camera_name range:=8">
+    <xacro:include filename="$(find follow_me_robot)/urdf/core/inertial.urdf.xacro" />
+    <xacro:macro name="camera" params="parent *origin camera_name">
         <joint name="${camera_name}_camera_joint" type="fixed">
             <parent link="${parent}" />

File: src/follow_me_robot/urdf/sensors/lidar.xacro (robot description, xacro)
@@ -1,6 +1,6 @@
 <?xml version="1.0"?>
 <robot xmlns:xacro="http://www.ros.org/wiki/xacro">
-    <xacro:include filename="$(find followme_robot_model)/urdf/physics/inertial.urdf.xacro" />
-    <xacro:include filename="$(find followme_robot_model)/urdf/material.xacro" />
+    <xacro:include filename="$(find follow_me_robot)/urdf/core/inertial.urdf.xacro" />
+    <xacro:include filename="$(find follow_me_robot)/urdf/core/material.xacro" />
     <xacro:macro name="lidar" params="parent *origin laser_name range:=12">
         <joint name="${laser_name}_laser_joint" type="fixed">
