Commit message: update robot model

File: src/follow_me_robot/urdf/core/follow_me_robot.gazebo.xacro (robot description, xacro)
@@ -4,10 +4,10 @@
 		<gazebo>
 			<plugin name="psuedo_mecanum" filename="libgazebo_ros_planar_move.so">
-				<commandTopic>cmd_vel</commandTopic>
-				<odometryTopic>odom</odometryTopic>
-				<odometryFrame>odom</odometryFrame>
-				<odometryRate>50.0</odometryRate>
-				<robotBaseFrame>base_footprint</robotBaseFrame>
-				<publishTF>true</publishTF>
+				<command_topic>cmd_vel</command_topic>
+				<odometry_topic>odom</odometry_topic>
+				<odometry_frame>odom</odometry_frame>
+				<odometry_rate>50.0</odometry_rate>
+				<robot_base_frame>base_footprint</robot_base_frame>
+				<publish_tf>true</publish_tf>
 			</plugin>
 		</gazebo>
@@ -22,5 +22,5 @@
 	<xacro:macro name="ros_joints_state_publisher" params="joints update_rate:=20">
 		<gazebo>
-			<plugin name="gazebo_ros_joint_state_publisher"
+			<plugin name="gazebo_ros_joints_state_publisher"
 				filename="libgazebo_ros_joint_state_publisher.so">
 				<update_rate>${update_rate}</update_rate>
@@ -38,9 +38,9 @@
 		</gazebo>
 	</xacro:macro>
-	<xacro:macro name="ros_joint_pose_trajectory">
+	<xacro:macro name="ros_joint_pose_trajectory" params="update_rate:=30">
 		<gazebo>
 			<plugin name="gazebo_ros_joint_pose_trajectory"
 				filename="libgazebo_ros_joint_pose_trajectory.so">
-				<update_rate>2</update_rate>
+				<update_rate>${update_rate}</update_rate>
 			</plugin>
 		</gazebo>

File: src/follow_me_robot/urdf/core/material.xacro (robot description, xacro)
@@ -1,4 +1,5 @@
 <?xml version="1.0"?>
 <robot xmlns:xacro="http://playerstage.sourceforge.net/gazebo/xmlschema/#interface">
+<xacro:macro name="materials">
     <material name="white">
         <color rgba="1 1 1 1" />
@@ -19,6 +20,7 @@
         <color rgba="0 1 0 1"/>
     </material>
-    <!-- <material name="orange">
-        <color rgba="${255/255} ${108/255} ${10/255} 1.0"/>
-    </material> -->
+    <material name="darkgrey">
+         <color rgba="0.1 0.1 0.1 1"/>
+    </material>
+</xacro:macro>
 </robot>

File: src/follow_me_robot/urdf/core/omni_wheel.urdf.xacro (robot description, xacro)
@@ -1,15 +1,15 @@
 <?xml version="1.0"?>
 <robot name="wheel" xmlns:xacro="http://www.ros.org/wiki/xacro">
-  <xacro:include filename="./inertial.urdf.xacro"/>
+  <xacro:include filename="inertial.urdf.xacro"/>
   <!-- Wheels -->
-  <xacro:property name="wheel_mass" value="6.5" /> <!-- in kg-->
   <xacro:macro name="omni_wheel_geometry" params="wheel_height wheel_radius reflect">
     <origin xyz="0 0 0" rpy="0 0 0" />
     <geometry>
-      <mesh filename="meshes/omni_wheel_${reflect}.dae" />
+      <mesh filename="file://$(find follow_me_robot)/urdf/meshes/omni_wheel_${reflect}.dae" />
       <cylinder length="${wheel_height}" radius="${wheel_radius}" />
     </geometry>
   </xacro:macro>
   <xacro:macro name="omni_wheel" params="prefix parent *origin reflect wheel_height wheel_radius update_rate:=20">
+    <xacro:property name="wheel_mass" value="6.5" /> <!-- in kg-->
     <joint name="${prefix}_wheel_joint" type="continuous">
       <parent link="${parent}"/>
@@ -22,21 +22,18 @@
     <link name="${prefix}_wheel_link">
       <visual>
-      <xacro:omni_wheel_geometry reflect="${reflect}"
-        wheel_height="${wheel_height}"
-        wheel_radius="${wheel_radius}" />
-        <!-- <origin xyz="0 0 0" rpy="0 0 0" />
-        <geometry>
-          <mesh filename="file://$(find follow_me_robot)/meshes/omni_wheel_${reflect}.dae" />
-        </geometry> -->
+        <xacro:omni_wheel_geometry reflect="${reflect}"
+          wheel_height="${wheel_height}"
+          wheel_radius="${wheel_radius}" />
       </visual>
       <collision>
 				<origin xyz="0 0 0" rpy="${pi/2} 0 0" />
-        <geometry>
-					<cylinder length="${wheel_height}" radius="${wheel_radius}" />
-        </geometry>
+        <!-- <origin xyz="0 0 0" rpy="0 0 0" /> -->
+      <geometry>
+        <!-- <mesh filename="file://$(find follow_me_robot)/urdf/meshes/omni_wheel_${reflect}.dae" /> -->
+        <cylinder length="${wheel_height}" radius="${wheel_radius}" />
+      </geometry>
       </collision>
       <inertial>
         <mass value="${wheel_mass}" />
-        <origin xyz="0 0 0" />
         <xacro:solid_cylinder_inertia  m="${wheel_mass}" r="${wheel_radius}" h="${wheel_height}" />
       </inertial>

File: src/follow_me_robot/urdf/core/robot_body.urdf.xacro (robot description, xacro)
@@ -1,15 +1,9 @@
 <?xml version="1.0"?>
 <robot name="robot" xmlns:xacro="http://www.ros.org/wiki/xacro">
-  <xacro:macro name="robot_body_geometry" >
-    </xacro:macro>
+  <xacro:include filename="inertial.urdf.xacro"/>
+  <xacro:include filename="material.xacro"/>
+  <xacro:include filename="follow_me_robot.gazebo.xacro" />
   <xacro:macro name="robot_body" params="wheel_radius body_length body_with body_heigth">
-      <xacro:include filename="core/follow_me_robot.gazebo.xacro" />
 	  <!-- Robot mechanical and motor parameters -->
-	<!-- BASE FOOTPRINT -->
-		<joint name="robot_footprint_joint" type="fixed">
-		  <parent link="base_footprint"/>
-		  <child link="robot_body_link" />
-      <origin xyz="0 0 ${wheel_radius}" rpy="0 0 0" />
-		</joint>
   <!-- BASE_LINK -->
   <link name="robot_body_link">
@@ -17,5 +11,5 @@
       <mass value="125.0" />
       <origin xyz="0 0 0" />
-      <inertia  ixx="1.391" ixy="0.004"  ixz="0.0"  iyy="6.853"  iyz="0.0"  izz="6.125" />
+      <xacro:solid_cuboid_inertia m="125.0" h="${body_heigth}" d="${body_length}" w="${body_with}" />
     </inertial>
     <visual>
@@ -24,11 +18,10 @@
             <box size="${body_length} ${body_with} ${body_heigth}"/>
         </geometry>
-       <material name="darkgrey">
-         <color rgba="0.1 0.1 0.1 1"/>
-       </material>
     </visual>
     <collision>
        <origin xyz="0 0 0" rpy="0 0 0 " />
-       <xacro:robot_body_geometry />
+       <geometry>
+            <box size="${body_length} ${body_with} ${body_heigth}"/>
+        </geometry>
     </collision>
   </link>

File: src/follow_me_robot/urdf/robot.urdf.xacro (robot description, xacro)
@@ -7,56 +7,50 @@
 	<xacro:property name="body_heigth" value="0.20"/>
 	<xacro:property name="wheel_height" value="0.087" />
-	<!-- Import summit XL wheels -->
+	<!-- Wheel parameters -->
+	<xacro:property name="wheel_offset_x" value="0.25" />
+	<!-- x,y,z in translation from base_link to the center of the wheel -->
+	<xacro:property name="wheel_offset_y" value="${(body_with/2)+(wheel_height/2)+0.01}" />
+	<xacro:property name="wheel_offset_z" value="0.0" />
+	<xacro:property name="wheel_radius" value="0.127" />
+	<xacro:property name="update_rate" value="20" />
+	<!-- BASE FOOTPRINT -->
+	<link name="base_footprint">
+		<visual>
+			<origin xyz="0 0 0" rpy="0 0 0" />
+			<geometry>
+				<box size="0.001 0.001 0.001" />
+			</geometry>
+		</visual>
+	</link>
+	<joint name="robot_footprint_joint" type="fixed">
+		<parent link="base_footprint"/>
+		<child link="robot_body_link" />
+		<origin xyz="0 0 ${wheel_radius}" rpy="0 0 0" />
+	</joint>
+	<xacro:include filename="core/material.xacro" />
+	<xacro:materials />
 	<xacro:include filename="core/omni_wheel.urdf.xacro" />
 	<xacro:include filename="core/robot_body.urdf.xacro" />
 	<xacro:include filename="core/follow_me_robot.gazebo.xacro" />
-	<xacro:include filename="sensors/lidar.xacro" />
-	<xacro:include filename="world_base.urdf.xacro" />
-	<xacro:include filename="sensors/camera.xacro" />
-	<xacro:include filename="sensors/gps.xacro" />
-	<xacro:include filename="sensors/imu.xacro" />
-	<!-- <xacro:include filename="$(find follow_me_robot)/urdf/sensors/camera_depth.xacro" /> -->
 	<!-- Additional params -->
-	<!-- Wheel parameters -->
-	<xacro:property name="wheel_offset_x" value="0.25" />
-	<!-- x,y,z in translation from base_link to the center of the wheel -->
-	<xacro:property name="wheel_offset_y" value="${(body_with/2)+(wheel_height/2)+0.005}" />
-	<xacro:property name="wheel_offset_z" value="0.0" />
-	<xacro:property name="wheel_radius" value="0.127" />
-	<xacro:property name="update_rate" value="20" />
-	<!-- <xacro:macro name="robot"> -->
 	<xacro:robot_body wheel_radius="${wheel_radius}" body_length="${body_length}" body_with="${body_with}" body_heigth="${body_heigth}" />
 	<xacro:omni_wheel prefix="front_right" parent="robot_body_link" reflect="2" wheel_height="${wheel_height}" wheel_radius="${wheel_radius}">
-		<origin xyz="${wheel_offset_x} -${wheel_offset_y} ${wheel_offset_z}" rpy="${pi/2} 0 0" />
+		<origin xyz="${wheel_offset_x} -${wheel_offset_y} ${wheel_offset_z}" rpy="0 0 0" />
 	</xacro:omni_wheel>
-	<xacro:omni_wheel prefix="front_left" parent="robot_body_link" reflect="1" wheel_height="${wheel_height}" wheel_radius="${wheel_radius}">
-		<origin xyz="${wheel_offset_x} ${wheel_offset_y} ${wheel_offset_z}" rpy="${pi/2} 0 0" />
+	<xacro:omni_wheel prefix="front_left" parent="robot_body_link" reflect="2" wheel_height="${wheel_height}" wheel_radius="${wheel_radius}">
+		<origin xyz="${wheel_offset_x} ${wheel_offset_y} ${wheel_offset_z}" rpy="0 0 0" />
 	</xacro:omni_wheel>
 	<xacro:omni_wheel prefix="back_left" parent="robot_body_link" reflect="1" wheel_height="${wheel_height}" wheel_radius="${wheel_radius}">
-		<origin xyz="-${wheel_offset_x} ${wheel_offset_y} ${wheel_offset_z}" rpy="${pi/2} 0 0" />
+		<origin xyz="-${wheel_offset_x} ${wheel_offset_y} ${wheel_offset_z}" rpy="0 0 0" />
 	</xacro:omni_wheel>
-	<xacro:omni_wheel prefix="back_right" parent="robot_body_link" reflect="2" wheel_height="${wheel_height}" wheel_radius="${wheel_radius}">
-		<origin xyz="-${wheel_offset_x} -${wheel_offset_y} ${wheel_offset_z}" rpy="${pi/2} 0 0" />
+	<xacro:omni_wheel prefix="back_right" parent="robot_body_link" reflect="1" wheel_height="${wheel_height}" wheel_radius="${wheel_radius}">
+		<origin xyz="-${wheel_offset_x} -${wheel_offset_y} ${wheel_offset_z}" rpy="0 0 0" />
 	</xacro:omni_wheel>
-	<xacro:lidar parent="robot_body_link" laser_name="1">
-		<origin xyz="0 0 ${body_heigth/2+0.03}" rpy="0 0 0" />
-	</xacro:lidar>
-	<xacro:camera camname="front" parent="robot_body_link">
-		<origin xyz="${body_length/2} 0 0.0"/>
-	</xacro:camera>
-	<xacro:gps parent="robot_body_link">
-		<origin xyz="0 0 0.0"/>
-	</xacro:gps>
-	<xacro:imu parent="robot_body_link">
-		<origin xyz="0 0 0.0"/>
-	</xacro:imu>
-	<!-- </xacro:macro>
-	<xacro:robot /> -->
 	<xacro:omni_steering />
-	<xacro:ros_joint_pose_trajectory />
+	<!-- <xacro:ros_joint_pose_trajectory /> -->
 	<gazebo>
 		<plugin name="gazebo_ros_joint_state_publisher" filename="libgazebo_ros_joint_state_publisher.so">
 			<update_rate>${update_rate}</update_rate>
-			<joint_name>robot_footprint_joint</joint_name>
+			<!-- <joint_name>robot_footprint_joint</joint_name> -->
 			<joint_name>front_right_wheel_joint</joint_name>
 			<joint_name>front_left_wheel_joint</joint_name>
@@ -64,4 +58,24 @@
 			<joint_name>back_right_wheel_joint</joint_name>
 		</plugin>
+		<plugin name="gazebo_ros_joint_pose_trajectory"
+			filename="libgazebo_ros_joint_pose_trajectory.so">
+			<update_rate>${update_rate}</update_rate>
+		</plugin>
 	</gazebo>
+	<xacro:include filename="sensors/lidar.xacro" />
+	<xacro:lidar parent="robot_body_link">
+		<origin xyz="0 0 ${body_heigth/2+0.03}" rpy="0 0 0" />
+	</xacro:lidar>
+	<!-- <xacro:include filename="sensors/gps.xacro" />
+	<xacro:gps parent="robot_body_link">
+		<origin xyz="0 0 0.0"/>
+	</xacro:gps> -->
+	<xacro:include filename="sensors/imu.xacro" />
+	<xacro:imu parent="robot_body_link">
+		<origin xyz="0 0 0.0"/>
+	</xacro:imu>
+	<xacro:include filename="sensors/camera.xacro" />
+	<xacro:camera cam_name="front" parent="robot_body_link">
+		<origin xyz="${body_length/2} 0 0.0"/>
+	</xacro:camera>
 </robot>

File: src/follow_me_robot/urdf/sensors/camera.xacro (robot description, xacro)
@@ -1,12 +1,12 @@
 <?xml version="1.0"?>
 <robot xmlns:xacro="http://www.ros.org/wiki/xacro" >
-<xacro:macro name="camera" params="camname parent *origin">
-    <xacro:include filename="sensors/gazebo/cam.gazebo"/>
-    <joint name="${camname}_camera_joint" type="fixed">
+<xacro:include filename="gazebo/cam.gazebo"/>
+<xacro:macro name="camera" params="cam_name parent *origin">
+    <joint name="${cam_name}_camera_joint" type="fixed">
         <parent link="${parent}"/>
-        <child link="${camname}_camera_link"/>
+        <child link="${cam_name}_camera_link"/>
         <xacro:insert_block name="origin" />
     </joint>
-    <link name="${camname}_camera_link">
+    <link name="${cam_name}_camera_link">
         <visual>
             <geometry>
@@ -23,8 +23,6 @@
         </visual>
     </link>
-    <xacro:camgazebo
-        cam_name="${camname}"
-        parent="${camname}_camera_link" >
-        <origin xyz="0.01 0 0" rpy="${-pi/2} 0 ${-pi/2}"/>
+    <xacro:camgazebo cam_name="${cam_name}">
+        <origin xyz="0.01 0 0" rpy="${-pi/2} ${-pi/2} ${-pi/2}"/>
     </xacro:camgazebo>
 </xacro:macro>

File: src/follow_me_robot/urdf/sensors/camera_depth.xacro (robot description, xacro)
@@ -1,6 +1,6 @@
 <?xml version="1.0"?>
 <robot xmlns:xacro="http://www.ros.org/wiki/xacro">
-    <xacro:include filename="core/inertial.urdf.xacro" />
-    <xacro:macro name="camera" params="parent *origin camera_name">
+    <xacro:include filename="../../core/inertial.urdf.xacro" />
+    <xacro:macro name="deph_camera" params="parent *origin camera_name">
         <joint name="${camera_name}_camera_joint" type="fixed">
             <parent link="${parent}" />

File: src/follow_me_robot/urdf/sensors/gps.xacro (robot description, xacro)
@@ -2,36 +2,38 @@
 <robot name="sensor"
   xmlns:xacro="http://playerstage.sourceforge.net/gazebo/xmlschema/#interface">
-  <xacro:macro name="gps" params="parent *origin gps_name=main">
-    <xacro:include filename="core/material.xacro"/>
-    <xacro:include filename="sensors/gazebo/gps.gazebo"/>
+  <xacro:include filename="../core/material.xacro"/>
+  <xacro:include filename="../core/inertial.urdf.xacro" />
+  <xacro:include filename="gazebo/gps.gazebo"/>
+  <xacro:macro name="gps" params="parent *origin gps_name:=sensor_0">
+    <xacro:property name="w" value="0.1"/>
+    <xacro:property name="h" value="0.1"/>
+    <xacro:property name="d" value="0.1"/>
     <joint name="${gps_name}_gps_joint" type="fixed">
       <parent link="${parent}"/>
       <child link="${gps_name}_gps_link"/>
+      <xacro:insert_block name="origin" />
     </joint>
     <link name="${gps_name}_gps_link">
       <collision>
-        <origin xyz="0 0 0.1" rpy="0 0 0"/>
+        <origin xyz="0 0 0" rpy="0 0 0"/>
         <geometry>
-          <box size="0.2 0.2 0.2"/>
+          <box size="${w} ${d} ${h}"/>
         </geometry>
       </collision>
       <visual>
-        <origin xyz="0 0 0.1" rpy="0 0 0"/>
+        <origin xyz="0 0 0" rpy="0 0 0"/>
         <geometry>
-          <box size="0.2 0.2 0.2"/>
+          <box size="${w} ${d} ${h}"/>
         </geometry>
         <material name="orange"/>
       </visual>
       <inertial>
-        <origin xyz="0 0 1" rpy="0 0 0"/>
+        <origin xyz="0 0 0" rpy="0 0 0"/>
         <mass value="1"/>
-        <inertia ixx="1.0" ixy="0.0" ixz="0.0" iyy="1.0" iyz="0.0" izz="1.0"/>
+        <xacro:solid_cuboid_inertia m="1" h="${h}" d="${d}" w="${w}" />
       </inertial>
     </link>
     <xacro:gazebogps gps_name="${gps_name}">
     </xacro:gazebogps>
-    <!-- <gazebo >
-      <material>Gazebo/Orange</material>
-    </gazebo> -->
   </xacro:macro>
 </robot>

File: src/follow_me_robot/urdf/sensors/imu.xacro (robot description, xacro)
@@ -2,7 +2,7 @@
 <robot name="sensor"
   xmlns:xacro="http://playerstage.sourceforge.net/gazebo/xmlschema/#interface">
-  <xacro:macro name="imu" params="parent *origin imu_name=main">
-    <xacro:include filename="core/inertial.urdf.xacro" />
-    <xacro:include filename="sensors/gazebo/imu.gazebo"/>
+  <xacro:include filename="../core/inertial.urdf.xacro" />
+  <xacro:include filename="gazebo/imu.gazebo"/>
+  <xacro:macro name="imu" params="parent *origin imu_name:=sensor_0">
     <joint name="${imu_name}_imu_joint" type="fixed">
       <parent link="${parent}" />
@@ -24,5 +24,4 @@
         <mass value="1e-5" />
         <origin xyz="0 0 0" rpy="0 0 0"/>
-        <!-- <inertia ixx="1e-6" ixy="0" ixz="0" iyy="1e-6" iyz="0" izz="1e-6" /> -->
         <xacro:solid_cuboid_inertia w="0.05" h="0.05" d="0.5" m="1e-5" />
       </inertial>

File: src/follow_me_robot/urdf/sensors/lidar.xacro (robot description, xacro)
@@ -2,6 +2,7 @@
 <robot xmlns:xacro="http://www.ros.org/wiki/xacro">
     <xacro:include filename="../core/inertial.urdf.xacro" />
-    <xacro:include filename="../core/material.xacro" />
-    <xacro:macro name="lidar" params="parent *origin laser_name">
+    <xacro:include filename="../core/material.xacro"/>
+    <xacro:include filename="gazebo/lidar.gazebo" />
+    <xacro:macro name="lidar" params="parent *origin laser_name:=sensor_0 update:=30">
         <joint name="${laser_name}_laser_joint" type="fixed">
             <parent link="${parent}" />
@@ -27,32 +28,5 @@
             </inertial>
         </link>
-        <gazebo reference="${laser_name}_laser_frame">
-            <material>Gazebo/Red</material>
-            <sensor name="laser" type="ray">
-                <pose> 0 0 0 0 0 0 </pose>
-                <visualize>true</visualize>
-                <update_rate>10</update_rate>
-                <ray>
-                    <scan>
-                        <horizontal>
-                            <samples>360</samples>
-                            <min_angle>-3.14</min_angle>
-                            <max_angle>3.14</max_angle>
-                        </horizontal>
-                    </scan>
-                    <range>
-                        <min>0.3</min>
-                        <max>10.0</max>
-                    </range>
-                </ray>
-                <plugin name="laser_controller" filename="libgazebo_ros_ray_sensor.so">
-                    <ros>
-                        <argument>--ros-args --remap ~/out:=scan</argument>
-                    </ros>
-                    <output_type>sensor_msgs/LaserScan</output_type>
-                    <frame_name>${laser_name}_laser_frame</frame_name>
-                </plugin>
-            </sensor>
-        </gazebo>
+        <xacro:gazebolidar laser_name="${laser_name}" update="${update}"/>
     </xacro:macro>
 </robot>

File: src/follow_me_robot/urdf/sensors/reciver.xacro (robot description, xacro)
@@ -1,17 +1,14 @@
 <?xml version="1.0"?>
 <robot xmlns:xacro="http://playerstage.sourceforge.net/gazebo/xmlschema/#interface">
-    <xacro:include filename="$(find follow_me_robot)/urdf/core/inertial.urdf.xacro" />
-    <xacro:include filename="$(find follow_me_robot)/urdf/material.xacro" />
-    <xacro:macro name="reciver" params="parent *origin">
-        <xacro:property name="recreciver_h" value="0.1" />
-        <xacro:property name="recreciver_w" value="0.1" />
-        <xacro:property name="recreciver_d" value="0.1" />
-        <xacro:property name="recreciver_m" value="0.1" />
-        <joint name="recover_joint">
+    <!-- <xacro:include filename="$(find follow_me_robot)/urdf/material.xacro" /> -->
+    <xacro:include filename="../core/inertial.urdf.xacro" />
+    <xacro:include filename="../core/material.xacro"/>
+    <xacro:macro name="reciver" params="reciver_name parent *origin recreciver_h=0.1 recreciver_w=0.1 recreciver_d=0.1 recreciver_m=0.1">
+        <joint name="${reciver_name}_recover_joint">
             <parent link="${parent}" />
-            <child link="reciver_link" />
+            <child link="${reciver_name}_reciver_link" />
             <xacro:insert_block name="origin" />
         </joint>
-        <link name="reciver_link">
+        <link name="${reciver_name}_reciver_link">
             <inertial>
                 <origin xyz="0.0 0.0 0.0" rpy="0.0 0.0 0.0"/>
@@ -23,5 +20,5 @@
                     w="${recreciver_w}" />
             </inertial>
-            <visual name="">
+            <visual>
                 <origin xyz="0.0 0.0 0.0" rpy="0.0 0.0 0.0"/>
                 <geometry>
@@ -37,5 +34,5 @@
             </collision>
         </link>
-        <gazebo reference="reciver_link">
+        <gazebo reference="${reciver_name}_reciver_link">
             <material>Gazebo/Black</material>
             <sensor name="reciver" type=""></sensor>

File: src/follow_me_robot/urdf/sensors/sonar.xacro (robot description, xacro)
@@ -2,5 +2,5 @@
 <robot name="follow_me_robot"
   xmlns:xacro="http://playerstage.sourceforge.net/gazebo/xmlschema/#interface">
-    <xacro:include filename="$(find follow_me_robot)/urdf/sensors/gazebo/sonar.gazebo"/>
+  <xacro:include filename="gazebo/sonar.gazebo"/>
   <xacro:macro name="sonar" params="side direction parent *origin">
     <xacro:property name="sufix" value="${side}_${direction}" />

File: src/follow_me_robot/urdf/world_base.urdf.xacro (robot description, xacro)
@@ -1,10 +1,2 @@
-<robot xmlns:xacro="http://www.ros.org/wiki/xacro" name="world_base_link">
-    <link name="base_footprint">
-		<visual>
-			<origin xyz="0 0 0" rpy="0 0 0" />
-			<geometry>
-				<box size="0.001 0.001 0.001" />
-			</geometry>
-		</visual>
-	</link>
+<robot xmlns:xacro="http://www.ros.org/wiki/xacro" name="robot">
 </robot>
