Commit message: refacrot robot model

File: src/follow_me_robot/urdf/core/follow_me_robot.gazebo.xacro (robot description, xacro)
@@ -4,43 +4,17 @@
 		<gazebo>
 			<plugin name="psuedo_mecanum" filename="libgazebo_ros_planar_move.so">
-				<command_topic>cmd_vel</command_topic>
-				<odometry_topic>odom</odometry_topic>
+			<ros>
+			<namespace>/</namespace>
+			</ros>
+				<update_rate>100</update_rate>
+				<publish_rate>50</publish_rate>
+				<!-- output -->
+				<publish_odom>true</publish_odom>
+				<publish_odom_tf>true</publish_odom_tf>
 				<odometry_frame>odom</odometry_frame>
-				<odometry_rate>50.0</odometry_rate>
 				<robot_base_frame>base_footprint</robot_base_frame>
-				<publish_tf>true</publish_tf>
-			</plugin>
-		</gazebo>
-	</xacro:macro>
-	<xacro:macro name="loop" params="joints:=^ *element">
-		<xacro:if value="${joints}">
-			<xacro:property name="joint" value="${joints.pop(0)}"/>
-			<joint_name>$(joint)</joint_name>
-			<xacro:loop />
-		</xacro:if>
-	</xacro:macro>
-	<xacro:macro name="ros_joints_state_publisher" params="joints update_rate:=20">
-		<gazebo>
-			<plugin name="gazebo_ros_joints_state_publisher"
-				filename="libgazebo_ros_joint_state_publisher.so">
-				<update_rate>${update_rate}</update_rate>
-				<xacro:loop joints="${joints}" />
-			</plugin>
-		</gazebo>
-	</xacro:macro>
-	<xacro:macro name="ros_joint_state_publisher" params="joint update_rate:=20">
-		<gazebo>
-			<plugin name="gazebo_ros_joint_state_publisher"
-				filename="libgazebo_ros_joint_state_publisher.so">
-				<update_rate>${update_rate}</update_rate>
-				<joint_name>${joint}</joint_name>
-			</plugin>
-		</gazebo>
-	</xacro:macro>
-	<xacro:macro name="ros_joint_pose_trajectory" params="update_rate:=30">
-		<gazebo>
-			<plugin name="gazebo_ros_joint_pose_trajectory"
-				filename="libgazebo_ros_joint_pose_trajectory.so">
-				<update_rate>${update_rate}</update_rate>
+				<covariance_x>0.0001</covariance_x>
+				<covariance_y>0.0001</covariance_y>
+				<covariance_yaw>0.01</covariance_yaw>
 			</plugin>
 		</gazebo>

File: src/follow_me_robot/urdf/core/omni_wheel.urdf.xacro (robot description, xacro)
@@ -1,40 +1,53 @@
 <?xml version="1.0"?>
-<robot name="wheel" xmlns:xacro="http://www.ros.org/wiki/xacro">
+<robot namee="wheel"  xmlns:xacro="http://www.ros.org/wiki/xacro">
   <xacro:include filename="inertial.urdf.xacro"/>
   <!-- Wheels -->
-  <xacro:macro name="omni_wheel_geometry" params="wheel_height wheel_radius reflect">
-    <origin xyz="0 0 0" rpy="0 0 0" />
-    <geometry>
-      <mesh filename="file://$(find follow_me_robot)/urdf/meshes/omni_wheel_${reflect}.dae" />
-      <cylinder length="${wheel_height}" radius="${wheel_radius}" />
-    </geometry>
-  </xacro:macro>
-  <xacro:macro name="omni_wheel" params="prefix parent *origin reflect wheel_height wheel_radius update_rate:=20">
-    <xacro:property name="wheel_mass" value="6.5" /> <!-- in kg-->
+  <xacro:macro name="omni_wheel" params="parent x y z reflect side position wheel_height wheel_radius update_rate:=20">
+    <xacro:property name="wheel_mass" value="6.5" />
+    <xacro:property name="prefix" value="${position}_${side}" />
+    <xacro:if value="${side == 'left'}">
+      <xacro:property name="origin_factor" value="1"/>
+    </xacro:if>
+    <xacro:if value="${side == 'right'}">
+      <xacro:property name="origin_factor" value="-1"/>
+    </xacro:if>
+    <joint name="${prefix}_wheel_motor_joint" type="fixed">
+      <parent link="${parent}"/>
+      <child link="${prefix}_wheel_motor_link"/>
+      <origin xyz="${x} ${y-0.04*origin_factor} ${z}" rpy="0 0 0"/>
+    </joint>
+    <link name="${prefix}_wheel_motor_link">
+      <visual>
+        <origin xyz="0 0 0" rpy="0 0 0" />
+        <geometry>
+          <box size="0.1 0.1 0.1"/>
+        </geometry>
+        <material name="darkgrey" />
+      </visual>
+    </link>
     <joint name="${prefix}_wheel_joint" type="continuous">
-      <parent link="${parent}"/>
+      <parent link="${prefix}_wheel_motor_link"/>
       <child link="${prefix}_wheel_link"/>
-      <xacro:insert_block name="origin" />
+      <origin xyz="0 ${(wheel_height/2 + 0.05) * origin_factor} 0" rpy="0 0 0" />
       <axis xyz="0 1 0" rpy="0 0 0" />
-      <limit effort="100" velocity="100"/>
-      <joint_properties damping="0.0" friction="0.0"/>
     </joint>
     <link name="${prefix}_wheel_link">
       <visual>
-        <xacro:omni_wheel_geometry reflect="${reflect}"
-          wheel_height="${wheel_height}"
-          wheel_radius="${wheel_radius}" />
+        <!-- <origin xyz="0 0 0" rpy="${pi/2} 0 0" /> -->
+        <origin xyz="0 0 0" rpy="0 0 0" />
+        <geometry>
+          <mesh filename="file://$(find follow_me_robot)/urdf/meshes/omni_wheel_${reflect}.dae" />
+          <!-- <cylinder length="${wheel_height}" radius="${wheel_radius}" /> -->
+        </geometry>
       </visual>
       <collision>
-				<origin xyz="0 0 0" rpy="${pi/2} 0 0" />
-        <!-- <origin xyz="0 0 0" rpy="0 0 0" /> -->
-      <geometry>
-        <!-- <mesh filename="file://$(find follow_me_robot)/urdf/meshes/omni_wheel_${reflect}.dae" /> -->
-        <cylinder length="${wheel_height}" radius="${wheel_radius}" />
-      </geometry>
+        <origin xyz="0 0 0" rpy="${pi/2} 0 0" />
+        <geometry>
+          <cylinder length="${wheel_height}" radius="${wheel_radius}" />
+        </geometry>
       </collision>
       <inertial>
         <mass value="${wheel_mass}" />
-        <xacro:solid_cylinder_inertia  m="${wheel_mass}" r="${wheel_radius}" h="${wheel_height}" />
+        <xacro:solid_cylinder_inertia m="${wheel_mass}" r="${wheel_radius}" h="${wheel_height}" />
       </inertial>
     </link>
@@ -42,19 +55,25 @@
     <transmission name="${prefix}_wheel_joint_trans">
       <type>transmission_interface/SimpleTransmission</type>
-      <joint name="${prefix}_wheel_joint" >
+      <joint name="${prefix}_wheel_joint">
         <hardwareInterface>hardware_interface/VelocityJointInterface</hardwareInterface>
       </joint>
-      <actuator name="${prefix}_wheel_joint_motor">
-         <mechanicalReduction>1</mechanicalReduction>
+      <actuator name="${prefix}_wheel_joint_actuator">
+        <mechanicalReduction>50</mechanicalReduction>
       </actuator>
     </transmission>
-    <gazebo reference="${prefix}_wheel_link">
-		<mu1 value="1.0"/>
-		<mu2 value="1.0"/>
-		<kp value="10000000.0" />
-		<kd value="1.0" />
-		<fdir1 value="1 0 0"/>
-        <turnGravityOff>false</turnGravityOff>
+    <gazebo reference="${prefix}_wheel_case">
+      <mu1 value="1.0"/>
+      <mu2 value="1.0"/>
+      <kp value="10000000.0" />
+      <kd value="1.0" />
+      <fdir1 value="1 0 0"/>
+      <turnGravityOff>false</turnGravityOff>
     </gazebo>
+    <!-- <gazebo>
+      <plugin name="gazebo_ros_joint_state_publisher_${prefix}" filename="libgazebo_ros_joint_state_publisher.so">
+      <update_rate>100</update_rate>
+      <joint_name>${prefix}_wheel_joint</joint_name>
+      </plugin>
+    </gazebo> -->
   </xacro:macro>
 </robot>

File: src/follow_me_robot/urdf/core/robot_body.urdf.xacro (robot description, xacro)
@@ -5,5 +5,5 @@
   <xacro:include filename="follow_me_robot.gazebo.xacro" />
   <xacro:macro name="robot_body" params="wheel_radius body_length body_with body_heigth">
-	  <!-- Robot mechanical and motor parameters -->
+  <!-- Robot mechanical and motor parameters -->
   <!-- BASE_LINK -->
   <link name="robot_body_link">
@@ -17,4 +17,5 @@
         <geometry>
             <box size="${body_length} ${body_with} ${body_heigth}"/>
+            <!-- <box size="0.01 ${body_with} 0.01"/> -->
         </geometry>
     </visual>

File: src/follow_me_robot/urdf/robot.urdf.xacro (robot description, xacro)
@@ -10,5 +10,5 @@
 	<xacro:property name="wheel_offset_x" value="0.25" />
 	<!-- x,y,z in translation from base_link to the center of the wheel -->
-	<xacro:property name="wheel_offset_y" value="${(body_with/2)+(wheel_height/2)+0.01}" />
+	<xacro:property name="wheel_offset_y" value="${(body_with/2)}" />
 	<xacro:property name="wheel_offset_z" value="0.0" />
 	<xacro:property name="wheel_radius" value="0.127" />
@@ -16,4 +16,5 @@
 	<!-- BASE FOOTPRINT -->
 	<link name="base_footprint">
+		<must_be_base_link>true</must_be_base_link>
 		<visual>
 			<origin xyz="0 0 0" rpy="0 0 0" />
@@ -35,40 +36,34 @@
 	<!-- Additional params -->
 	<xacro:robot_body wheel_radius="${wheel_radius}" body_length="${body_length}" body_with="${body_with}" body_heigth="${body_heigth}" />
-	<xacro:omni_wheel prefix="front_right" parent="robot_body_link" reflect="2" wheel_height="${wheel_height}" wheel_radius="${wheel_radius}">
-		<origin xyz="${wheel_offset_x} -${wheel_offset_y} ${wheel_offset_z}" rpy="0 0 0" />
-	</xacro:omni_wheel>
-	<xacro:omni_wheel prefix="front_left" parent="robot_body_link" reflect="2" wheel_height="${wheel_height}" wheel_radius="${wheel_radius}">
-		<origin xyz="${wheel_offset_x} ${wheel_offset_y} ${wheel_offset_z}" rpy="0 0 0" />
-	</xacro:omni_wheel>
-	<xacro:omni_wheel prefix="back_left" parent="robot_body_link" reflect="1" wheel_height="${wheel_height}" wheel_radius="${wheel_radius}">
-		<origin xyz="-${wheel_offset_x} ${wheel_offset_y} ${wheel_offset_z}" rpy="0 0 0" />
-	</xacro:omni_wheel>
-	<xacro:omni_wheel prefix="back_right" parent="robot_body_link" reflect="1" wheel_height="${wheel_height}" wheel_radius="${wheel_radius}">
-		<origin xyz="-${wheel_offset_x} -${wheel_offset_y} ${wheel_offset_z}" rpy="0 0 0" />
-	</xacro:omni_wheel>
+	<xacro:omni_wheel position="front" side="right" parent="robot_body_link" reflect="2" wheel_height="${wheel_height}" wheel_radius="${wheel_radius}" x="${wheel_offset_x}" y="-${wheel_offset_y}" z="${wheel_offset_z}" />
+	<xacro:omni_wheel position="front" side="left" parent="robot_body_link" reflect="2" wheel_height="${wheel_height}" wheel_radius="${wheel_radius}" x="${wheel_offset_x}" y="${wheel_offset_y}" z="${wheel_offset_z}"/>
+	<xacro:omni_wheel position="back" side="left" parent="robot_body_link" reflect="1" wheel_height="${wheel_height}" wheel_radius="${wheel_radius}" x="-${wheel_offset_x}" y="${wheel_offset_y}" z="${wheel_offset_z}" />
+	<xacro:omni_wheel position="back" side="right" parent="robot_body_link" reflect="1" wheel_height="${wheel_height}" wheel_radius="${wheel_radius}" x="-${wheel_offset_x}" y="-${wheel_offset_y}" z="${wheel_offset_z}" />
 	<xacro:omni_steering />
 	<!-- <xacro:ros_joint_pose_trajectory /> -->
 	<gazebo>
 		<plugin name="gazebo_ros_joint_state_publisher" filename="libgazebo_ros_joint_state_publisher.so">
-			<update_rate>${update_rate}</update_rate>
-			<!-- <joint_name>robot_footprint_joint</joint_name> -->
-			<joint_name>front_right_wheel_joint</joint_name>
-			<joint_name>front_left_wheel_joint</joint_name>
-			<joint_name>back_left_wheel_joint</joint_name>
-			<joint_name>back_right_wheel_joint</joint_name>
+		<ros>
+			<namespace>/</namespace>
+			<remapping>joint_states:=joint_states</remapping>
+		</ros>
+		<update_rate>2</update_rate>
+		<joint_name>front_right_wheel_joint</joint_name>
+		<joint_name>front_left_wheel_joint</joint_name>
+		<joint_name>back_left_wheel_joint</joint_name>
+		<joint_name>back_right_wheel_joint</joint_name>
 		</plugin>
-		<plugin name="gazebo_ros_joint_pose_trajectory"
-			filename="libgazebo_ros_joint_pose_trajectory.so">
-			<update_rate>${update_rate}</update_rate>
+		<plugin name="gazebo_ros_joint_pose_trajectory" filename="libgazebo_ros_joint_pose_trajectory.so">
+			<update_rate>2</update_rate>
 		</plugin>
 	</gazebo>
-	<xacro:include filename="sensors/lidar.xacro" />
+	<!-- <xacro:include filename="sensors/lidar.xacro" />
 	<xacro:lidar parent="robot_body_link">
 		<origin xyz="0 0 ${body_heigth/2+0.03}" rpy="0 0 0" />
 	</xacro:lidar>
-	<!-- <xacro:include filename="sensors/gps.xacro" />
+	<xacro:include filename="sensors/gps.xacro" />
 	<xacro:gps parent="robot_body_link">
 		<origin xyz="0 0 0.0"/>
-	</xacro:gps> -->
+	</xacro:gps>
 	<xacro:include filename="sensors/imu.xacro" />
 	<xacro:imu parent="robot_body_link">
@@ -78,4 +73,4 @@
 	<xacro:camera cam_name="front" parent="robot_body_link">
 		<origin xyz="${body_length/2} 0 0.0"/>
-	</xacro:camera>
+	</xacro:camera> -->
 </robot>

File: src/follow_me_robot/urdf/sensors/lidar.xacro (robot description, xacro)
@@ -2,5 +2,4 @@
 <robot xmlns:xacro="http://www.ros.org/wiki/xacro">
     <xacro:include filename="../core/inertial.urdf.xacro" />
-    <xacro:include filename="../core/material.xacro"/>
     <xacro:include filename="gazebo/lidar.gazebo" />
     <xacro:macro name="lidar" params="parent *origin laser_name:=sensor_0 update:=30">

Commit message: refactor code and test nodes

File: src/follow_me_robot/urdf/core/follow_me_robot.gazebo.xacro (robot description, xacro)
@@ -4,17 +4,9 @@
 		<gazebo>
 			<plugin name="psuedo_mecanum" filename="libgazebo_ros_planar_move.so">
-			<ros>
-			<namespace>/</namespace>
-			</ros>
-				<update_rate>100</update_rate>
-				<publish_rate>50</publish_rate>
-				<!-- output -->
-				<publish_odom>true</publish_odom>
-				<publish_odom_tf>true</publish_odom_tf>
-				<odometry_frame>odom</odometry_frame>
-				<robot_base_frame>base_footprint</robot_base_frame>
-				<covariance_x>0.0001</covariance_x>
-				<covariance_y>0.0001</covariance_y>
-				<covariance_yaw>0.01</covariance_yaw>
+				<commandTopic>cmd_vel</commandTopic>
+				<odometryTopic>odom</odometryTopic>
+				<odometryFrame>odom</odometryFrame>
+				<odometryRate>20.0</odometryRate>
+				<robotBaseFrame>base_footprint</robotBaseFrame>
 			</plugin>
 		</gazebo>

File: src/follow_me_robot/urdf/core/omni_wheel.urdf.xacro (robot description, xacro)
@@ -22,7 +22,8 @@
           <box size="${motor_d} ${motor_w} ${motor_h}" />
         </geometry>
+        <material name="darkgrey" />
       </visual>
       <collision>
-        <origin xyz="0 0 0" rpy="0 0 0" />
+        <origin xyz="0 ${motor_offset} 0" rpy="0 0 0" />
         <geometry>
           <box size="${motor_d} ${motor_w} ${motor_h}" />
@@ -46,16 +47,22 @@
       <child link="${prefix}_link"/>
       <xacro:insert_block name="origin" />
-      <axis xyz="0 1 0" />
-      <limit effort="100" velocity="0"/>
+      <axis xyz="0 0 1" />
+      <!-- <limit effort="100" velocity="0"/> -->
       <joint_properties damping="0.0" friction="1.0"/>
     </joint>
     <link name="${prefix}_link">
       <visual>
-        <!-- <origin xyz="0 0 0" rpy="0 0 0" /> -->
+        <origin xyz="0 0 0" rpy="0 0 0" />
+        <geometry>
+          <cylinder length="${wheel_height}" radius="${wheel_radius}" />
+        </geometry>
+        <material name="black" />
+      </visual>
+      <visual>
         <origin xyz="0 0 0" rpy="${pi/2} 0 0" />
         <geometry>
           <mesh filename="file://$(find follow_me_robot)/urdf/meshes/omni_wheel_${wheel_img}.dae" />
-          <!-- <cylinder length="${wheel_height}" radius="${wheel_radius}" /> -->
         </geometry>
+        <material name="black" />
       </visual>
       <collision>
@@ -91,4 +98,10 @@
       <turnGravityOff>false</turnGravityOff>
     </gazebo>
+    <!-- <gazebo>
+      <plugin name="${prefix}_joint_state_publisher" filename="libgazebo_ros_joint_state_publisher.so">
+        <update_rate>2</update_rate>
+        <joint_name>${prefix}_joint</joint_name>
+      </plugin>
+    </gazebo> -->
   </xacro:macro>
 </robot>

File: src/follow_me_robot/urdf/robot.urdf.xacro (robot description, xacro)
@@ -44,20 +44,16 @@
 	</xacro:wheel_motor>
 	<xacro:omni_steering />
-	<!-- <xacro:ros_joint_pose_trajectory /> -->
 	<gazebo>
-		<plugin name="gazebo_ros_joint_pose_trajectory" filename="libgazebo_ros_joint_pose_trajectory.so">
+		<!-- <plugin name="gazebo_ros_joint_pose_trajectory"
+    	filename="libgazebo_ros_joint_pose_trajectory.so">
 			<update_rate>2</update_rate>
-		</plugin>
-		<plugin name="gazebo_ros_joint_state_publisher" filename="libgazebo_ros_joint_state_publisher.so">
-		<!-- <ros>
-			<namespace>/</namespace>
-			<remapping>joint_states:=joint_states</remapping>
-		</ros> -->
-		<update_rate>2</update_rate>
+		</plugin> -->
+		<!-- <plugin name="gazebo_ros_joint_state_publisher" filename="libgazebo_ros_joint_state_publisher.so">
+		<update_rate>100</update_rate>
 		<joint_name>front_right_wheel_joint</joint_name>
 		<joint_name>front_left_wheel_joint</joint_name>
 		<joint_name>back_left_wheel_joint</joint_name>
 		<joint_name>back_right_wheel_joint</joint_name>
-		</plugin>
+		</plugin> -->
 	</gazebo>
 	<xacro:include filename="sensors/lidar.xacro" />
