Commit message: add motor joint to robot model

File: src/follow_me_robot/urdf/core/omni_wheel.urdf.xacro (robot description, xacro)
@@ -1,41 +1,65 @@
 <?xml version="1.0"?>
-<robot namee="wheel"  xmlns:xacro="http://www.ros.org/wiki/xacro">
+<robot name="wheel"
+  xmlns:xacro="http://www.ros.org/wiki/xacro">
   <xacro:include filename="inertial.urdf.xacro"/>
   <!-- Wheels -->
-  <xacro:macro name="omni_wheel" params="parent x y z reflect side position wheel_height wheel_radius update_rate:=20">
+  <xacro:macro name="omni_wheel_geometry" params="parent *origin wheel_img side position wheel_height wheel_radius update_rate:=20">
+    <xacro:solid_sphere name="${position}_${side}_wheel" mass="6.5" visual="omni_wheel_${wheel_img}.dae" xyz_axis="0 1 0">
+      <xacro:insert_block name="origin" />
+      <geometry></geometry>
+    </xacro:solid_sphere>
+  </xacro:macro>
+  <xacro:macro name="wheel_motor" params="parent *origin wheel_img reflect side position wheel_height wheel_radius update_rate:=20">
+    <xacro:property name="prefix" value="${position}_${side}_wheel" />
+    <xacro:property name="motor_mass" value="0.1" />
+    <xacro:property name="motor_h" value="0.1" />
+    <xacro:property name="motor_d" value="0.1" />
+    <xacro:property name="motor_w" value="0.1" />
+    <xacro:property name="motor_offset" value="${motor_w/1.08 * reflect * -1}"/>
+    <joint name="${prefix}_motor_joint" type="fixed">
+      <parent link="${parent}"/>
+      <child link="${prefix}_motor_link" />
+      <xacro:insert_block name="origin" />
+    </joint>
+    <link name="${prefix}_motor_link">
+      <visual>
+        <origin xyz="0 ${motor_offset} 0" rpy="0 0 0" />
+        <geometry>
+          <box size="${motor_d} ${motor_w} ${motor_h}" />
+        </geometry>
+      </visual>
+      <collision>
+        <origin xyz="0 0 0" rpy="0 0 0" />
+        <geometry>
+          <box size="${motor_d} ${motor_w} ${motor_h}" />
+        </geometry>
+      </collision>
+      <inertial>
+        <mass value="${motor_mass}" />
+        <xacro:solid_cuboid_inertia m="${motor_mass}" d="${motor_d}" w="${motor_w}" h="${motor_h}"/>
+      </inertial>
+    </link>
+    <xacro:omni_wheel parent="${prefix}_motor_link" wheel_img="${wheel_img}" side="${side}" position="${position}" wheel_height="${wheel_height}" wheel_radius="${wheel_radius}" update_rate="${update_rate}">
+      <origin xyz="0 ${motor_offset+(wheel_height+0.01)*reflect} 0" />
+    </xacro:omni_wheel>
+  </xacro:macro>
+  <xacro:macro name="omni_wheel" params="parent *origin wheel_img side position wheel_height wheel_radius update_rate:=20">
     <xacro:property name="wheel_mass" value="6.5" />
-    <xacro:property name="prefix" value="${position}_${side}" />
-    <xacro:if value="${side == 'left'}">
-      <xacro:property name="origin_factor" value="1"/>
-    </xacro:if>
-    <xacro:if value="${side == 'right'}">
-      <xacro:property name="origin_factor" value="-1"/>
-    </xacro:if>
-    <joint name="${prefix}_wheel_motor_joint" type="fixed">
+    <xacro:property name="prefix" value="${position}_${side}_wheel" />
+    <!-- in kg-->
+    <joint name="${prefix}_joint" type="continuous">
       <parent link="${parent}"/>
-      <child link="${prefix}_wheel_motor_link"/>
-      <origin xyz="${x} ${y-0.04*origin_factor} ${z}" rpy="0 0 0"/>
+      <child link="${prefix}_link"/>
+      <xacro:insert_block name="origin" />
+      <axis xyz="0 1 0" />
+      <limit effort="100" velocity="0"/>
+      <joint_properties damping="0.0" friction="1.0"/>
     </joint>
-    <link name="${prefix}_wheel_motor_link">
+    <link name="${prefix}_link">
       <visual>
         <origin xyz="0 0 0" rpy="0 0 0" />
+        <!-- <origin xyz="0 0 0" rpy="${pi/2} 0 0" /> -->
         <geometry>
-          <box size="0.1 0.1 0.1"/>
-        </geometry>
-        <material name="darkgrey" />
-      </visual>
-    </link>
-    <joint name="${prefix}_wheel_joint" type="continuous">
-      <parent link="${prefix}_wheel_motor_link"/>
-      <child link="${prefix}_wheel_link"/>
-      <origin xyz="0 ${(wheel_height/2 + 0.05) * origin_factor} 0" rpy="0 0 0" />
-      <axis xyz="0 1 0" rpy="0 0 0" />
-    </joint>
-    <link name="${prefix}_wheel_link">
-      <visual>
-        <!-- <origin xyz="0 0 0" rpy="${pi/2} 0 0" /> -->
-        <origin xyz="0 0 0" rpy="0 0 0" />
-        <geometry>
-          <mesh filename="file://$(find follow_me_robot)/urdf/meshes/omni_wheel_${reflect}.dae" />
+          <mesh filename="file://$(find follow_me_robot)/urdf/meshes/omni_wheel_${wheel_img}.dae" />
           <!-- <cylinder length="${wheel_height}" radius="${wheel_radius}" /> -->
         </geometry>
@@ -44,4 +68,5 @@
         <origin xyz="0 0 0" rpy="${pi/2} 0 0" />
         <geometry>
+          <!-- <mesh filename="file://$(find follow_me_robot)/urdf/meshes/omni_wheel_${reflect}.dae" /> -->
           <cylinder length="${wheel_height}" radius="${wheel_radius}" />
         </geometry>
@@ -53,14 +78,16 @@
     </link>
     <!-- Transmission is important to link the joints and the controller (see robot_control/config/robot_control.yaml)-->
-    <transmission name="${prefix}_wheel_joint_trans">
+    <transmission name="${prefix}_joint_trans" type="transmission_interface/SimpleTransmission">
       <type>transmission_interface/SimpleTransmission</type>
-      <joint name="${prefix}_wheel_joint">
-        <hardwareInterface>hardware_interface/VelocityJointInterface</hardwareInterface>
+      <joint name="${prefix}_joint">
+        <!-- <hardwareInterface>hardware_interface/VelocityJointInterface</hardwareInterface> -->
+        <hardwareInterface>EffortJointInterface</hardwareInterface>
       </joint>
-      <actuator name="${prefix}_wheel_joint_actuator">
-        <mechanicalReduction>50</mechanicalReduction>
+      <actuator name="${prefix}_motor">
+        <mechanicalReduction>1</mechanicalReduction>
+        <hardwareInterface>EffortJointInterface</hardwareInterface>
       </actuator>
     </transmission>
-    <gazebo reference="${prefix}_wheel_case">
+    <gazebo reference="${prefix}_link">
       <mu1 value="1.0"/>
       <mu2 value="1.0"/>
@@ -70,10 +97,4 @@
       <turnGravityOff>false</turnGravityOff>
     </gazebo>
-    <!-- <gazebo>
-      <plugin name="gazebo_ros_joint_state_publisher_${prefix}" filename="libgazebo_ros_joint_state_publisher.so">
-      <update_rate>100</update_rate>
-      <joint_name>${prefix}_wheel_joint</joint_name>
-      </plugin>
-    </gazebo> -->
   </xacro:macro>
 </robot>

File: src/follow_me_robot/urdf/core/robot_body.urdf.xacro (robot description, xacro)
@@ -1,4 +1,4 @@
 <?xml version="1.0"?>
-<robot name="robot" xmlns:xacro="http://www.ros.org/wiki/xacro">
+<robot xmlns="http://www.ros.org" name="robot" xmlns:xacro="http://www.ros.org/wiki/xacro">
   <xacro:include filename="inertial.urdf.xacro"/>
   <xacro:include filename="material.xacro"/>
@@ -6,4 +6,9 @@
   <xacro:macro name="robot_body" params="wheel_radius body_length body_with body_heigth">
   <!-- Robot mechanical and motor parameters -->
+  <joint name="robot_body_joint" type="fixed">
+		<parent link="base_footprint"/>
+		<child link="robot_body_link" />
+		<origin xyz="0 0 ${wheel_radius}" rpy="0 0 0" />
+	</joint>
   <!-- BASE_LINK -->
   <link name="robot_body_link">

File: src/follow_me_robot/urdf/robot.urdf.xacro (robot description, xacro)
@@ -1,4 +1,4 @@
 <?xml version="1.0"?>
-<robot name="robot"
+<robot xmlns="http://www.ros.org" name="robot"
 	xmlns:xacro="http://www.ros.org/wiki/xacro">
 	<!-- Robot Size -->
@@ -10,5 +10,5 @@
 	<xacro:property name="wheel_offset_x" value="0.25" />
 	<!-- x,y,z in translation from base_link to the center of the wheel -->
-	<xacro:property name="wheel_offset_y" value="${(body_with/2)}" />
+	<xacro:property name="wheel_offset_y" value="${(body_with/2+0.051)}" />
 	<xacro:property name="wheel_offset_z" value="0.0" />
 	<xacro:property name="wheel_radius" value="0.127" />
@@ -24,9 +24,4 @@
 		</visual>
 	</link>
-	<joint name="robot_footprint_joint" type="fixed">
-		<parent link="base_footprint"/>
-		<child link="robot_body_link" />
-		<origin xyz="0 0 ${wheel_radius}" rpy="0 0 0" />
-	</joint>
 	<xacro:include filename="core/material.xacro" />
 	<xacro:materials />
@@ -36,16 +31,27 @@
 	<!-- Additional params -->
 	<xacro:robot_body wheel_radius="${wheel_radius}" body_length="${body_length}" body_with="${body_with}" body_heigth="${body_heigth}" />
-	<xacro:omni_wheel position="front" side="right" parent="robot_body_link" reflect="2" wheel_height="${wheel_height}" wheel_radius="${wheel_radius}" x="${wheel_offset_x}" y="-${wheel_offset_y}" z="${wheel_offset_z}" />
-	<xacro:omni_wheel position="front" side="left" parent="robot_body_link" reflect="2" wheel_height="${wheel_height}" wheel_radius="${wheel_radius}" x="${wheel_offset_x}" y="${wheel_offset_y}" z="${wheel_offset_z}"/>
-	<xacro:omni_wheel position="back" side="left" parent="robot_body_link" reflect="1" wheel_height="${wheel_height}" wheel_radius="${wheel_radius}" x="-${wheel_offset_x}" y="${wheel_offset_y}" z="${wheel_offset_z}" />
-	<xacro:omni_wheel position="back" side="right" parent="robot_body_link" reflect="1" wheel_height="${wheel_height}" wheel_radius="${wheel_radius}" x="-${wheel_offset_x}" y="-${wheel_offset_y}" z="${wheel_offset_z}" />
+	<xacro:wheel_motor parent="robot_body_link" position="front" side="right" reflect="-1" wheel_img="2" wheel_height="${wheel_height}" wheel_radius="${wheel_radius}" >
+		<origin xyz="${wheel_offset_x} -${wheel_offset_y} ${wheel_offset_z}" rpy="0.0 0.0 0.0"/>
+	</xacro:wheel_motor>
+	<xacro:wheel_motor parent="robot_body_link" position="front" side="left" reflect="1" wheel_img="2" wheel_height="${wheel_height}" wheel_radius="${wheel_radius}">
+		<origin xyz="${wheel_offset_x} ${wheel_offset_y} ${wheel_offset_z}" rpy="0 0 0" />
+	</xacro:wheel_motor>
+	<xacro:wheel_motor parent="robot_body_link" position="back" side="left" reflect="1"  wheel_img="1" wheel_height="${wheel_height}" wheel_radius="${wheel_radius}">
+		<origin xyz="-${wheel_offset_x} ${wheel_offset_y} ${wheel_offset_z}" rpy="0 0 0" />
+	</xacro:wheel_motor>
+	<xacro:wheel_motor parent="robot_body_link" position="back" side="right" reflect="-1" wheel_img="1" wheel_height="${wheel_height}" wheel_radius="${wheel_radius}">
+		<origin xyz="-${wheel_offset_x} -${wheel_offset_y} ${wheel_offset_z}" rpy="0 0 0" />
+	</xacro:wheel_motor>
 	<xacro:omni_steering />
 	<!-- <xacro:ros_joint_pose_trajectory /> -->
 	<gazebo>
+		<plugin name="gazebo_ros_joint_pose_trajectory" filename="libgazebo_ros_joint_pose_trajectory.so">
+			<update_rate>2</update_rate>
+		</plugin>
 		<plugin name="gazebo_ros_joint_state_publisher" filename="libgazebo_ros_joint_state_publisher.so">
-		<ros>
+		<!-- <ros>
 			<namespace>/</namespace>
 			<remapping>joint_states:=joint_states</remapping>
-		</ros>
+		</ros> -->
 		<update_rate>2</update_rate>
 		<joint_name>front_right_wheel_joint</joint_name>
@@ -53,7 +59,4 @@
 		<joint_name>back_left_wheel_joint</joint_name>
 		<joint_name>back_right_wheel_joint</joint_name>
-		</plugin>
-		<plugin name="gazebo_ros_joint_pose_trajectory" filename="libgazebo_ros_joint_pose_trajectory.so">
-			<update_rate>2</update_rate>
 		</plugin>
 	</gazebo>

Commit message: update robot model

File: src/follow_me_robot/urdf/core/omni_wheel.urdf.xacro (robot description, xacro)
@@ -4,10 +4,4 @@
   <xacro:include filename="inertial.urdf.xacro"/>
   <!-- Wheels -->
-  <xacro:macro name="omni_wheel_geometry" params="parent *origin wheel_img side position wheel_height wheel_radius update_rate:=20">
-    <xacro:solid_sphere name="${position}_${side}_wheel" mass="6.5" visual="omni_wheel_${wheel_img}.dae" xyz_axis="0 1 0">
-      <xacro:insert_block name="origin" />
-      <geometry></geometry>
-    </xacro:solid_sphere>
-  </xacro:macro>
   <xacro:macro name="wheel_motor" params="parent *origin wheel_img reflect side position wheel_height wheel_radius update_rate:=20">
     <xacro:property name="prefix" value="${position}_${side}_wheel" />
@@ -41,5 +35,5 @@
     </link>
     <xacro:omni_wheel parent="${prefix}_motor_link" wheel_img="${wheel_img}" side="${side}" position="${position}" wheel_height="${wheel_height}" wheel_radius="${wheel_radius}" update_rate="${update_rate}">
-      <origin xyz="0 ${motor_offset+(wheel_height+0.01)*reflect} 0" />
+      <origin xyz="0 ${motor_offset+(wheel_height+0.01)*reflect} 0" rpy="${pi/2} ${pi/2} 0"/>
     </xacro:omni_wheel>
   </xacro:macro>
@@ -58,6 +52,6 @@
     <link name="${prefix}_link">
       <visual>
-        <origin xyz="0 0 0" rpy="0 0 0" />
-        <!-- <origin xyz="0 0 0" rpy="${pi/2} 0 0" /> -->
+        <!-- <origin xyz="0 0 0" rpy="0 0 0" /> -->
+        <origin xyz="0 0 0" rpy="${pi/2} 0 0" />
         <geometry>
           <mesh filename="file://$(find follow_me_robot)/urdf/meshes/omni_wheel_${wheel_img}.dae" />
@@ -66,5 +60,5 @@
       </visual>
       <collision>
-        <origin xyz="0 0 0" rpy="${pi/2} 0 0" />
+        <origin xyz="0 0 0" rpy="0 0 0" />
         <geometry>
           <!-- <mesh filename="file://$(find follow_me_robot)/urdf/meshes/omni_wheel_${reflect}.dae" /> -->

File: src/follow_me_robot/urdf/core/robot_body.urdf.xacro (robot description, xacro)
@@ -16,5 +16,7 @@
       <mass value="125.0" />
       <origin xyz="0 0 0" />
-      <xacro:solid_cuboid_inertia m="125.0" h="${body_heigth}" d="${body_length}" w="${body_with}" />
+      <!-- <xacro:solid_cuboid_inertia m="125.0" h="${body_heigth}" d="${body_length}" w="${body_with}" /> -->
+      <!-- <xacro:solid_cuboid_inertia m="125.0" h="${body_length}" d="${body_with}" w="${body_heigth}" /> -->
+      <xacro:solid_cuboid_inertia m="125.0" h="${body_with}" d="${body_heigth}" w="${body_length}" />
     </inertial>
     <visual>

File: src/follow_me_robot/urdf/robot.urdf.xacro (robot description, xacro)
@@ -32,5 +32,5 @@
 	<xacro:robot_body wheel_radius="${wheel_radius}" body_length="${body_length}" body_with="${body_with}" body_heigth="${body_heigth}" />
 	<xacro:wheel_motor parent="robot_body_link" position="front" side="right" reflect="-1" wheel_img="2" wheel_height="${wheel_height}" wheel_radius="${wheel_radius}" >
-		<origin xyz="${wheel_offset_x} -${wheel_offset_y} ${wheel_offset_z}" rpy="0.0 0.0 0.0"/>
+		<origin xyz="${wheel_offset_x} -${wheel_offset_y} ${wheel_offset_z}" rpy="0 0 0.0"/>
 	</xacro:wheel_motor>
 	<xacro:wheel_motor parent="robot_body_link" position="front" side="left" reflect="1" wheel_img="2" wheel_height="${wheel_height}" wheel_radius="${wheel_radius}">
