Commit message: Refactor/setup scripts (#1)

File: src/follow_me_robot/urdf/core/omni_wheel.urdf.xacro (robot description, xacro)
@@ -1,59 +1,93 @@
 <?xml version="1.0"?>
-<robot name="wheel" xmlns:xacro="http://www.ros.org/wiki/xacro">
+<robot name="wheel"
+  xmlns:xacro="http://www.ros.org/wiki/xacro">
   <xacro:include filename="inertial.urdf.xacro"/>
   <!-- Wheels -->
-  <xacro:macro name="omni_wheel_geometry" params="wheel_height wheel_radius reflect">
-    <origin xyz="0 0 0" rpy="0 0 0" />
-    <geometry>
-      <mesh filename="file://$(find follow_me_robot)/urdf/meshes/omni_wheel_${reflect}.dae" />
-      <cylinder length="${wheel_height}" radius="${wheel_radius}" />
-    </geometry>
-  </xacro:macro>
-  <xacro:macro name="omni_wheel" params="prefix parent *origin reflect wheel_height wheel_radius update_rate:=20">
-    <xacro:property name="wheel_mass" value="6.5" /> <!-- in kg-->
-    <joint name="${prefix}_wheel_joint" type="continuous">
+  <xacro:macro name="wheel_motor" params="parent *origin wheel_img reflect side position wheel_height wheel_radius update_rate:=20">
+    <xacro:property name="prefix" value="${position}_${side}_wheel" />
+    <xacro:property name="motor_mass" value="0.1" />
+    <xacro:property name="motor_h" value="0.1" />
+    <xacro:property name="motor_d" value="0.1" />
+    <xacro:property name="motor_w" value="0.1" />
+    <xacro:property name="motor_offset" value="${motor_w/1.08 * reflect * -1}"/>
+    <joint name="${prefix}_motor_joint" type="fixed">
       <parent link="${parent}"/>
-      <child link="${prefix}_wheel_link"/>
+      <child link="${prefix}_motor_link" />
       <xacro:insert_block name="origin" />
-      <axis xyz="0 1 0" rpy="0 0 0" />
-      <limit effort="100" velocity="100"/>
-      <joint_properties damping="0.0" friction="0.0"/>
     </joint>
-    <link name="${prefix}_wheel_link">
+    <link name="${prefix}_motor_link">
       <visual>
-        <xacro:omni_wheel_geometry reflect="${reflect}"
-          wheel_height="${wheel_height}"
-          wheel_radius="${wheel_radius}" />
+        <origin xyz="0 ${motor_offset} 0" rpy="0 0 0" />
+        <geometry>
+          <box size="${motor_d} ${motor_w} ${motor_h}" />
+        </geometry>
       </visual>
       <collision>
-				<origin xyz="0 0 0" rpy="${pi/2} 0 0" />
+        <origin xyz="0 0 0" rpy="0 0 0" />
+        <geometry>
+          <box size="${motor_d} ${motor_w} ${motor_h}" />
+        </geometry>
+      </collision>
+      <inertial>
+        <mass value="${motor_mass}" />
+        <xacro:solid_cuboid_inertia m="${motor_mass}" d="${motor_d}" w="${motor_w}" h="${motor_h}"/>
+      </inertial>
+    </link>
+    <xacro:omni_wheel parent="${prefix}_motor_link" wheel_img="${wheel_img}" side="${side}" position="${position}" wheel_height="${wheel_height}" wheel_radius="${wheel_radius}" update_rate="${update_rate}">
+      <origin xyz="0 ${motor_offset+(wheel_height+0.01)*reflect} 0" rpy="${pi/2} ${pi/2} 0"/>
+    </xacro:omni_wheel>
+  </xacro:macro>
+  <xacro:macro name="omni_wheel" params="parent *origin wheel_img side position wheel_height wheel_radius update_rate:=20">
+    <xacro:property name="wheel_mass" value="6.5" />
+    <xacro:property name="prefix" value="${position}_${side}_wheel" />
+    <!-- in kg-->
+    <joint name="${prefix}_joint" type="continuous">
+      <parent link="${parent}"/>
+      <child link="${prefix}_link"/>
+      <xacro:insert_block name="origin" />
+      <axis xyz="0 1 0" />
+      <limit effort="100" velocity="0"/>
+      <joint_properties damping="0.0" friction="1.0"/>
+    </joint>
+    <link name="${prefix}_link">
+      <visual>
         <!-- <origin xyz="0 0 0" rpy="0 0 0" /> -->
-      <geometry>
-        <!-- <mesh filename="file://$(find follow_me_robot)/urdf/meshes/omni_wheel_${reflect}.dae" /> -->
-        <cylinder length="${wheel_height}" radius="${wheel_radius}" />
-      </geometry>
+        <origin xyz="0 0 0" rpy="${pi/2} 0 0" />
+        <geometry>
+          <mesh filename="file://$(find follow_me_robot)/urdf/meshes/omni_wheel_${wheel_img}.dae" />
+          <!-- <cylinder length="${wheel_height}" radius="${wheel_radius}" /> -->
+        </geometry>
+      </visual>
+      <collision>
+        <origin xyz="0 0 0" rpy="0 0 0" />
+        <geometry>
+          <!-- <mesh filename="file://$(find follow_me_robot)/urdf/meshes/omni_wheel_${reflect}.dae" /> -->
+          <cylinder length="${wheel_height}" radius="${wheel_radius}" />
+        </geometry>
       </collision>
       <inertial>
         <mass value="${wheel_mass}" />
-        <xacro:solid_cylinder_inertia  m="${wheel_mass}" r="${wheel_radius}" h="${wheel_height}" />
+        <xacro:solid_cylinder_inertia m="${wheel_mass}" r="${wheel_radius}" h="${wheel_height}" />
       </inertial>
     </link>
     <!-- Transmission is important to link the joints and the controller (see robot_control/config/robot_control.yaml)-->
-    <transmission name="${prefix}_wheel_joint_trans">
+    <transmission name="${prefix}_joint_trans" type="transmission_interface/SimpleTransmission">
       <type>transmission_interface/SimpleTransmission</type>
-      <joint name="${prefix}_wheel_joint" >
-        <hardwareInterface>hardware_interface/VelocityJointInterface</hardwareInterface>
+      <joint name="${prefix}_joint">
+        <!-- <hardwareInterface>hardware_interface/VelocityJointInterface</hardwareInterface> -->
+        <hardwareInterface>EffortJointInterface</hardwareInterface>
       </joint>
-      <actuator name="${prefix}_wheel_joint_motor">
-         <mechanicalReduction>1</mechanicalReduction>
+      <actuator name="${prefix}_motor">
+        <mechanicalReduction>1</mechanicalReduction>
+        <hardwareInterface>EffortJointInterface</hardwareInterface>
       </actuator>
     </transmission>
-    <gazebo reference="${prefix}_wheel_link">
-		<mu1 value="1.0"/>
-		<mu2 value="1.0"/>
-		<kp value="10000000.0" />
-		<kd value="1.0" />
-		<fdir1 value="1 0 0"/>
-        <turnGravityOff>false</turnGravityOff>
+    <gazebo reference="${prefix}_link">
+      <mu1 value="1.0"/>
+      <mu2 value="1.0"/>
+      <kp value="10000000.0" />
+      <kd value="1.0" />
+      <fdir1 value="1 0 0"/>
+      <turnGravityOff>false</turnGravityOff>
     </gazebo>
   </xacro:macro>

File: src/follow_me_robot/urdf/core/robot_body.urdf.xacro (robot description, xacro)
@@ -1,9 +1,14 @@
 <?xml version="1.0"?>
-<robot name="robot" xmlns:xacro="http://www.ros.org/wiki/xacro">
+<robot xmlns="http://www.ros.org" name="robot" xmlns:xacro="http://www.ros.org/wiki/xacro">
   <xacro:include filename="inertial.urdf.xacro"/>
   <xacro:include filename="material.xacro"/>
   <xacro:include filename="follow_me_robot.gazebo.xacro" />
   <xacro:macro name="robot_body" params="wheel_radius body_length body_with body_heigth">
-	  <!-- Robot mechanical and motor parameters -->
+  <!-- Robot mechanical and motor parameters -->
+  <joint name="robot_body_joint" type="fixed">
+		<parent link="base_footprint"/>
+		<child link="robot_body_link" />
+		<origin xyz="0 0 ${wheel_radius}" rpy="0 0 0" />
+	</joint>
   <!-- BASE_LINK -->
   <link name="robot_body_link">
@@ -11,5 +16,7 @@
       <mass value="125.0" />
       <origin xyz="0 0 0" />
-      <xacro:solid_cuboid_inertia m="125.0" h="${body_heigth}" d="${body_length}" w="${body_with}" />
+      <!-- <xacro:solid_cuboid_inertia m="125.0" h="${body_heigth}" d="${body_length}" w="${body_with}" /> -->
+      <!-- <xacro:solid_cuboid_inertia m="125.0" h="${body_length}" d="${body_with}" w="${body_heigth}" /> -->
+      <xacro:solid_cuboid_inertia m="125.0" h="${body_with}" d="${body_heigth}" w="${body_length}" />
     </inertial>
     <visual>
@@ -17,4 +24,5 @@
         <geometry>
             <box size="${body_length} ${body_with} ${body_heigth}"/>
+            <!-- <box size="0.01 ${body_with} 0.01"/> -->
         </geometry>
     </visual>

File: src/follow_me_robot/urdf/robot.urdf.xacro (robot description, xacro)
@@ -1,4 +1,4 @@
 <?xml version="1.0"?>
-<robot name="robot"
+<robot xmlns="http://www.ros.org" name="robot"
 	xmlns:xacro="http://www.ros.org/wiki/xacro">
 	<!-- Robot Size -->
@@ -10,5 +10,5 @@
 	<xacro:property name="wheel_offset_x" value="0.25" />
 	<!-- x,y,z in translation from base_link to the center of the wheel -->
-	<xacro:property name="wheel_offset_y" value="${(body_with/2)+(wheel_height/2)+0.01}" />
+	<xacro:property name="wheel_offset_y" value="${(body_with/2+0.051)}" />
 	<xacro:property name="wheel_offset_z" value="0.0" />
 	<xacro:property name="wheel_radius" value="0.127" />
@@ -16,4 +16,5 @@
 	<!-- BASE FOOTPRINT -->
 	<link name="base_footprint">
+		<must_be_base_link>true</must_be_base_link>
 		<visual>
 			<origin xyz="0 0 0" rpy="0 0 0" />
@@ -23,9 +24,4 @@
 		</visual>
 	</link>
-	<joint name="robot_footprint_joint" type="fixed">
-		<parent link="base_footprint"/>
-		<child link="robot_body_link" />
-		<origin xyz="0 0 ${wheel_radius}" rpy="0 0 0" />
-	</joint>
 	<xacro:include filename="core/material.xacro" />
 	<xacro:materials />
@@ -35,30 +31,32 @@
 	<!-- Additional params -->
 	<xacro:robot_body wheel_radius="${wheel_radius}" body_length="${body_length}" body_with="${body_with}" body_heigth="${body_heigth}" />
-	<xacro:omni_wheel prefix="front_right" parent="robot_body_link" reflect="2" wheel_height="${wheel_height}" wheel_radius="${wheel_radius}">
-		<origin xyz="${wheel_offset_x} -${wheel_offset_y} ${wheel_offset_z}" rpy="0 0 0" />
-	</xacro:omni_wheel>
-	<xacro:omni_wheel prefix="front_left" parent="robot_body_link" reflect="2" wheel_height="${wheel_height}" wheel_radius="${wheel_radius}">
+	<xacro:wheel_motor parent="robot_body_link" position="front" side="right" reflect="-1" wheel_img="2" wheel_height="${wheel_height}" wheel_radius="${wheel_radius}" >
+		<origin xyz="${wheel_offset_x} -${wheel_offset_y} ${wheel_offset_z}" rpy="0 0 0.0"/>
+	</xacro:wheel_motor>
+	<xacro:wheel_motor parent="robot_body_link" position="front" side="left" reflect="1" wheel_img="2" wheel_height="${wheel_height}" wheel_radius="${wheel_radius}">
 		<origin xyz="${wheel_offset_x} ${wheel_offset_y} ${wheel_offset_z}" rpy="0 0 0" />
-	</xacro:omni_wheel>
-	<xacro:omni_wheel prefix="back_left" parent="robot_body_link" reflect="1" wheel_height="${wheel_height}" wheel_radius="${wheel_radius}">
+	</xacro:wheel_motor>
+	<xacro:wheel_motor parent="robot_body_link" position="back" side="left" reflect="1"  wheel_img="1" wheel_height="${wheel_height}" wheel_radius="${wheel_radius}">
 		<origin xyz="-${wheel_offset_x} ${wheel_offset_y} ${wheel_offset_z}" rpy="0 0 0" />
-	</xacro:omni_wheel>
-	<xacro:omni_wheel prefix="back_right" parent="robot_body_link" reflect="1" wheel_height="${wheel_height}" wheel_radius="${wheel_radius}">
+	</xacro:wheel_motor>
+	<xacro:wheel_motor parent="robot_body_link" position="back" side="right" reflect="-1" wheel_img="1" wheel_height="${wheel_height}" wheel_radius="${wheel_radius}">
 		<origin xyz="-${wheel_offset_x} -${wheel_offset_y} ${wheel_offset_z}" rpy="0 0 0" />
-	</xacro:omni_wheel>
+	</xacro:wheel_motor>
 	<xacro:omni_steering />
 	<!-- <xacro:ros_joint_pose_trajectory /> -->
 	<gazebo>
+		<plugin name="gazebo_ros_joint_pose_trajectory" filename="libgazebo_ros_joint_pose_trajectory.so">
+			<update_rate>2</update_rate>
+		</plugin>
 		<plugin name="gazebo_ros_joint_state_publisher" filename="libgazebo_ros_joint_state_publisher.so">
-			<update_rate>${update_rate}</update_rate>
-			<!-- <joint_name>robot_footprint_joint</joint_name> -->
-			<joint_name>front_right_wheel_joint</joint_name>
-			<joint_name>front_left_wheel_joint</joint_name>
-			<joint_name>back_left_wheel_joint</joint_name>
-			<joint_name>back_right_wheel_joint</joint_name>
-		</plugin>
-		<plugin name="gazebo_ros_joint_pose_trajectory"
-			filename="libgazebo_ros_joint_pose_trajectory.so">
-			<update_rate>${update_rate}</update_rate>
+		<!-- <ros>
+			<namespace>/</namespace>
+			<remapping>joint_states:=joint_states</remapping>
+		</ros> -->
+		<update_rate>2</update_rate>
+		<joint_name>front_right_wheel_joint</joint_name>
+		<joint_name>front_left_wheel_joint</joint_name>
+		<joint_name>back_left_wheel_joint</joint_name>
+		<joint_name>back_right_wheel_joint</joint_name>
 		</plugin>
 	</gazebo>
@@ -67,8 +65,8 @@
 		<origin xyz="0 0 ${body_heigth/2+0.03}" rpy="0 0 0" />
 	</xacro:lidar>
-	<!-- <xacro:include filename="sensors/gps.xacro" />
+	<xacro:include filename="sensors/gps.xacro" />
 	<xacro:gps parent="robot_body_link">
 		<origin xyz="0 0 0.0"/>
-	</xacro:gps> -->
+	</xacro:gps>
 	<xacro:include filename="sensors/imu.xacro" />
 	<xacro:imu parent="robot_body_link">
