Commit message: let robot detect tag from walking actor

File: src/follow_me_robot/urdf/core/omni_wheel.urdf.xacro (robot description, xacro)
@@ -1,8 +1,8 @@
 <?xml version="1.0"?>
-<robot name="wheel"
-  xmlns:xacro="http://www.ros.org/wiki/xacro">
-  <xacro:include filename="inertial.urdf.xacro"/>
-  <!-- Wheels -->
-  <xacro:macro name="wheel_motor" params="parent *origin wheel_img reflect side position wheel_height wheel_radius update_rate:=20">
+<robot name="wheel" xmlns:xacro="http://www.ros.org/wiki/xacro">
+  <xacro:include filename="inertial.urdf.xacro" />
+  <!-- Motro -->
+  <xacro:macro name="wheel_motor"
+    params="parent *origin wheel_img reflect side position wheel_height wheel_radius update_rate:=20">
     <xacro:property name="prefix" value="${position}_${side}_wheel" />
     <xacro:property name="motor_mass" value="0.1" />
@@ -10,7 +10,7 @@
     <xacro:property name="motor_d" value="0.1" />
     <xacro:property name="motor_w" value="0.1" />
-    <xacro:property name="motor_offset" value="${motor_w/1.08 * reflect * -1}"/>
+    <xacro:property name="motor_offset" value="${motor_w/1.08 * reflect * -1}" />
     <joint name="${prefix}_motor_joint" type="fixed">
-      <parent link="${parent}"/>
+      <parent link="${parent}" />
       <child link="${prefix}_motor_link" />
       <xacro:insert_block name="origin" />
@@ -32,22 +32,25 @@
       <inertial>
         <mass value="${motor_mass}" />
-        <xacro:solid_cuboid_inertia m="${motor_mass}" d="${motor_d}" w="${motor_w}" h="${motor_h}"/>
+        <xacro:solid_cuboid_inertia m="${motor_mass}" d="${motor_d}" w="${motor_w}" h="${motor_h}" />
       </inertial>
     </link>
-    <xacro:omni_wheel parent="${prefix}_motor_link" wheel_img="${wheel_img}" side="${side}" position="${position}" wheel_height="${wheel_height}" wheel_radius="${wheel_radius}" update_rate="${update_rate}">
-      <origin xyz="0 ${motor_offset+(wheel_height+0.01)*reflect} 0" rpy="${pi/2} ${pi/2} 0"/>
+    <xacro:omni_wheel parent="${prefix}_motor_link" wheel_img="${wheel_img}" side="${side}"
+      position="${position}" wheel_height="${wheel_height}" wheel_radius="${wheel_radius}"
+      update_rate="${update_rate}">
+      <origin xyz="0 ${motor_offset+(wheel_height+0.01)*reflect} 0" rpy="${pi/2} ${pi/2} 0" />
     </xacro:omni_wheel>
   </xacro:macro>
-  <xacro:macro name="omni_wheel" params="parent *origin wheel_img side position wheel_height wheel_radius update_rate:=20">
+  <!-- Wheel -->
+  <xacro:macro name="omni_wheel"
+    params="parent *origin wheel_img side position wheel_height wheel_radius update_rate:=20">
+    <!-- in kg-->
     <xacro:property name="wheel_mass" value="6.5" />
     <xacro:property name="prefix" value="${position}_${side}_wheel" />
-    <!-- in kg-->
     <joint name="${prefix}_joint" type="continuous">
-      <parent link="${parent}"/>
-      <child link="${prefix}_link"/>
+      <parent link="${parent}" />
+      <child link="${prefix}_link" />
       <xacro:insert_block name="origin" />
       <axis xyz="0 0 1" />
-      <!-- <limit effort="100" velocity="0"/> -->
-      <joint_properties damping="0.0" friction="1.0"/>
+      <joint_properties damping="0.0" friction="1.0" />
     </joint>
     <link name="${prefix}_link">
@@ -64,10 +67,8 @@
           <mesh filename="file://$(find follow_me_robot)/urdf/meshes/omni_wheel_${wheel_img}.dae" />
         </geometry>
-        <material name="black" />
       </visual>
       <collision>
         <origin xyz="0 0 0" rpy="0 0 0" />
         <geometry>
-          <!-- <mesh filename="file://$(find follow_me_robot)/urdf/meshes/omni_wheel_${reflect}.dae" /> -->
           <cylinder length="${wheel_height}" radius="${wheel_radius}" />
         </geometry>
@@ -78,5 +79,6 @@
       </inertial>
     </link>
-    <!-- Transmission is important to link the joints and the controller (see robot_control/config/robot_control.yaml)-->
+    <!-- Transmission is important to link the joints and the controller (see
+    robot_control/config/robot_control.yaml)-->
     <transmission name="${prefix}_joint_trans" type="transmission_interface/SimpleTransmission">
       <type>transmission_interface/SimpleTransmission</type>
@@ -91,9 +93,9 @@
     </transmission>
     <gazebo reference="${prefix}_link">
-      <mu1 value="1.0"/>
-      <mu2 value="1.0"/>
+      <mu1 value="1.0" />
+      <mu2 value="1.0" />
       <kp value="10000000.0" />
       <kd value="1.0" />
-      <fdir1 value="1 0 0"/>
+      <fdir1 value="1 0 0" />
       <turnGravityOff>false</turnGravityOff>
     </gazebo>

File: src/follow_me_robot/urdf/core/robot_body.urdf.xacro (robot description, xacro)
@@ -1,37 +1,35 @@
 <?xml version="1.0"?>
 <robot xmlns="http://www.ros.org" name="robot" xmlns:xacro="http://www.ros.org/wiki/xacro">
-  <xacro:include filename="inertial.urdf.xacro"/>
-  <xacro:include filename="material.xacro"/>
-  <xacro:include filename="follow_me_robot.gazebo.xacro" />
+  <xacro:include filename="inertial.urdf.xacro" />
+  <xacro:include filename="material.xacro" />
   <xacro:macro name="robot_body" params="wheel_radius body_length body_with body_heigth">
-  <!-- Robot mechanical and motor parameters -->
-  <joint name="robot_body_joint" type="fixed">
-		<parent link="base_link"/>
-		<child link="robot_body_link" />
-		<origin xyz="0 0 ${wheel_radius}" rpy="0 0 0" />
-	</joint>
-  <!-- BASE_LINK -->
-  <link name="robot_body_link">
-    <inertial>
-      <mass value="125.0" />
-      <origin xyz="0 0 0" />
-      <!-- <xacro:solid_cuboid_inertia m="125.0" h="${body_heigth}" d="${body_length}" w="${body_with}" /> -->
-      <!-- <xacro:solid_cuboid_inertia m="125.0" h="${body_length}" d="${body_with}" w="${body_heigth}" /> -->
-      <xacro:solid_cuboid_inertia m="125.0" h="${body_with}" d="${body_heigth}" w="${body_length}" />
-    </inertial>
-    <visual>
-       <origin xyz="0 0 0" rpy="0 0 0" />
+    <!-- Robot mechanical and motor parameters -->
+    <joint name="robot_body_joint" type="fixed">
+      <parent link="base_link" />
+      <child link="robot_body_link" />
+      <origin xyz="0 0 ${wheel_radius}" rpy="0 0 0" />
+    </joint>
+    <!-- BASE_LINK -->
+    <link name="robot_body_link">
+      <inertial>
+        <mass value="125.0" />
+        <origin xyz="0 0 0" />
+        <xacro:solid_cuboid_inertia m="125.0" h="${body_with}" d="${body_heigth}" w="${body_length}" />
+      </inertial>
+      <visual>
+        <origin xyz="0 0 0" rpy="0 0 0" />
+        <material name="orange" />
         <geometry>
-            <box size="${body_length} ${body_with} ${body_heigth}"/>
-            <!-- <box size="0.01 ${body_with} 0.01"/> -->
+          <box size="${body_length} ${body_with} ${body_heigth}" />
+          <!-- <box size="0.01 ${body_with} 0.01"/> -->
         </geometry>
-    </visual>
-    <collision>
-       <origin xyz="0 0 0" rpy="0 0 0 " />
-       <geometry>
-            <box size="${body_length} ${body_with} ${body_heigth}"/>
+      </visual>
+      <collision>
+        <origin xyz="0 0 0" rpy="0 0 0 " />
+        <geometry>
+          <box size="${body_length} ${body_with} ${body_heigth}" />
         </geometry>
-    </collision>
-  </link>
+      </collision>
+    </link>
   </xacro:macro>
 </robot>

File: src/follow_me_robot/urdf/robot.urdf.xacro (robot description, xacro)
@@ -4,6 +4,6 @@
 	<!-- Robot Size -->
 	<xacro:property name="body_length" value="0.80" />
-	<xacro:property name="body_with" value="0.5"/>
-	<xacro:property name="body_heigth" value="0.20"/>
+	<xacro:property name="body_with" value="0.5" />
+	<xacro:property name="body_heigth" value="0.20" />
 	<xacro:property name="wheel_height" value="0.087" />
 	<!-- Wheel parameters -->
@@ -13,11 +13,11 @@
 	<xacro:property name="wheel_offset_z" value="0.0" />
 	<xacro:property name="wheel_radius" value="0.127" />
-	<xacro:property name="update_rate" value="20" />
-	<link name="base_footprint"/>
+	<xacro:property name="update_rate" value="30" />
+	<link name="base_footprint" />
 	<joint name="odom_joint" type="fixed">
-    <parent link="base_footprint"/>
-    <child link="base_link" />
+		<parent link="base_footprint" />
+		<child link="base_link" />
 		<origin xyz="0 0 0.001" />
-  </joint>
+	</joint>
 	<!-- BASE FOOTPRINT -->
 	<link name="base_link"></link>
@@ -26,48 +26,61 @@
 	<xacro:include filename="core/omni_wheel.urdf.xacro" />
 	<xacro:include filename="core/robot_body.urdf.xacro" />
-	<xacro:include filename="core/follow_me_robot.gazebo.xacro" />
 	<!-- Additional params -->
-	<xacro:robot_body wheel_radius="${wheel_radius}" body_length="${body_length}" body_with="${body_with}" body_heigth="${body_heigth}" />
-	<xacro:wheel_motor parent="robot_body_link" position="front" side="right" reflect="-1" wheel_img="2" wheel_height="${wheel_height}" wheel_radius="${wheel_radius}" >
-		<origin xyz="${wheel_offset_x} -${wheel_offset_y} ${wheel_offset_z}" rpy="0 0 0.0"/>
+	<xacro:robot_body wheel_radius="${wheel_radius}" body_length="${body_length}"
+		body_with="${body_with}" body_heigth="${body_heigth}" />
+	<xacro:wheel_motor parent="robot_body_link" position="front" side="right" reflect="-1"
+		wheel_img="2" wheel_height="${wheel_height}" wheel_radius="${wheel_radius}">
+		<origin xyz="${wheel_offset_x} -${wheel_offset_y} ${wheel_offset_z}" rpy="0 0 0.0" />
 	</xacro:wheel_motor>
-	<xacro:wheel_motor parent="robot_body_link" position="front" side="left" reflect="1" wheel_img="2" wheel_height="${wheel_height}" wheel_radius="${wheel_radius}">
+	<xacro:wheel_motor parent="robot_body_link" position="front" side="left" reflect="1" wheel_img="2"
+		wheel_height="${wheel_height}" wheel_radius="${wheel_radius}">
 		<origin xyz="${wheel_offset_x} ${wheel_offset_y} ${wheel_offset_z}" rpy="0 0 0" />
 	</xacro:wheel_motor>
-	<xacro:wheel_motor parent="robot_body_link" position="back" side="left" reflect="1"  wheel_img="1" wheel_height="${wheel_height}" wheel_radius="${wheel_radius}">
+	<xacro:wheel_motor parent="robot_body_link" position="back" side="left" reflect="1" wheel_img="1"
+		wheel_height="${wheel_height}" wheel_radius="${wheel_radius}">
 		<origin xyz="-${wheel_offset_x} ${wheel_offset_y} ${wheel_offset_z}" rpy="0 0 0" />
 	</xacro:wheel_motor>
-	<xacro:wheel_motor parent="robot_body_link" position="back" side="right" reflect="-1" wheel_img="1" wheel_height="${wheel_height}" wheel_radius="${wheel_radius}">
+	<xacro:wheel_motor parent="robot_body_link" position="back" side="right" reflect="-1"
+		wheel_img="1" wheel_height="${wheel_height}" wheel_radius="${wheel_radius}">
 		<origin xyz="-${wheel_offset_x} -${wheel_offset_y} ${wheel_offset_z}" rpy="0 0 0" />
 	</xacro:wheel_motor>
-	<xacro:omni_steering />
 	<gazebo>
-		<!-- <plugin name="gazebo_ros_joint_pose_trajectory"
-			filename="libgazebo_ros_joint_pose_trajectory.so">
-			<update_rate>2</update_rate>
-		</plugin>	 -->
-		<plugin name="gazebo_ros_joint_state_publisher" filename="libgazebo_ros_joint_state_publisher.so">
-		<update_rate>100</update_rate>
-		<joint_name>front_right_wheel_joint</joint_name>
-		<joint_name>front_left_wheel_joint</joint_name>
-		<joint_name>back_left_wheel_joint</joint_name>
-		<joint_name>back_right_wheel_joint</joint_name>
+		<plugin name="psuedo_mecanum" filename="libgazebo_ros_planar_move.so">
+			<commandTopic>/cmd_vel</commandTopic>
+			<odometryTopic>odom</odometryTopic>
+			<odometryFrame>odom</odometryFrame>
+			<odometryRate>20.0</odometryRate>
+			<robotBaseFrame>base_link</robotBaseFrame>
+			<update_rate>${update_rate}</update_rate>
+			<publish_rate>${update_rate}</publish_rate>
+		</plugin>
+		<plugin name="gazebo_ros_joint_state_publisher"
+			filename="libgazebo_ros_joint_state_publisher.so">
+			<update_rate>${update_rate}</update_rate>
+			<joint_name>front_right_wheel_joint</joint_name>
+			<joint_name>front_left_wheel_joint</joint_name>
+			<joint_name>back_left_wheel_joint</joint_name>
+			<joint_name>back_right_wheel_joint</joint_name>
 		</plugin>
 	</gazebo>
 	<xacro:include filename="sensors/lidar.xacro" />
-	<xacro:lidar parent="robot_body_link" update="10">
+	<xacro:lidar parent="robot_body_link" update="${update_rate}">
 		<origin xyz="0 0 ${body_heigth/2+0.03}" rpy="0 0 0" />
 	</xacro:lidar>
-	<!-- <xacro:include filename="sensors/gps.xacro" />
-	<xacro:gps parent="robot_body_link">
-		<origin xyz="0 0 0.0"/>
-	</xacro:gps> -->
 	<xacro:include filename="sensors/imu.xacro" />
-	<xacro:imu parent="robot_body_link">
-		<origin xyz="0 0 0.0"/>
+	<xacro:imu parent="robot_body_link" update="${update_rate}">
+		<origin xyz="0 0 0" />
 	</xacro:imu>
 	<xacro:include filename="sensors/camera.xacro" />
-	<xacro:camera cam_name="front" parent="robot_body_link">
-		<origin xyz="${body_length/2} 0 0.0"/>
+	<xacro:camera cam_name="front" parent="robot_body_link" update="${update_rate}" visualize="true">
+		<origin xyz="${body_length/2} 0 0.1" rpy="0 -0.3 0" />
 	</xacro:camera>
+	<xacro:include filename="sensors/sonar.xacro" />
+	<xacro:sonar sonar_name="front_mid" parent="robot_body_link" update="${update_rate}">
+		<origin xyz="${body_length/2} 0 -0.05" rpy="0 0.2 0" />
+	</xacro:sonar>
+	<!-- <xacro:include filename="sensors/gps.xacro" />
+	<xacro:gps parent="robot_body_link" update="${update_rate}">
+		<origin xyz="0 0 0.0" />
+	</xacro:gps> -->
 </robot>

File: src/follow_me_robot/urdf/sensors/camera.xacro (robot description, xacro)
@@ -1,29 +1,63 @@
 <?xml version="1.0"?>
-<robot xmlns:xacro="http://www.ros.org/wiki/xacro" >
-<xacro:include filename="gazebo/cam.gazebo"/>
-<xacro:macro name="camera" params="cam_name parent *origin">
+<robot xmlns:xacro="http://www.ros.org/wiki/xacro">
+  <xacro:include filename="./macros.xacro" />
+  <xacro:macro name="camera" params="cam_name parent *origin update:=30 visualize:=false">
     <joint name="${cam_name}_camera_joint" type="fixed">
-        <parent link="${parent}"/>
-        <child link="${cam_name}_camera_link"/>
-        <xacro:insert_block name="origin" />
+      <parent link="${parent}" />
+      <child link="${cam_name}_camera_link" />
+      <xacro:insert_block name="origin" />
     </joint>
     <link name="${cam_name}_camera_link">
-        <visual>
-            <geometry>
-                <box size="0.010 0.03 0.03"/>
-            </geometry>
-            <material name="blue"/>
-        </visual>
-        <visual>
-            <origin xyz="0.005 0 0" rpy="0 ${pi/2} 0"/>
-            <geometry>
-                <cylinder radius="0.01" length="0.01"/>
-            </geometry>
-            <material name="blue"/>
-        </visual>
+      <visual>
+        <geometry>
+          <box size="0.010 0.03 0.03" />
+        </geometry>
+        <material name="blue" />
+      </visual>
+      <visual>
+        <origin xyz="0.005 0 0" rpy="0 ${pi/2} 0" />
+        <geometry>
+          <cylinder radius="0.01" length="0.01" />
+        </geometry>
+        <material name="red" />
+      </visual>
     </link>
-    <xacro:camgazebo cam_name="${cam_name}">
-        <origin xyz="0.01 0 0" rpy="${-pi/2} ${-pi/2} ${-pi/2}"/>
-    </xacro:camgazebo>
-</xacro:macro>
+    <joint name="${cam_name}_camera_optical_joint" type="fixed">
+      <parent link="${cam_name}_camera_link" />
+      <child link="${cam_name}_camera_link_optical" />
+      <origin xyz="0.01 0 0" rpy="0 0 0" />
+    </joint>
+    <link name="${cam_name}_camera_link_optical" />
+    <gazebo reference="${cam_name}_camera_link_optical">
+      <sensor type="camera" name="${cam_name}_cam">
+        <always_on>true</always_on>
+        <update_rate>${update}</update_rate>
+        <visualize>${visualize}</visualize>
+        <camera name="${cam_name}_head">
+          <horizontal_fov>1.3962634</horizontal_fov>
+          <image>
+            <width>640</width>
+            <height>480</height>
+            <format>B8G8R8</format>
+          </image>
+          <clip>
+            <near>0.002</near>
+            <far>300</far>
+          </clip>
+          <xacro:sensor_noise />
+        </camera>
+        <plugin name="camera_controller_${cam_name}" filename="libgazebo_ros_camera.so">
+          <ros>
+            <namespace>/cam</namespace>
+            <remapping>~/image_raw:=/image_raw</remapping>
+            <remapping>~/camera_info:=/camera_info</remapping>
+          </ros>
+          <camera_name>${cam_name}</camera_name>
+          <hack_baseline>0.07</hack_baseline>
+          <min_depth>0.002</min_depth>
+          <max_depth>300.0</max_depth>
+        </plugin>
+      </sensor>
+    </gazebo>
+  </xacro:macro>
 </robot>

File: src/follow_me_robot/urdf/sensors/camera_depth.xacro (robot description, xacro)
@@ -6,10 +6,10 @@
             <parent link="${parent}" />
             <child link="${camera_name}_camera_link" />
-            <origin xyz="0.305 0.5 0.08" rpy="0 0 0"/>
+            <origin xyz="0.305 0.5 0.08" rpy="0 0 0" />
         </joint>
         <link name="${camera_name}_camera_link">
             <visual>
                 <geometry>
-                    <box size="0.01 0.06 0.03"/>
+                    <box size="0.01 0.06 0.03" />
                 </geometry>
                 <material name="red" />
@@ -17,7 +17,7 @@
         </link>
         <joint name="camera_optical_joint" type="fixed">
-            <parent link="${camera_name}_camera_link"/>
-            <child link="camera_link_optical"/>
-            <origin xyz="0 0 0" rpy="0 0 0"/>
+            <parent link="${camera_name}_camera_link" />
+            <child link="camera_link_optical" />
+            <origin xyz="0 0 0" rpy="0 0 0" />
         </joint>
         <link name="camera_link_optical"></link>

File: src/follow_me_robot/urdf/sensors/gps.xacro (robot description, xacro)
@@ -2,38 +2,69 @@
 <robot name="sensor"
   xmlns:xacro="http://playerstage.sourceforge.net/gazebo/xmlschema/#interface">
-  <xacro:include filename="../core/material.xacro"/>
   <xacro:include filename="../core/inertial.urdf.xacro" />
-  <xacro:include filename="gazebo/gps.gazebo"/>
-  <xacro:macro name="gps" params="parent *origin gps_name:=sensor_0">
-    <xacro:property name="w" value="0.1"/>
-    <xacro:property name="h" value="0.1"/>
-    <xacro:property name="d" value="0.1"/>
+  <xacro:include filename="./macros.xacro" />
+  <xacro:macro name="gps" params="parent *origin gps_name:=sensor_0 update:=30">
+    <xacro:property name="w" value="0.1" />
+    <xacro:property name="h" value="0.1" />
+    <xacro:property name="d" value="0.1" />
     <joint name="${gps_name}_gps_joint" type="fixed">
-      <parent link="${parent}"/>
-      <child link="${gps_name}_gps_link"/>
+      <parent link="${parent}" />
+      <child link="${gps_name}_gps_link" />
       <xacro:insert_block name="origin" />
     </joint>
     <link name="${gps_name}_gps_link">
       <collision>
-        <origin xyz="0 0 0" rpy="0 0 0"/>
+        <origin xyz="0 0 0" rpy="0 0 0" />
         <geometry>
-          <box size="${w} ${d} ${h}"/>
+          <box size="${w} ${d} ${h}" />
         </geometry>
       </collision>
       <visual>
-        <origin xyz="0 0 0" rpy="0 0 0"/>
+        <origin xyz="0 0 0" rpy="0 0 0" />
         <geometry>
-          <box size="${w} ${d} ${h}"/>
+          <box size="${w} ${d} ${h}" />
         </geometry>
-        <material name="orange"/>
+        <material name="red" />
       </visual>
       <inertial>
-        <origin xyz="0 0 0" rpy="0 0 0"/>
-        <mass value="1"/>
+        <origin xyz="0 0 0" rpy="0 0 0" />
+        <mass value="1" />
         <xacro:solid_cuboid_inertia m="1" h="${h}" d="${d}" w="${w}" />
       </inertial>
     </link>
-    <xacro:gazebogps gps_name="${gps_name}">
-    </xacro:gazebogps>
+    <gazebo reference="${gps_name}_gps_link">
+      <sensor name="${gps_name}_gps" type="gps">
+        <always_on>true</always_on>
+        <update_rate>${update}</update_rate>
+        <gps>
+          <position_sensing>
+            <horizontal>
+              <xacro:sensor_noise />
+            </horizontal>
+            <vertical>
+              <xacro:sensor_noise />
+            </vertical>
+          </position_sensing>
+        </gps>
+        <plugin name="gazebo_ros_gps_${gps_name}" filename="libgazebo_ros_gps_sensor.so">
+          <ros>
+            <remapping>~/out:=gps</remapping>
+          </ros>
+          <!-- <bodyName>${gps_name}_gps_link</bodyName>
+      <frameId>${gps_name}_gps_link</frameId> -->
+          <!-- <topicName>/gps/fix/${gps_name}</topicName> -->
+          <!-- <velocityTopicName>/gps/fix_velocity</velocityTopicName>
+      <referenceLatitude>-30.06022459407145675</referenceLatitude>
+      <referenceLongitude>-51.173913575780311191</referenceLongitude>
+      <referenceHeading>90</referenceHeading>
+      <referenceAltitude>10</referenceAltitude>
+      <offset>0 0 0</offset>
+      <drift>0.001 0.001 0.001</drift>
+      <gaussianNoise>0.05 0.05 0.05</gaussianNoise>
+      <velocityDrift>0.001 0.001 0.001</velocityDrift>
+      <velocityGaussianNoise>0.5 0.5 0.5</velocityGaussianNoise> -->
+        </plugin>
+      </sensor>
+    </gazebo>
   </xacro:macro>
 </robot>
