Commit message: let robot detect tag from walking actor

File: src/follow_me_robot/urdf/sensors/imu.xacro (robot description, xacro)
@@ -3,6 +3,5 @@
   xmlns:xacro="http://playerstage.sourceforge.net/gazebo/xmlschema/#interface">
   <xacro:include filename="../core/inertial.urdf.xacro" />
-  <xacro:include filename="gazebo/imu.gazebo"/>
-  <xacro:macro name="imu" params="parent *origin imu_name:=sensor_0">
+  <xacro:macro name="imu" params="parent *origin imu_name:=sensor_0 update:=30">
     <joint name="${imu_name}_imu_joint" type="fixed">
       <parent link="${parent}" />
@@ -13,19 +12,63 @@
       <visual>
         <geometry>
-          <box size="0.05 0.05 0.05"/>
+          <box size="0.05 0.05 0.05" />
         </geometry>
+        <material name="red" />
       </visual>
       <collision>
         <geometry>
-          <box size="0.05 0.05 0.05"/>
+          <box size="0.05 0.05 0.05" />
         </geometry>
       </collision>
       <inertial>
         <mass value="1e-5" />
-        <origin xyz="0 0 0" rpy="0 0 0"/>
+        <origin xyz="0 0 0" rpy="0 0 0" />
         <xacro:solid_cuboid_inertia w="0.05" h="0.05" d="0.5" m="1e-5" />
       </inertial>
     </link>
-    <xacro:gazeboimu imu_name="${imu_name}"/>
+    <gazebo reference="${imu_name}_imu_link">
+      <sensor name="${imu_name}_imu_sensor" type="imu">
+        <gravity>true</gravity>
+        <always_on>true</always_on>
+        <update_rate>${update}</update_rate>
+        <visualize>true</visualize>
+        <imu>
+          <orientation_reference_frame>
+            <localization>CUSTOM</localization>
+            <custom_rpy parent_frame="${parent}">0 0 0</custom_rpy>
+            <grav_dir_x parent_frame="${parent}">1 0 0</grav_dir_x>
+          </orientation_reference_frame>
+          <angular_velocity>
+            <x>
+              <xacro:sensor_noise />
+            </x>
+            <y>
+              <xacro:sensor_noise />
+            </y>
+            <z>
+              <xacro:sensor_noise />
+            </z>
+          </angular_velocity>
+          <linear_acceleration>
+            <x>
+              <xacro:sensor_noise />
+            </x>
+            <y>
+              <xacro:sensor_noise />
+            </y>
+            <z>
+              <xacro:sensor_noise />
+            </z>
+          </linear_acceleration>
+          <enable_orientation>true</enable_orientation>
+        </imu>
+        <plugin name="${imu_name}_imu_plugin" filename="libgazebo_ros_imu_sensor.so">
+          <ros>
+            <remapping>~/out:=imu</remapping>
+          </ros>
+          <initial_orientation_as_reference>false</initial_orientation_as_reference>
+        </plugin>
+      </sensor>
+    </gazebo>
   </xacro:macro>
 </robot>

File: src/follow_me_robot/urdf/sensors/lidar.xacro (robot description, xacro)
@@ -2,12 +2,12 @@
 <robot xmlns:xacro="http://www.ros.org/wiki/xacro">
     <xacro:include filename="../core/inertial.urdf.xacro" />
-    <xacro:include filename="gazebo/lidar.gazebo" />
+    <xacro:include filename="./macros.xacro" />
     <xacro:macro name="lidar" params="parent *origin laser_name:=sensor_0 update:=30">
         <joint name="${laser_name}_laser_joint" type="fixed">
             <parent link="${parent}" />
-            <child link="${laser_name}_laser_frame" />
+            <child link="${laser_name}_laser_link" />
             <xacro:insert_block name="origin" />
         </joint>
-        <link name="${laser_name}_laser_frame">
+        <link name="${laser_name}_laser_link">
             <visual>
                 <geometry>
@@ -27,5 +27,36 @@
             </inertial>
         </link>
-        <xacro:gazebolidar laser_name="${laser_name}" update="${update}"/>
+        <gazebo reference="${laser_name}_laser_link">
+            <material>Gazebo/Red</material>
+            <sensor type="ray" name="${laser_name}_laser_sensor">
+                <pose>0 0 0 0 0 0</pose>
+                <visualize>false</visualize>
+                <always_on>true</always_on>
+                <update_rate>${update}</update_rate>
+                <ray>
+                    <scan>
+                        <horizontal>
+                            <samples>360</samples>
+                            <resolution>10</resolution>
+                            <min_angle>-3.14</min_angle>
+                            <max_angle>3.14</max_angle>
+                        </horizontal>
+                    </scan>
+                    <range>
+                        <min>0.1</min>
+                        <max>30</max>
+                        <resolution>10</resolution>
+                    </range>
+                    <xacro:sensor_noise />
+                </ray>
+                <plugin name="gazebo_ros_laser_controller_${laser_name}"
+                    filename="libgazebo_ros_ray_sensor.so">
+                    <ros>
+                        <remapping>~/out:=scan</remapping>
+                    </ros>
+                    <output_type>sensor_msgs/LaserScan</output_type>
+                </plugin>
+            </sensor>
+        </gazebo>
     </xacro:macro>
 </robot>

File: src/follow_me_robot/urdf/sensors/reciver.xacro (robot description, xacro)
@@ -3,6 +3,7 @@
     <!-- <xacro:include filename="$(find follow_me_robot)/urdf/material.xacro" /> -->
     <xacro:include filename="../core/inertial.urdf.xacro" />
-    <xacro:include filename="../core/material.xacro"/>
-    <xacro:macro name="reciver" params="reciver_name parent *origin recreciver_h=0.1 recreciver_w=0.1 recreciver_d=0.1 recreciver_m=0.1">
+    <xacro:include filename="../core/material.xacro" />
+    <xacro:macro name="reciver"
+        params="reciver_name parent *origin recreciver_h=0.1 recreciver_w=0.1 recreciver_d=0.1 recreciver_m=0.1 update:=30">
         <joint name="${reciver_name}_recover_joint">
             <parent link="${parent}" />
@@ -12,6 +13,6 @@
         <link name="${reciver_name}_reciver_link">
             <inertial>
-                <origin xyz="0.0 0.0 0.0" rpy="0.0 0.0 0.0"/>
-                <mass value="${recreciver_m}"/>
+                <origin xyz="0.0 0.0 0.0" rpy="0.0 0.0 0.0" />
+                <mass value="${recreciver_m}" />
                 <xacro:solid_cuboid_inertia
                     m="${recreciver_m}"
@@ -21,14 +22,14 @@
             </inertial>
             <visual>
-                <origin xyz="0.0 0.0 0.0" rpy="0.0 0.0 0.0"/>
+                <origin xyz="0.0 0.0 0.0" rpy="0.0 0.0 0.0" />
                 <geometry>
-                    <box size="${recreciver_w} ${recreciver_d} ${recreciver_h}"/>
+                    <box size="${recreciver_w} ${recreciver_d} ${recreciver_h}" />
                 </geometry>
-                <material name="black" />
+                <material name="red" />
             </visual>
             <collision>
-                <origin xyz="0.0 0.0 0.0" rpy="0.0 0.0 0.0"/>
+                <origin xyz="0.0 0.0 0.0" rpy="0.0 0.0 0.0" />
                 <geometry>
-                    <box size="${recreciver_w} ${recreciver_d} ${recreciver_h}"/>
+                    <box size="${recreciver_w} ${recreciver_d} ${recreciver_h}" />
                 </geometry>
             </collision>

File: src/follow_me_robot/urdf/sensors/sonar.xacro (robot description, xacro)
@@ -2,17 +2,20 @@
 <robot name="follow_me_robot"
   xmlns:xacro="http://playerstage.sourceforge.net/gazebo/xmlschema/#interface">
-  <xacro:include filename="gazebo/sonar.gazebo"/>
-  <xacro:macro name="sonar" params="side direction parent *origin">
-    <xacro:property name="sufix" value="${side}_${direction}" />
-    <joint name="${side}_${direction}_sonar_joint" type="fixed">
+  <xacro:include filename="./macros.xacro" />
+  <xacro:macro name="sonar" params="sonar_name parent *origin angel:=0.5 update:=30">
+    <joint name="${sonar_name}_sonar_joint" type="fixed">
       <xacro:insert_block name="origin" />
-      <parent link="${parent}"/>
-      <child link="${side}_${direction}_sonar_link"/>
+      <parent link="${parent}" />
+      <child link="${sonar_name}_sonar_link" />
     </joint>
-    <link name="${side}_${direction}_sonar_link">
+    <link name="${sonar_name}_sonar_link">
       <visual>
+        <!-- <geometry>
+          <mesh filename="file://$(find follow_me_robot)/urdf/meshes/max_sonar_ez4.dae" />
+        </geometry> -->
         <geometry>
-          <mesh filename="package://follow_me_robot/urdf/meshes/max_sonar_ez4.dae"/>
+          <box size="0.01 0.01 0.01" />
         </geometry>
+        <material name="red" />
       </visual>
       <collision>
@@ -26,5 +29,44 @@
       </inertial>
     </link>
-    <xacro:sonarsensor side="${side}" direction="${direction}" />
+    <gazebo reference="${sonar_name}_sonar_link">
+      <material>Gazebo/Red</material>
+      <sensor type="ray" name="${sonar_name}_sonar_sensor">
+        <xacro:property name="samples" value="1" />
+        <xacro:property name="resolution" value="1" />
+        <always_on>true</always_on>
+        <update_rate>${update}</update_rate>
+        <visualize>true</visualize>
+        <ray>
+          <scan>
+            <horizontal>
+              <samples>${samples}</samples>
+              <resolution>${resolution}</resolution>
+              <min_angle>-${angel}</min_angle>
+              <max_angle>${angel}</max_angle>
+            </horizontal>
+            <vertical>
+              <samples>${samples}</samples>
+              <resolution>${resolution}</resolution>
+              <min_angle>-${angel}</min_angle>
+              <max_angle>${angel}</max_angle>
+            </vertical>
+          </scan>
+          <range>
+            <min>0.3</min>
+            <max>10</max>
+            <resolution>0.1</resolution>
+          </range>
+          <xacro:sensor_noise />
+        </ray>
+        <plugin name="gazebo_ros_sonar_${sonar_name}" filename="libgazebo_ros_ray_sensor.so">
+          <ros>
+            <namespace>/sonar/${sonar_name}</namespace>
+            <remapping>~/out:=range</remapping>
+          </ros>
+          <output_type>sensor_msgs/Range</output_type>
+          <radiation_type>ultrasound</radiation_type>
+        </plugin>
+      </sensor>
+    </gazebo>
   </xacro:macro>
 </robot>

Commit message: add path finding

File: src/follow_me_robot/urdf/core/omni_wheel.urdf.xacro (robot description, xacro)
@@ -62,10 +62,10 @@
         <material name="black" />
       </visual>
-      <visual>
+      <!-- <visual>
         <origin xyz="0 0 0" rpy="${pi/2} 0 0" />
         <geometry>
           <mesh filename="file://$(find follow_me_robot)/urdf/meshes/omni_wheel_${wheel_img}.dae" />
         </geometry>
-      </visual>
+      </visual> -->
       <collision>
         <origin xyz="0 0 0" rpy="0 0 0" />
@@ -92,5 +92,5 @@
       </actuator>
     </transmission>
-    <gazebo reference="${prefix}_link">
+    <!-- <gazebo reference="${prefix}_link">
       <mu1 value="1.0" />
       <mu2 value="1.0" />
@@ -99,9 +99,11 @@
       <fdir1 value="1 0 0" />
       <turnGravityOff>false</turnGravityOff>
-    </gazebo>
+    </gazebo> -->
     <!-- <gazebo>
-      <plugin name="${prefix}_joint_state_publisher" filename="libgazebo_ros_joint_state_publisher.so">
+      <plugin name="${prefix}_joint_state_publisher"
+        filename="libgazebo_ros_joint_state_publisher.so">
         <update_rate>2</update_rate>
         <joint_name>${prefix}_joint</joint_name>
+        <frame_name>${parent}</frame_name>
       </plugin>
     </gazebo> -->

File: src/follow_me_robot/urdf/core/robot_body.urdf.xacro (robot description, xacro)
@@ -3,13 +3,13 @@
   <xacro:include filename="inertial.urdf.xacro" />
   <xacro:include filename="material.xacro" />
-  <xacro:macro name="robot_body" params="wheel_radius body_length body_with body_heigth">
+  <xacro:macro name="robot_body" params="parent wheel_radius body_length body_with body_heigth">
     <!-- Robot mechanical and motor parameters -->
-    <joint name="robot_body_joint" type="fixed">
-      <parent link="base_link" />
-      <child link="robot_body_link" />
+    <joint name="base_link_joint" type="fixed">
+      <parent link="${parent}" />
+      <child link="base_link" />
       <origin xyz="0 0 ${wheel_radius}" rpy="0 0 0" />
     </joint>
     <!-- BASE_LINK -->
-    <link name="robot_body_link">
+    <link name="base_link">
       <inertial>
         <mass value="125.0" />

File: src/follow_me_robot/urdf/robot.urdf.xacro (robot description, xacro)
@@ -14,12 +14,7 @@
 	<xacro:property name="wheel_radius" value="0.127" />
 	<xacro:property name="update_rate" value="30" />
+	<xacro:property name="publish_rate" value="30" />
 	<link name="base_footprint" />
-	<joint name="odom_joint" type="fixed">
-		<parent link="base_footprint" />
-		<child link="base_link" />
-		<origin xyz="0 0 0.001" />
-	</joint>
 	<!-- BASE FOOTPRINT -->
-	<link name="base_link"></link>
 	<xacro:include filename="core/material.xacro" />
 	<xacro:materials />
@@ -27,19 +22,20 @@
 	<xacro:include filename="core/robot_body.urdf.xacro" />
 	<!-- Additional params -->
-	<xacro:robot_body wheel_radius="${wheel_radius}" body_length="${body_length}"
+	<xacro:robot_body parent="base_footprint" wheel_radius="${wheel_radius}"
+		body_length="${body_length}"
 		body_with="${body_with}" body_heigth="${body_heigth}" />
-	<xacro:wheel_motor parent="robot_body_link" position="front" side="right" reflect="-1"
+	<xacro:wheel_motor parent="base_link" position="front" side="right" reflect="-1"
 		wheel_img="2" wheel_height="${wheel_height}" wheel_radius="${wheel_radius}">
 		<origin xyz="${wheel_offset_x} -${wheel_offset_y} ${wheel_offset_z}" rpy="0 0 0.0" />
 	</xacro:wheel_motor>
-	<xacro:wheel_motor parent="robot_body_link" position="front" side="left" reflect="1" wheel_img="2"
+	<xacro:wheel_motor parent="base_link" position="front" side="left" reflect="1" wheel_img="2"
 		wheel_height="${wheel_height}" wheel_radius="${wheel_radius}">
 		<origin xyz="${wheel_offset_x} ${wheel_offset_y} ${wheel_offset_z}" rpy="0 0 0" />
 	</xacro:wheel_motor>
-	<xacro:wheel_motor parent="robot_body_link" position="back" side="left" reflect="1" wheel_img="1"
+	<xacro:wheel_motor parent="base_link" position="back" side="left" reflect="1" wheel_img="1"
 		wheel_height="${wheel_height}" wheel_radius="${wheel_radius}">
 		<origin xyz="-${wheel_offset_x} ${wheel_offset_y} ${wheel_offset_z}" rpy="0 0 0" />
 	</xacro:wheel_motor>
-	<xacro:wheel_motor parent="robot_body_link" position="back" side="right" reflect="-1"
+	<xacro:wheel_motor parent="base_link" position="back" side="right" reflect="-1"
 		wheel_img="1" wheel_height="${wheel_height}" wheel_radius="${wheel_radius}">
 		<origin xyz="-${wheel_offset_x} -${wheel_offset_y} ${wheel_offset_z}" rpy="0 0 0" />
@@ -47,39 +43,44 @@
 	<gazebo>
 		<plugin name="psuedo_mecanum" filename="libgazebo_ros_planar_move.so">
-			<commandTopic>/cmd_vel</commandTopic>
-			<odometryTopic>odom</odometryTopic>
-			<odometryFrame>odom</odometryFrame>
-			<odometryRate>20.0</odometryRate>
-			<robotBaseFrame>base_link</robotBaseFrame>
-			<update_rate>${update_rate}</update_rate>
-			<publish_rate>${update_rate}</publish_rate>
+			<command_topic>/cmd_vel</command_topic>
+			<odometry_topic>/odom</odometry_topic>
+			<odometry_frame>odom</odometry_frame>
+			<robot_base_frame>base_link</robot_base_frame>
+			<ground_truth>false</ground_truth>
+			<control_mode>position</control_mode>
+			<publish_odometry>false</publish_odometry>
+			<publish_tf>false</publish_tf>
+			<publish_imu>false</publish_imu>
+			<publish_rate>0</publish_rate>
 		</plugin>
 		<plugin name="gazebo_ros_joint_state_publisher"
 			filename="libgazebo_ros_joint_state_publisher.so">
 			<update_rate>${update_rate}</update_rate>
-			<joint_name>front_right_wheel_joint</joint_name>
-			<joint_name>front_left_wheel_joint</joint_name>
-			<joint_name>back_left_wheel_joint</joint_name>
-			<joint_name>back_right_wheel_joint</joint_name>
+			<joint_names>
+				front_right_wheel_joint,front_left_wheel_joint,back_left_wheel_joint,back_right_wheel_joint
+			</joint_names>
+			<publish_selected_only>1</publish_selected_only>
 		</plugin>
 	</gazebo>
 	<xacro:include filename="sensors/lidar.xacro" />
-	<xacro:lidar parent="robot_body_link" update="${update_rate}">
+	<xacro:lidar parent="base_link" frame="base_link" update="${update_rate}">
 		<origin xyz="0 0 ${body_heigth/2+0.03}" rpy="0 0 0" />
 	</xacro:lidar>
 	<xacro:include filename="sensors/imu.xacro" />
-	<xacro:imu parent="robot_body_link" update="${update_rate}">
+	<xacro:imu parent="base_link" frame="base_link" visualize="true" update="${update_rate}">
 		<origin xyz="0 0 0" />
 	</xacro:imu>
 	<xacro:include filename="sensors/camera.xacro" />
-	<xacro:camera cam_name="front" parent="robot_body_link" update="${update_rate}" visualize="true">
+	<xacro:camera cam_name="front" parent="base_link" update="15"
+		visualize="true">
 		<origin xyz="${body_length/2} 0 0.1" rpy="0 -0.3 0" />
 	</xacro:camera>
 	<xacro:include filename="sensors/sonar.xacro" />
-	<xacro:sonar sonar_name="front_mid" parent="robot_body_link" update="${update_rate}">
+	<xacro:sonar sonar_name="front_mid" frame="base_link" parent="base_link"
+		update="${update_rate}">
 		<origin xyz="${body_length/2} 0 -0.05" rpy="0 0.2 0" />
 	</xacro:sonar>
-	<!-- <xacro:include filename="sensors/gps.xacro" />
-	<xacro:gps parent="robot_body_link" update="${update_rate}">
+	<!-- <xacro:include filename="sensors/gps.xacro" /> -->
+	<!-- <xacro:gps parent="base_link" update="${update_rate}">
 		<origin xyz="0 0 0.0" />
 	</xacro:gps> -->

File: src/follow_me_robot/urdf/sensors/camera.xacro (robot description, xacro)
@@ -57,4 +57,5 @@
           <min_depth>0.002</min_depth>
           <max_depth>300.0</max_depth>
+          <frame_name>${cam_name}_camera_link_optical</frame_name>
         </plugin>
       </sensor>

File: src/follow_me_robot/urdf/sensors/gps.xacro (robot description, xacro)
@@ -51,4 +51,5 @@
             <remapping>~/out:=gps</remapping>
           </ros>
+          <frame_name>${parent}</frame_name>
           <!-- <bodyName>${gps_name}_gps_link</bodyName>
       <frameId>${gps_name}_gps_link</frameId> -->

File: src/follow_me_robot/urdf/sensors/imu.xacro (robot description, xacro)
@@ -3,5 +3,6 @@
   xmlns:xacro="http://playerstage.sourceforge.net/gazebo/xmlschema/#interface">
   <xacro:include filename="../core/inertial.urdf.xacro" />
-  <xacro:macro name="imu" params="parent *origin imu_name:=sensor_0 update:=30">
+  <xacro:macro name="imu"
+    params="parent frame *origin imu_name:=sensor_0 update:=30 visualize:=false">
     <joint name="${imu_name}_imu_joint" type="fixed">
       <parent link="${parent}" />
@@ -32,5 +33,5 @@
         <always_on>true</always_on>
         <update_rate>${update}</update_rate>
-        <visualize>true</visualize>
+        <visualize>${visualize}</visualize>
         <imu>
           <orientation_reference_frame>
@@ -63,4 +64,5 @@
           <enable_orientation>true</enable_orientation>
         </imu>
+        <visualize>true</visualize>
         <plugin name="${imu_name}_imu_plugin" filename="libgazebo_ros_imu_sensor.so">
           <ros>
@@ -68,4 +70,5 @@
           </ros>
           <initial_orientation_as_reference>false</initial_orientation_as_reference>
+          <frame_name>${parent}</frame_name>
         </plugin>
       </sensor>

File: src/follow_me_robot/urdf/sensors/lidar.xacro (robot description, xacro)
@@ -3,5 +3,6 @@
     <xacro:include filename="../core/inertial.urdf.xacro" />
     <xacro:include filename="./macros.xacro" />
-    <xacro:macro name="lidar" params="parent *origin laser_name:=sensor_0 update:=30">
+    <xacro:macro name="lidar"
+        params="parent frame *origin laser_name:=sensor_0 update:=30 visualize:=false">
         <joint name="${laser_name}_laser_joint" type="fixed">
             <parent link="${parent}" />
@@ -34,4 +35,5 @@
                 <always_on>true</always_on>
                 <update_rate>${update}</update_rate>
+                <visualize>${visualize}</visualize>
                 <ray>
                     <scan>
@@ -56,4 +58,5 @@
                     </ros>
                     <output_type>sensor_msgs/LaserScan</output_type>
+                    <frame_name>${parent}</frame_name>
                 </plugin>
             </sensor>

File: src/follow_me_robot/urdf/sensors/macros.xacro (robot description, xacro)
@@ -2,5 +2,5 @@
 <robot name="sensor"
     xmlns:xacro="http://wiki.ros.org/xacro">
-    <xacro:macro name="sensor_noise" params="mean:=0.0 stddev:=1e-3">
+    <xacro:macro name="sensor_noise" params="mean:=0.0 stddev:=0.0">
         <noise type="gaussian">
             <type>gaussian</type>

File: src/follow_me_robot/urdf/sensors/sonar.xacro (robot description, xacro)
@@ -3,5 +3,6 @@
   xmlns:xacro="http://playerstage.sourceforge.net/gazebo/xmlschema/#interface">
   <xacro:include filename="./macros.xacro" />
-  <xacro:macro name="sonar" params="sonar_name parent *origin angel:=0.5 update:=30">
+  <xacro:macro name="sonar"
+    params="parent frame *origin sonar_name:=sonar_0 angel:=0.5 update:=30 visualize:=false">
     <joint name="${sonar_name}_sonar_joint" type="fixed">
       <xacro:insert_block name="origin" />
@@ -36,5 +37,5 @@
         <always_on>true</always_on>
         <update_rate>${update}</update_rate>
-        <visualize>true</visualize>
+        <visualize>${visualize}</visualize>
         <ray>
           <scan>
@@ -66,4 +67,5 @@
           <output_type>sensor_msgs/Range</output_type>
           <radiation_type>ultrasound</radiation_type>
+          <frame_name>${parent}</frame_name>
         </plugin>
       </sensor>
