Commit message: add STL models and rezise robot model

File: src/follow_me_robot/urdf/core/omni_wheel.urdf.xacro (robot description, xacro)
@@ -6,8 +6,8 @@
     params="parent *origin wheel_img reflect side position wheel_height wheel_radius update_rate:=20">
     <xacro:property name="prefix" value="${position}_${side}_wheel" />
-    <xacro:property name="motor_mass" value="0.1" />
-    <xacro:property name="motor_h" value="0.1" />
-    <xacro:property name="motor_d" value="0.1" />
-    <xacro:property name="motor_w" value="0.1" />
+    <xacro:property name="motor_mass" value="0.2" />
+    <xacro:property name="motor_h" value="0.04" />
+    <xacro:property name="motor_d" value="0.04" />
+    <xacro:property name="motor_w" value="0.04" />
     <xacro:property name="motor_offset" value="${motor_w/1.08 * reflect * -1}" />
     <joint name="${prefix}_motor_joint" type="fixed">
@@ -55,17 +55,17 @@
     </joint>
     <link name="${prefix}_link">
-      <visual>
+      <!-- <visual>
         <origin xyz="0 0 0" rpy="0 0 0" />
         <geometry>
           <cylinder length="${wheel_height}" radius="${wheel_radius}" />
         </geometry>
-        <material name="black" />
-      </visual>
-      <!-- <visual>
+        <material name="blue" />
+      </visual> -->
+      <visual>
         <origin xyz="0 0 0" rpy="${pi/2} 0 0" />
         <geometry>
-          <mesh filename="file://$(find follow_me_robot)/urdf/meshes/omni_wheel_${wheel_img}.dae" />
+          <mesh filename="file://$(find follow_me_robot)/urdf/meshes/omni_wheel_${wheel_img}.dae" scale="0.35 0.35 0.35" />
         </geometry>
-      </visual> -->
+      </visual>
       <collision>
         <origin xyz="0 0 0" rpy="0 0 0" />
@@ -92,9 +92,4 @@
       </actuator>
     </transmission>
-    <plugin name="wheel_state_publisher" filename="libgazebo_ros_joint_state_publisher.so">
-      <update_rate>${update_rate}</update_rate>
-      <joint_name>${prefix}_joint</joint_name>
-      <!-- <publish_selected_only>1</publish_selected_only> -->
-    </plugin>
     <gazebo reference="${prefix}_link">
       <mu1 value="1.0" />
@@ -105,12 +100,4 @@
       <turnGravityOff>true</turnGravityOff>
     </gazebo>
-    <!-- <gazebo>
-      <plugin name="${prefix}_joint_state_publisher"
-        filename="libgazebo_ros_joint_state_publisher.so">
-        <update_rate>2</update_rate>
-        <joint_name>${prefix}_joint</joint_name>
-        <frame_name>${parent}</frame_name>
-      </plugin>
-    </gazebo> -->
   </xacro:macro>
 </robot>

File: src/follow_me_robot/urdf/core/robot_body.urdf.xacro (robot description, xacro)
@@ -22,7 +22,13 @@
         <geometry>
           <box size="${body_length} ${body_with} ${body_heigth}" />
-          <!-- <box size="0.01 ${body_with} 0.01"/> -->
         </geometry>
       </visual>
+      <!-- <visual>
+        <origin xyz="0 0 0" rpy="0 0 0" />
+        <material name="orange" />
+        <geometry>
+          <mesh filename="file://$(find follow_me_robot)/urdf/meshes/EXAM_robot_2022_without_motor.STL" />
+        </geometry>
+      </visual> -->
       <collision>
         <origin xyz="0 0 0" rpy="0 0 0 " />

File: src/follow_me_robot/urdf/robot.urdf.xacro (robot description, xacro)
@@ -3,14 +3,14 @@
 	xmlns:xacro="http://www.ros.org/wiki/xacro">
 	<!-- Robot Size -->
-	<xacro:property name="body_length" value="0.80" />
-	<xacro:property name="body_with" value="0.5" />
-	<xacro:property name="body_heigth" value="0.20" />
-	<xacro:property name="wheel_height" value="0.087" />
+	<xacro:property name="body_length" value="0.36" />
+	<xacro:property name="body_with" value="0.19" />
+	<xacro:property name="body_heigth" value="0.06" />
+	<xacro:property name="wheel_height" value="0.04" />
 	<!-- Wheel parameters -->
-	<xacro:property name="wheel_offset_x" value="0.25" />
+	<xacro:property name="wheel_offset_x" value="0.11" />
 	<!-- x,y,z in translation from base_link to the center of the wheel -->
-	<xacro:property name="wheel_offset_y" value="${(body_with/2)+0.051}" />
-	<xacro:property name="wheel_offset_z" value="0.0" />
-	<xacro:property name="wheel_radius" value="0.127" />
+	<xacro:property name="wheel_offset_y" value="${(body_with/2)}" />
+	<xacro:property name="wheel_offset_z" value="-0.01" />
+	<xacro:property name="wheel_radius" value="0.045" />
 	<xacro:property name="update_rate" value="30" />
 	<xacro:property name="publish_rate" value="30" />
@@ -64,6 +64,6 @@
 	</gazebo>
 	<xacro:include filename="sensors/lidar.xacro" />
-	<xacro:lidar parent="base_link" frame="base_link" update="${update_rate}">
-		<origin xyz="0 0 ${body_heigth/2+0.03}" rpy="0 0 0" />
+	<xacro:lidar parent="base_link" frame="base_link" update="${update_rate}" visualize="true">
+		<origin xyz="0 0 ${body_heigth/2+0.05}" rpy="0 0 0" />
 	</xacro:lidar>
 	<xacro:include filename="sensors/imu.xacro" />
@@ -73,11 +73,11 @@
 	<xacro:include filename="sensors/camera.xacro" />
 	<xacro:camera cam_name="front" parent="base_link" update="15"
-		visualize="true">
-		<origin xyz="${body_length/2} 0 0.1" rpy="0 -0.35 0" />
+		visualize="false">
+		<origin xyz="${body_length/2} 0 0.05" rpy="0 -0.35 0" />
 	</xacro:camera>
-	<xacro:include filename="sensors/sonar.xacro" />
+	<!-- <xacro:include filename="sensors/sonar.xacro" />
 	<xacro:sonar sonar_name="front_mid" frame="base_link" parent="base_link"
 		update="${update_rate}">
 		<origin xyz="${body_length/2} 0 -0.05" rpy="0 0.2 0" />
-	</xacro:sonar>
+	</xacro:sonar> -->
 </robot>

File: src/follow_me_robot/urdf/sensors/camera.xacro (robot description, xacro)
@@ -11,5 +11,5 @@
       <visual>
         <geometry>
-          <box size="0.01 0.03 0.06" />
+          <box size="0.01 0.06 0.03" />
         </geometry>
         <material name="blue" />
@@ -31,4 +31,5 @@
     </link>
     <gazebo reference="${cam_name}_camera_link_optical">
+      <material>Gazebo/Red</material>
       <sensor type="camera" name="${cam_name}_cam">
         <always_on>true</always_on>

Commit message: use resize stl model

File: src/follow_me_robot/urdf/core/omni_wheel.urdf.xacro (robot description, xacro)
@@ -2,13 +2,15 @@
 <robot name="wheel" xmlns:xacro="http://www.ros.org/wiki/xacro">
   <xacro:include filename="inertial.urdf.xacro" />
-  <!-- Motro -->
+  <!-- Motro Macro -->
   <xacro:macro name="wheel_motor"
     params="parent *origin wheel_img reflect side position wheel_height wheel_radius update_rate:=20">
     <xacro:property name="prefix" value="${position}_${side}_wheel" />
+    <!-- Motor parameters -->
     <xacro:property name="motor_mass" value="0.2" />
-    <xacro:property name="motor_h" value="0.04" />
+    <xacro:property name="motor_h" value="0.06" />
     <xacro:property name="motor_d" value="0.04" />
     <xacro:property name="motor_w" value="0.04" />
     <xacro:property name="motor_offset" value="${motor_w/1.08 * reflect * -1}" />
+    <!-- Motor to Parent Joint -->
     <joint name="${prefix}_motor_joint" type="fixed">
       <parent link="${parent}" />
@@ -16,5 +18,7 @@
       <xacro:insert_block name="origin" />
     </joint>
+    <!-- Motor Link (Visual, Collision, Inertial) -->
     <link name="${prefix}_motor_link">
+      <!-- Visual -->
       <visual>
         <origin xyz="0 ${motor_offset} 0" rpy="0 0 0" />
@@ -24,4 +28,5 @@
         <material name="darkgrey" />
       </visual>
+      <!-- Collision -->
       <collision>
         <origin xyz="0 ${motor_offset} 0" rpy="0 0 0" />
@@ -30,4 +35,5 @@
         </geometry>
       </collision>
+      <!-- Inertial -->
       <inertial>
         <mass value="${motor_mass}" />
@@ -35,4 +41,5 @@
       </inertial>
     </link>
+    <!-- Motor to Wheel -->
     <xacro:omni_wheel parent="${prefix}_motor_link" wheel_img="${wheel_img}" side="${side}"
       position="${position}" wheel_height="${wheel_height}" wheel_radius="${wheel_radius}"
@@ -41,5 +48,5 @@
     </xacro:omni_wheel>
   </xacro:macro>
-  <!-- Wheel -->
+  <!-- Wheel Macro -->
   <xacro:macro name="omni_wheel"
     params="parent *origin wheel_img side position wheel_height wheel_radius update_rate:=20">
@@ -47,4 +54,5 @@
     <xacro:property name="wheel_mass" value="6.5" />
     <xacro:property name="prefix" value="${position}_${side}_wheel" />
+    <!-- Wheek to Parent Joint -->
     <joint name="${prefix}_joint" type="continuous">
       <parent link="${parent}" />
@@ -54,5 +62,7 @@
       <joint_properties damping="0.0" friction="1.0" />
     </joint>
+    <!-- Wheel Link (Visual, Collision, Inertial) -->
     <link name="${prefix}_link">
+      <!-- Simple visual (use in windows foxglove) -->
       <!-- <visual>
         <origin xyz="0 0 0" rpy="0 0 0" />
@@ -62,4 +72,5 @@
         <material name="blue" />
       </visual> -->
+      <!-- Complex visual -->
       <visual>
         <origin xyz="0 0 0" rpy="${pi/2} 0 0" />
@@ -68,4 +79,5 @@
         </geometry>
       </visual>
+      <!-- Collision -->
       <collision>
         <origin xyz="0 0 0" rpy="0 0 0" />
@@ -74,4 +86,5 @@
         </geometry>
       </collision>
+      <!-- Inertial -->
       <inertial>
         <mass value="${wheel_mass}" />
@@ -79,11 +92,11 @@
       </inertial>
     </link>
-    <!-- Transmission is important to link the joints and the controller (see
-    robot_control/config/robot_control.yaml)-->
+    <!-- Transmission is important to link the joints and the controller (see robot_control/config/robot_control.yaml) -->
     <transmission name="${prefix}_joint_trans" type="transmission_interface/SimpleTransmission">
       <type>transmission_interface/SimpleTransmission</type>
       <joint name="${prefix}_joint">
-        <!-- <hardwareInterface>hardware_interface/VelocityJointInterface</hardwareInterface> -->
-        <hardwareInterface>EffortJointInterface</hardwareInterface>
+        <hardwareInterface>hardware_interface/VelocityJointInterface</hardwareInterface>
+        <!-- <hardwareInterface>VelocityJointInterface</hardwareInterface> -->
+        <!-- <hardwareInterface>EffortJointInterface</hardwareInterface> -->
       </joint>
       <actuator name="${prefix}_motor">

File: src/follow_me_robot/urdf/core/robot_body.urdf.xacro (robot description, xacro)
@@ -10,12 +10,8 @@
       <origin xyz="0 0 ${wheel_radius}" rpy="0 0 0" />
     </joint>
-    <!-- BASE_LINK -->
+    <!-- BASE_LINK (used by movement) -->
     <link name="base_link">
-      <inertial>
-        <mass value="125.0" />
-        <origin xyz="0 0 0" />
-        <xacro:solid_cuboid_inertia m="125.0" h="${body_with}" d="${body_heigth}" w="${body_length}" />
-      </inertial>
-      <visual>
+      <!-- Simple visual (use in windows foxglove) -->
+      <!-- <visual>
         <origin xyz="0 0 0" rpy="0 0 0" />
         <material name="orange" />
@@ -23,12 +19,14 @@
           <box size="${body_length} ${body_with} ${body_heigth}" />
         </geometry>
-      </visual>
-      <!-- <visual>
+      </visual> -->
+      <!-- Complex visual -->
+      <visual>
         <origin xyz="0 0 0" rpy="0 0 0" />
         <material name="orange" />
         <geometry>
-          <mesh filename="file://$(find follow_me_robot)/urdf/meshes/EXAM_robot_2022_without_motor.STL" />
+          <mesh filename="file://$(find follow_me_robot)/urdf/meshes/EXAM_robot_2022.stl" />
         </geometry>
-      </visual> -->
+      </visual>
+      <!-- Collision -->
       <collision>
         <origin xyz="0 0 0" rpy="0 0 0 " />
@@ -37,4 +35,10 @@
         </geometry>
       </collision>
+      <!-- Inertial -->
+      <inertial>
+        <mass value="125.0" />
+        <origin xyz="0 0 0" />
+        <xacro:solid_cuboid_inertia m="125.0" h="${body_with}" d="${body_heigth}" w="${body_length}" />
+      </inertial>
     </link>
   </xacro:macro>

File: src/follow_me_robot/urdf/robot.urdf.xacro (robot description, xacro)
@@ -8,5 +8,5 @@
 	<xacro:property name="wheel_height" value="0.04" />
 	<!-- Wheel parameters -->
-	<xacro:property name="wheel_offset_x" value="0.11" />
+	<xacro:property name="wheel_offset_x" value="0.095" />
 	<!-- x,y,z in translation from base_link to the center of the wheel -->
 	<xacro:property name="wheel_offset_y" value="${(body_with/2)}" />
@@ -15,31 +15,59 @@
 	<xacro:property name="update_rate" value="30" />
 	<xacro:property name="publish_rate" value="30" />
-	<link name="base_footprint" />
-	<!-- BASE FOOTPRINT -->
+	<!-- Includes -->
 	<xacro:include filename="core/material.xacro" />
 	<xacro:materials />
 	<xacro:include filename="core/omni_wheel.urdf.xacro" />
 	<xacro:include filename="core/robot_body.urdf.xacro" />
-	<!-- Additional params -->
+	<!-- BASE FOOTPRINT -->
+	<link name="base_footprint" />
+	<!-- Robot Body -->
 	<xacro:robot_body parent="base_footprint" wheel_radius="${wheel_radius}"
 		body_length="${body_length}"
 		body_with="${body_with}" body_heigth="${body_heigth}" />
+	<!-- Wheel Front Right -->
 	<xacro:wheel_motor parent="base_link" position="front" side="right" reflect="-1"
 		wheel_img="2" wheel_height="${wheel_height}" wheel_radius="${wheel_radius}">
 		<origin xyz="${wheel_offset_x} -${wheel_offset_y} ${wheel_offset_z}" rpy="0 0 0.0" />
 	</xacro:wheel_motor>
+	<!-- Wheel Front Left -->
 	<xacro:wheel_motor parent="base_link" position="front" side="left" reflect="1" wheel_img="2"
 		wheel_height="${wheel_height}" wheel_radius="${wheel_radius}">
 		<origin xyz="${wheel_offset_x} ${wheel_offset_y} ${wheel_offset_z}" rpy="0 0 0" />
 	</xacro:wheel_motor>
+	<!-- Wheel Back Left -->
 	<xacro:wheel_motor parent="base_link" position="back" side="left" reflect="1" wheel_img="1"
 		wheel_height="${wheel_height}" wheel_radius="${wheel_radius}">
 		<origin xyz="-${wheel_offset_x} ${wheel_offset_y} ${wheel_offset_z}" rpy="0 0 0" />
 	</xacro:wheel_motor>
+	<!-- Wheel Back Right -->
 	<xacro:wheel_motor parent="base_link" position="back" side="right" reflect="-1"
 		wheel_img="1" wheel_height="${wheel_height}" wheel_radius="${wheel_radius}">
 		<origin xyz="-${wheel_offset_x} -${wheel_offset_y} ${wheel_offset_z}" rpy="0 0 0" />
 	</xacro:wheel_motor>
+	<!-- Lidar Sensor -->
+	<xacro:include filename="sensors/lidar.xacro" />
+	<xacro:lidar parent="base_link" frame="base_link" update="${update_rate}" visualize="true">
+		<origin xyz="0 0 ${body_heigth/2+0.05}" rpy="0 0 0" />
+	</xacro:lidar>
+	<!-- IMU Sensor -->
+	<xacro:include filename="sensors/imu.xacro" />
+	<xacro:imu parent="base_link" frame="base_link" visualize="true" update="${update_rate}">
+		<origin xyz="0 0 0" />
+	</xacro:imu>
+	<!-- Camera Sensor -->
+	<xacro:include filename="sensors/camera.xacro" />
+	<xacro:camera cam_name="front" parent="base_link" update="15"
+		visualize="false">
+		<origin xyz="${body_length/2} -0.0252 -0.005" rpy="0 -0.35 0" />
+	</xacro:camera>
+	<!-- <xacro:include filename="sensors/sonar.xacro" />
+	<xacro:sonar sonar_name="front_mid" frame="base_link" parent="base_link"
+		update="${update_rate}">
+		<origin xyz="${body_length/2} 0 -0.05" rpy="0 0.2 0" />
+	</xacro:sonar> -->
+	<!-- Gazebo Plugins -->
 	<gazebo>
+		<!-- Plugin for the robot's movement -->
 		<plugin name="psuedo_mecanum" filename="libgazebo_ros_planar_move.so">
 			<command_topic>/cmd_vel</command_topic>
@@ -54,4 +82,5 @@
 			<publish_rate>0</publish_rate>
 		</plugin>
+		<!-- Plugin for the robot's joint state -->
 		<plugin name="gazebo_ros_joint_state_publisher"
 			filename="libgazebo_ros_joint_state_publisher.so">
@@ -63,21 +92,3 @@
 		</plugin>
 	</gazebo>
-	<xacro:include filename="sensors/lidar.xacro" />
-	<xacro:lidar parent="base_link" frame="base_link" update="${update_rate}" visualize="true">
-		<origin xyz="0 0 ${body_heigth/2+0.05}" rpy="0 0 0" />
-	</xacro:lidar>
-	<xacro:include filename="sensors/imu.xacro" />
-	<xacro:imu parent="base_link" frame="base_link" visualize="true" update="${update_rate}">
-		<origin xyz="0 0 0" />
-	</xacro:imu>
-	<xacro:include filename="sensors/camera.xacro" />
-	<xacro:camera cam_name="front" parent="base_link" update="15"
-		visualize="false">
-		<origin xyz="${body_length/2} 0 0.05" rpy="0 -0.35 0" />
-	</xacro:camera>
-	<!-- <xacro:include filename="sensors/sonar.xacro" />
-	<xacro:sonar sonar_name="front_mid" frame="base_link" parent="base_link"
-		update="${update_rate}">
-		<origin xyz="${body_length/2} 0 -0.05" rpy="0 0.2 0" />
-	</xacro:sonar> -->
 </robot>

File: src/follow_me_robot/urdf/sensors/camera.xacro (robot description, xacro)
@@ -15,11 +15,4 @@
         <material name="blue" />
       </visual>
-      <visual>
-        <origin xyz="0.005 0 0" rpy="0 ${pi/2} 0" />
-        <geometry>
-          <cylinder radius="0.01" length="0.01" />
-        </geometry>
-        <material name="red" />
-      </visual>
     </link>
     <joint name="${cam_name}_camera_link_optical_joint" type="fixed">
@@ -29,4 +22,11 @@
     </joint>
     <link name="${cam_name}_camera_link_optical">
+      <visual>
+        <origin xyz="0.005 0 0" rpy="0 0 0" />
+        <geometry>
+          <cylinder radius="0.02" length="0.02" />
+          <material name="red" />
+        </geometry>
+      </visual>
     </link>
     <gazebo reference="${cam_name}_camera_link_optical">

File: src/follow_me_robot/urdf/sensors/imu.xacro (robot description, xacro)
@@ -5,4 +5,5 @@
   <xacro:macro name="imu"
     params="parent frame *origin imu_name:=sensor_0 update:=30 visualize:=false">
+    <xacro:property name="box_size" value="0.01" />
     <joint name="${imu_name}_imu_joint" type="fixed">
       <parent link="${parent}" />
@@ -13,5 +14,5 @@
       <visual>
         <geometry>
-          <box size="0.05 0.05 0.05" />
+          <box size="${box_size} ${box_size} ${box_size}" />
         </geometry>
         <material name="red" />
@@ -19,5 +20,5 @@
       <collision>
         <geometry>
-          <box size="0.05 0.05 0.05" />
+          <box size="${box_size} ${box_size} ${box_size}" />
         </geometry>
       </collision>
@@ -25,8 +26,9 @@
         <mass value="1e-5" />
         <origin xyz="0 0 0" rpy="0 0 0" />
-        <xacro:solid_cuboid_inertia w="0.05" h="0.05" d="0.5" m="1e-5" />
+        <xacro:solid_cuboid_inertia w="${box_size}" h="${box_size}" d="${box_size}" m="1e-5" />
       </inertial>
     </link>
     <gazebo reference="${imu_name}_imu_link">
+      <material>Gazebo/Red</material>
       <sensor name="${imu_name}_imu_sensor" type="imu">
         <parent link="${imu_name}_imu_link" />
