Commit message: fixed some more warnings

File: src/follow_me_robot/urdf/core/robot_body.urdf.xacro (robot description, xacro)
@@ -14,7 +14,7 @@
 		</link>
 		<joint name="robot_footprint_joint" type="fixed">
-		  <origin xyz="0 0 ${wheel_radius}" rpy="0 0 0" /> <!-- ${wheel_radius} property must be defined inside wheel description -->
 		  <parent link="robot_footprint"/>
 		  <child link="robot_body_link" />
+      <origin xyz="0 0 ${wheel_radius}" rpy="0 0 0" />
 		</joint>
   <!-- BASE_LINK -->

File: src/follow_me_robot/urdf/sensors/camera.xacro (robot description, xacro)
@@ -48,5 +48,5 @@
                 <frame_name>camera_link_optical</frame_name>
                 <ros>
-                    <argument>~/out:=range</argument>
+                    <argument>--ros-args --remap ~/out:=range</argument>
                 </ros>
                 <output_type>sensor_msgs/Range</output_type>

File: src/follow_me_robot/urdf/sensors/lidar.xacro (robot description, xacro)
@@ -48,5 +48,5 @@
                 <plugin name="laser_controller" filename="libgazebo_ros_ray_sensor.so">
                     <ros>
-                        <argument>~/out:=scan</argument>
+                        <argument>--ros-args --remap ~/out:=scan</argument>
                     </ros>
                     <output_type>sensor_msgs/LaserScan</output_type>

Commit message: [WIP] refactor scripts

File: src/follow_me_robot/urdf/core/robot_body.urdf.xacro (robot description, xacro)
@@ -7,5 +7,5 @@
   <!-- Robot mechanical and motor parameters -->
   <joint name="robot_body_joint" type="fixed">
-		<parent link="base_footprint"/>
+		<parent link="base_link"/>
 		<child link="robot_body_link" />
 		<origin xyz="0 0 ${wheel_radius}" rpy="0 0 0" />

File: src/follow_me_robot/urdf/robot.urdf.xacro (robot description, xacro)
@@ -10,18 +10,16 @@
 	<xacro:property name="wheel_offset_x" value="0.25" />
 	<!-- x,y,z in translation from base_link to the center of the wheel -->
-	<xacro:property name="wheel_offset_y" value="${(body_with/2+0.051)}" />
+	<xacro:property name="wheel_offset_y" value="${(body_with/2)+0.051}" />
 	<xacro:property name="wheel_offset_z" value="0.0" />
 	<xacro:property name="wheel_radius" value="0.127" />
 	<xacro:property name="update_rate" value="20" />
+	<link name="base_footprint"/>
+	<joint name="odom_joint" type="fixed">
+    <parent link="base_footprint"/>
+    <child link="base_link" />
+		<origin xyz="0 0 0.001" />
+  </joint>
 	<!-- BASE FOOTPRINT -->
-	<link name="base_footprint">
-		<must_be_base_link>true</must_be_base_link>
-		<visual>
-			<origin xyz="0 0 0" rpy="0 0 0" />
-			<geometry>
-				<box size="0.001 0.001 0.001" />
-			</geometry>
-		</visual>
-	</link>
+	<link name="base_link"></link>
 	<xacro:include filename="core/material.xacro" />
 	<xacro:materials />
@@ -45,8 +43,8 @@
 	<xacro:omni_steering />
 	<gazebo>
-		<plugin name="gazebo_ros_joint_pose_trajectory"
+		<!-- <plugin name="gazebo_ros_joint_pose_trajectory"
 			filename="libgazebo_ros_joint_pose_trajectory.so">
 			<update_rate>2</update_rate>
-		</plugin>
+		</plugin>	 -->
 		<plugin name="gazebo_ros_joint_state_publisher" filename="libgazebo_ros_joint_state_publisher.so">
 		<update_rate>100</update_rate>
@@ -58,11 +56,11 @@
 	</gazebo>
 	<xacro:include filename="sensors/lidar.xacro" />
-	<xacro:lidar parent="robot_body_link">
+	<xacro:lidar parent="robot_body_link" update="10">
 		<origin xyz="0 0 ${body_heigth/2+0.03}" rpy="0 0 0" />
 	</xacro:lidar>
-	<xacro:include filename="sensors/gps.xacro" />
+	<!-- <xacro:include filename="sensors/gps.xacro" />
 	<xacro:gps parent="robot_body_link">
 		<origin xyz="0 0 0.0"/>
-	</xacro:gps>
+	</xacro:gps> -->
 	<xacro:include filename="sensors/imu.xacro" />
 	<xacro:imu parent="robot_body_link">

Commit message: add robot mock to follow

File: src/follow_me_robot/urdf/core/robot_body.urdf.xacro (robot description, xacro)
@@ -23,5 +23,4 @@
       <visual>
         <origin xyz="0 0 0" rpy="0 0 0" />
-        <material name="orange" />
         <geometry>
           <mesh filename="file://$(find follow_me_robot)/urdf/meshes/EXAM_robot_2022.stl" />

File: src/follow_me_robot/urdf/robot.urdf.xacro (robot description, xacro)
@@ -48,10 +48,17 @@
 	<!-- Lidar Sensor -->
 	<xacro:include filename="sensors/lidar.xacro" />
-	<xacro:lidar parent="base_link" frame="base_link" update="${update_rate}" visualize="true">
+	<xacro:lidar
+		parent="base_link"
+		frame="base_link"
+	 	update="${update_rate}"
+		visualize="false"
+		max_range="20"
+		resolution="10"
+		>
 		<origin xyz="0 0 ${body_heigth/2+0.05}" rpy="0 0 0" />
 	</xacro:lidar>
 	<!-- IMU Sensor -->
 	<xacro:include filename="sensors/imu.xacro" />
-	<xacro:imu parent="base_link" frame="base_link" visualize="true" update="${update_rate}">
+	<xacro:imu parent="base_link" frame="base_link" visualize="false" update="${update_rate}">
 		<origin xyz="0 0 0" />
 	</xacro:imu>

File: src/follow_me_robot/urdf/sensors/lidar.xacro (robot description, xacro)
@@ -4,10 +4,17 @@
     <xacro:include filename="./macros.xacro" />
     <xacro:macro name="lidar"
-        params="parent frame *origin laser_name:=sensor_0 update:=30 visualize:=false min_range:=0.1 max_range:=30">
+        params="parent frame *origin laser_name:=sensor_0 update:=30 visualize:=false min_range:=0.1 max_range:=30 resolution:=10">
         <joint name="${laser_name}_laser_joint" type="fixed">
             <parent link="${parent}" />
             <child link="${laser_name}_laser_link" />
             <xacro:insert_block name="origin" />
+            <joint_properties damping="1.0" friction="1.0" />
         </joint>
+        <gazebo reference="${laser_name}_laser_joint">
+            <preserveFixedJoint>true</preserveFixedJoint>
+        </gazebo>
+        <gazebo reference="${laser_name}_laser_joint">
+            <material>Gazebo/DarkGrey</material>
+        </gazebo>
         <link name="${laser_name}_laser_link">
             <visual>
@@ -33,5 +40,4 @@
                 <parent link="${laser_name}_laser_link" />
                 <pose>0 0 0 0 0 0</pose>
-                <visualize>false</visualize>
                 <always_on>true</always_on>
                 <update_rate>${update}</update_rate>
@@ -41,5 +47,5 @@
                         <horizontal>
                             <samples>360</samples>
-                            <resolution>10</resolution>
+                            <resolution>${resolution}</resolution>
                             <min_angle>-3.14</min_angle>
                             <max_angle>3.14</max_angle>
@@ -49,5 +55,5 @@
                         <min>${min_range}</min>
                         <max>${max_range}</max>
-                        <resolution>10</resolution>
+                        <resolution>${resolution}</resolution>
                     </range>
                     <xacro:sensor_noise />
