Commit message: setup simulation

File: src/follow_me_robot/urdf/sensors/gazebo/macros.xacro (robot description, xacro)
@@ -9,3 +9,6 @@
         </noise>
     </xacro:macro>
+    <xacro:macro name="sensor_topic_ns" params="type name">
+        <namespace>/sensor/${type}/${name}</namespace>
+    </xacro:macro>
 </robot>
