Commit message: cleanup code

File: src/follow_me_robot/urdf/sensors/gps.xacro (robot description, xacro)
@@ -35,4 +35,5 @@
     <gazebo reference="${gps_name}_gps_link">
       <sensor name="${gps_name}_gps" type="gps">
+        <parent link="${gps_name}_gps_link" />
         <always_on>true</always_on>
         <update_rate>${update}</update_rate>

File: src/follow_me_robot/urdf/sensors/imu.xacro (robot description, xacro)
@@ -30,4 +30,5 @@
     <gazebo reference="${imu_name}_imu_link">
       <sensor name="${imu_name}_imu_sensor" type="imu">
+        <parent link="${imu_name}_imu_link" />
         <gravity>true</gravity>
         <always_on>true</always_on>

File: src/follow_me_robot/urdf/sensors/lidar.xacro (robot description, xacro)
@@ -4,5 +4,5 @@
     <xacro:include filename="./macros.xacro" />
     <xacro:macro name="lidar"
-        params="parent frame *origin laser_name:=sensor_0 update:=30 visualize:=false">
+        params="parent frame *origin laser_name:=sensor_0 update:=30 visualize:=false min_range:=0.1 max_range:=30">
         <joint name="${laser_name}_laser_joint" type="fixed">
             <parent link="${parent}" />
@@ -31,4 +31,5 @@
             <material>Gazebo/Red</material>
             <sensor type="ray" name="${laser_name}_laser_sensor">
+                <parent link="${laser_name}_laser_link" />
                 <pose>0 0 0 0 0 0</pose>
                 <visualize>false</visualize>
@@ -46,6 +47,6 @@
                     </scan>
                     <range>
-                        <min>0.1</min>
-                        <max>30</max>
+                        <min>${min_range}</min>
+                        <max>${max_range}</max>
                         <resolution>10</resolution>
                     </range>

File: src/follow_me_robot/urdf/sensors/sonar.xacro (robot description, xacro)
@@ -4,5 +4,5 @@
   <xacro:include filename="./macros.xacro" />
   <xacro:macro name="sonar"
-    params="parent frame *origin sonar_name:=sonar_0 angel:=0.5 update:=30 visualize:=false">
+    params="parent frame *origin sonar_name:=sonar_0 angel:=0.5 update:=30 visualize:=false min_range:=0.1 max_range:=30">
     <joint name="${sonar_name}_sonar_joint" type="fixed">
       <xacro:insert_block name="origin" />
@@ -54,6 +54,6 @@
           </scan>
           <range>
-            <min>0.3</min>
-            <max>10</max>
+            <min>${min_range}</min>
+            <max>${max_range}</max>
             <resolution>0.1</resolution>
           </range>
