Commit message: fix camera rotation

File: src/follow_me_robot/urdf/sensors/camera.xacro (robot description, xacro)
@@ -9,11 +9,4 @@
     </joint>
     <link name="${cam_name}_camera_link">
-    </link>
-    <joint name="${cam_name}_camera_link_optical_joint" type="fixed">
-      <parent link="${cam_name}_camera_link" />
-      <child link="${cam_name}_camera_link_optical" />
-      <origin xyz="0 0 0" rpy="${pi/2} 0 ${pi/2}" />
-    </joint>
-    <link name="${cam_name}_camera_link_optical">
       <visual>
         <geometry>
@@ -30,5 +23,5 @@
       </visual>
     </link>
-    <gazebo reference="${cam_name}_camera_link_optical">
+    <gazebo reference="${cam_name}_camera_link">
       <sensor type="camera" name="${cam_name}_cam">
         <always_on>true</always_on>
@@ -36,6 +29,4 @@
         <visualize>${visualize}</visualize>
         <camera name="${cam_name}_head">
-          <pose>0.0
-            0 0.0 ${pi/2} -${pi/2} 0</pose>
           <horizontal_fov>${70 * pi/180.0}</horizontal_fov>
           <image>
@@ -60,5 +51,5 @@
           <min_depth>0.002</min_depth>
           <max_depth>300.0</max_depth>
-          <frame_name>${cam_name}_camera_link_optical</frame_name>
+          <frame_name>${cam_name}_camera_link</frame_name>
         </plugin>
       </sensor>

Commit message: rotate camera in sim

File: src/follow_me_robot/urdf/sensors/camera.xacro (robot description, xacro)
@@ -8,13 +8,13 @@
       <xacro:insert_block name="origin" />
     </joint>
-    <link name="${cam_name}_camera_link">
+    <link name="${cam_name}_camera_link" >
       <visual>
         <geometry>
-          <box size="0.06 0.03 0.010" />
+          <box size="0.01 0.03 0.06" />
         </geometry>
         <material name="blue" />
       </visual>
       <visual>
-        <origin xyz="0 0 0.005" rpy="0 0 0" />
+        <origin xyz="0.005 0 0" rpy="0 ${pi/2} 0" />
         <geometry>
           <cylinder radius="0.01" length="0.01" />
@@ -23,5 +23,12 @@
       </visual>
     </link>
-    <gazebo reference="${cam_name}_camera_link">
+    <joint name="${cam_name}_camera_link_optical_joint" type="fixed">
+      <parent link="${cam_name}_camera_link" />
+      <child link="${cam_name}_camera_link_optical" />
+      <origin xyz="0 0 0" rpy="${pi/2} 0 ${pi/2}" />
+    </joint>
+    <link name="${cam_name}_camera_link_optical">
+    </link>
+    <gazebo reference="${cam_name}_camera_link_optical">
       <sensor type="camera" name="${cam_name}_cam">
         <always_on>true</always_on>
@@ -29,4 +36,5 @@
         <visualize>${visualize}</visualize>
         <camera name="${cam_name}_head">
+          <pose>0.0 0 0.0 ${pi/2} -${pi/2} 0</pose>
           <horizontal_fov>${70 * pi/180.0}</horizontal_fov>
           <image>
@@ -51,5 +59,5 @@
           <min_depth>0.002</min_depth>
           <max_depth>300.0</max_depth>
-          <frame_name>${cam_name}_camera_link</frame_name>
+          <frame_name>${cam_name}_camera_link_optical</frame_name>
         </plugin>
       </sensor>

Commit message: add comments to the code

File: src/follow_me_robot/urdf/sensors/camera.xacro (robot description, xacro)
@@ -9,10 +9,10 @@
     </joint>
     <link name="${cam_name}_camera_link" >
-      <visual>
+      <!-- <visual>
         <geometry>
           <box size="0.01 0.06 0.03" />
         </geometry>
         <material name="blue" />
-      </visual>
+      </visual> -->
     </link>
     <joint name="${cam_name}_camera_link_optical_joint" type="fixed">
