Commit message: fixed console error with lidar

File: src/follow_me_robot/urdf/robot.urdf.xacro (robot description, xacro)
@@ -28,5 +28,5 @@
 			<origin xyz="-${wheel_offset_x} -${wheel_offset_y} ${wheel_offset_z}" rpy="0 0 0" />
 		</xacro:omni_wheel>
-		<xacro:lidar parent="robot_body_link" laser_name="1" range="10">
+		<xacro:lidar parent="robot_body_link" laser_name="1">
 			<origin xyz="0 0 0.3" rpy="0 0 0" />
 		</xacro:lidar>

File: src/follow_me_robot/urdf/sensors/lidar.xacro (robot description, xacro)
@@ -3,5 +3,5 @@
     <xacro:include filename="$(find follow_me_robot)/urdf/core/inertial.urdf.xacro" />
     <xacro:include filename="$(find follow_me_robot)/urdf/core/material.xacro" />
-    <xacro:macro name="lidar" params="parent *origin laser_name range:=12">
+    <xacro:macro name="lidar" params="parent *origin laser_name">
         <joint name="${laser_name}_laser_joint" type="fixed">
             <parent link="${parent}" />
@@ -43,5 +43,5 @@
                     <range>
                         <min>0.3</min>
-                        <max>${range}</max>
+                        <max>10.0</max>
                     </range>
                 </ray>

Commit message: add tag to goal node

File: src/follow_me_robot/urdf/robot.urdf.xacro (robot description, xacro)
@@ -57,8 +57,9 @@
 			filename="libgazebo_ros_joint_state_publisher.so">
 			<update_rate>${update_rate}</update_rate>
-			<joint_names>
-				front_right_wheel_joint,front_left_wheel_joint,back_left_wheel_joint,back_right_wheel_joint
-			</joint_names>
-			<publish_selected_only>1</publish_selected_only>
+			<joint_name>front_right_wheel_joint</joint_name>
+			<joint_name>front_left_wheel_joint</joint_name>
+			<joint_name>back_left_wheel_joint</joint_name>
+			<joint_name>back_right_wheel_joint</joint_name>
+			<!-- <publish_selected_only>1</publish_selected_only> -->
 		</plugin>
 	</gazebo>
@@ -74,5 +75,7 @@
 	<xacro:camera cam_name="front" parent="base_link" update="15"
 		visualize="true">
+		<!-- <origin xyz="${body_length/2} 0 0.1" rpy="${pi/2} 0 ${pi/2}" /> -->
 		<origin xyz="${body_length/2} 0 0.1" rpy="0 -0.3 0" />
+		<!-- <origin xyz="${body_length/2} 0 0.1" rpy="0 -0.3 ${pi/2}" /> -->
 	</xacro:camera>
 	<xacro:include filename="sensors/sonar.xacro" />

File: src/follow_me_robot/urdf/sensors/camera.xacro (robot description, xacro)
@@ -9,12 +9,19 @@
     </joint>
     <link name="${cam_name}_camera_link">
+    </link>
+    <joint name="${cam_name}_camera_link_optical_joint" type="fixed">
+      <parent link="${cam_name}_camera_link" />
+      <child link="${cam_name}_camera_link_optical" />
+      <origin xyz="0 0 0" rpy="${pi/2} 0 ${pi/2}" />
+    </joint>
+    <link name="${cam_name}_camera_link_optical">
       <visual>
         <geometry>
-          <box size="0.010 0.03 0.03" />
+          <box size="0.06 0.03 0.010" />
         </geometry>
         <material name="blue" />
       </visual>
       <visual>
-        <origin xyz="0.005 0 0" rpy="0 ${pi/2} 0" />
+        <origin xyz="0 0 0.005" rpy="0 0 0" />
         <geometry>
           <cylinder radius="0.01" length="0.01" />
@@ -23,10 +30,4 @@
       </visual>
     </link>
-    <joint name="${cam_name}_camera_optical_joint" type="fixed">
-      <parent link="${cam_name}_camera_link" />
-      <child link="${cam_name}_camera_link_optical" />
-      <origin xyz="0.01 0 0" rpy="0 0 0" />
-    </joint>
-    <link name="${cam_name}_camera_link_optical" />
     <gazebo reference="${cam_name}_camera_link_optical">
       <sensor type="camera" name="${cam_name}_cam">
@@ -35,5 +36,7 @@
         <visualize>${visualize}</visualize>
         <camera name="${cam_name}_head">
-          <horizontal_fov>1.3962634</horizontal_fov>
+          <pose>0.0
+            0 0.0 ${pi/2} -${pi/2} 0</pose>
+          <horizontal_fov>${70 * pi/180.0}</horizontal_fov>
           <image>
             <width>640</width>
@@ -54,5 +57,5 @@
           </ros>
           <camera_name>${cam_name}</camera_name>
-          <hack_baseline>0.07</hack_baseline>
+          <!-- <hack_baseline>0.07</hack_baseline> -->
           <min_depth>0.002</min_depth>
           <max_depth>300.0</max_depth>

Commit message: make robot following tag

File: src/follow_me_robot/urdf/robot.urdf.xacro (robot description, xacro)
@@ -54,5 +54,5 @@
 			<publish_rate>0</publish_rate>
 		</plugin>
-		<!-- <plugin name="gazebo_ros_joint_state_publisher"
+		<plugin name="gazebo_ros_joint_state_publisher"
 			filename="libgazebo_ros_joint_state_publisher.so">
 			<update_rate>${update_rate}</update_rate>
@@ -61,5 +61,5 @@
 			<joint_name>back_left_wheel_joint</joint_name>
 			<joint_name>back_right_wheel_joint</joint_name>
-		</plugin> -->
+		</plugin>
 	</gazebo>
 	<xacro:include filename="sensors/lidar.xacro" />
@@ -76,4 +76,5 @@
 		<!-- <origin xyz="${body_length/2} 0 0.1" rpy="${pi/2} 0 ${pi/2}" /> -->
 		<origin xyz="${body_length/2} 0 0.1" rpy="0 -0.3 0" />
+		<!-- <origin xyz="${body_length/2} 0 0.1" rpy="0 0 0" /> -->
 		<!-- <origin xyz="${body_length/2} 0 0.1" rpy="0 -0.3 ${pi/2}" /> -->
 	</xacro:camera>

Commit message: fix code and configs

File: src/follow_me_robot/urdf/robot.urdf.xacro (robot description, xacro)
@@ -74,8 +74,5 @@
 	<xacro:camera cam_name="front" parent="base_link" update="15"
 		visualize="true">
-		<!-- <origin xyz="${body_length/2} 0 0.1" rpy="${pi/2} 0 ${pi/2}" /> -->
-		<origin xyz="${body_length/2} 0 0.1" rpy="0 -0.3 0" />
-		<!-- <origin xyz="${body_length/2} 0 0.1" rpy="0 0 0" /> -->
-		<!-- <origin xyz="${body_length/2} 0 0.1" rpy="0 -0.3 ${pi/2}" /> -->
+		<origin xyz="${body_length/2} 0 0.1" rpy="0 -0.35 0" />
 	</xacro:camera>
 	<xacro:include filename="sensors/sonar.xacro" />
@@ -84,7 +81,3 @@
 		<origin xyz="${body_length/2} 0 -0.05" rpy="0 0.2 0" />
 	</xacro:sonar>
-	<!-- <xacro:include filename="sensors/gps.xacro" /> -->
-	<!-- <xacro:gps parent="base_link" update="${update_rate}">
-		<origin xyz="0 0 0.0" />
-	</xacro:gps> -->
 </robot>

File: src/follow_me_robot/urdf/sensors/camera.xacro (robot description, xacro)
@@ -56,5 +56,4 @@
           </ros>
           <camera_name>${cam_name}</camera_name>
-          <!-- <hack_baseline>0.07</hack_baseline> -->
           <min_depth>0.002</min_depth>
           <max_depth>300.0</max_depth>
